Commit message: updating URDFs

File: robotiq_hande_gripper_description/urdf/hande_gripper_hros_support.urdf.xacro (robot description, xacro)
@@ -1,103 +1,44 @@
 <?xml version="1.0"?>
-<robot xmlns:xacro="http://ros.org/wiki/xacro">
-  <xacro:macro name="robotiq_hande"  params="prefix">
-    <link name="robotiq_hande_base_link">
-      <inertial>
-        <origin xyz="8.625E-08 -4.6583E-06 0.03145" rpy="0 0 0" />
-        <mass value="0.22652" />
-        <inertia ixx="0.00020005" ixy="0" ixz="0" iyy="0.00017832" iyz="0" izz="0.00013478" />
-      </inertial>
-      <visual>
-        <origin xyz="0 0 0" rpy="0 0 1.57" />
-        <geometry>
-          <mesh filename="package://robotiq_hande_gripper_description/meshes/hand-e.dae" scale="0.001 0.001 0.001"/>
-        </geometry>
-        <material name="">
-          <color rgba="0.1 0.1 0.1 1" />
-        </material>
-      </visual>
-      <collision>
-        <origin xyz="0 0 0" rpy="0 0 1.57" />
-        <geometry>
-          <mesh filename="package://robotiq_hande_gripper_description/meshes/hand-e.dae" scale="0.001 0.001 0.001"/>
-        </geometry>
-      </collision>
-    </link>
-    <gazebo reference="robotiq_hande_base_link">
-      <material>Gazebo/Grey</material>
-      <selfCollide>True</selfCollide>
-    </gazebo>
-    <link name="finger1">
-      <inertial>
-        <origin rpy="0 0 0" xyz="8.625E-08 -4.6583E-06 0.03145"/>
-        <mass value="0.22652"/>
-        <inertia ixx="0.00020005" ixy="0" ixz="0" iyy="0.00017832" iyz="0" izz="0.00013478"/>
-      </inertial>
-      <visual>
-        <origin rpy="0 0 1.57" xyz="0 0 0"/>
-        <geometry>
-          <mesh filename="package://robotiq_hande_gripper_description/meshes/finger_1.dae" scale="0.001 0.001 0.001"/>
-        </geometry>
-        <material name="">
-          <color rgba="0.1 0.1 0.1 1"/>
-        </material>
-      </visual>
-      <collision>
-        <origin rpy="0 0 1.57" xyz="0 0 0"/>
-        <geometry>
-          <mesh filename="package://robotiq_hande_gripper_description/meshes/finger_1.dae" scale="0.001 0.001 0.001"/>
-        </geometry>
-      </collision>
-    </link>
-    <gazebo reference="finger1">
-      <material>Gazebo/Grey</material>
-      <selfCollide>True</selfCollide>
-    </gazebo>
-    <link name="finger2">
-      <inertial>
-        <origin rpy="0 0 0" xyz="8.625E-08 -4.6583E-06 0.03145"/>
-        <mass value="0.22652"/>
-        <inertia ixx="0.00020005" ixy="0" ixz="0" iyy="0.00017832" iyz="0" izz="0.00013478"/>
-      </inertial>
-      <visual>
-        <origin rpy="0 0 1.57" xyz="0 0 0"/>
-        <geometry>
-          <mesh filename="package://robotiq_hande_gripper_description/meshes/finger_2.dae" scale="0.001 0.001 0.001"/>
-        </geometry>
-        <material name="">
-          <color rgba="0.1 0.1 0.1 1"/>
-        </material>
-      </visual>
-      <collision>
-        <origin rpy="0 0 1.57" xyz="0 0 0"/>
-        <geometry>
-          <mesh filename="package://robotiq_hande_gripper_description/meshes/finger_2.dae" scale="0.001 0.001 0.001"/>
-        </geometry>
-      </collision>
-    </link>
-    <gazebo reference="finger2">
-      <material>Gazebo/Grey</material>
-      <selfCollide>True</selfCollide>
-    </gazebo>
-    <gazebo>
-      <plugin filename="librobotiq_linear_gripper_gazebo_plugin.so" name="robotiq_hande_gripper">
-        <left_joint>finger1_joint</left_joint>
-        <right_joint>finger2_joint</right_joint>
-      </plugin>
-    </gazebo>
-    <joint name="finger1_joint" type="prismatic">
-      <origin rpy="0 0 0" xyz="0 0 0.0"/>
-      <parent link="robotiq_hande_base_link"/>
-      <child link="finger1"/>
-      <axis xyz="0 0 -1"/>
-      <limit effort="1000" lower="0" upper="0.024858" velocity="2.0"/>
-    </joint>
-    <joint name="finger2_joint" type="prismatic">
-      <origin rpy="0 0 0" xyz="0 0 0.0"/>
-      <parent link="robotiq_hande_base_link"/>
-      <child link="finger2"/>
-      <axis xyz="0 0 1"/>
-      <limit effort="1000" lower="0" upper="0.024858" velocity="2.0"/>
-    </joint>
-  </xacro:macro>
+<robot xmlns:xacro="http://ros.org/wiki/xacro"
+       name="robotiq_hande" >
+  <!-- robotiq hande_gripper -->
+  <xacro:include filename="$(find robotiq_hande_gripper_description)/urdf/robotiq_hande.urdf.xacro" />
+  <xacro:robotiq_hande prefix=""/>
+  <link name="world" />
+  <link name="robotiq_adapter_link">
+    <inertial>
+      <origin xyz="8.625E-08 -4.6583E-06 0.03145" rpy="0 0 0" />
+      <mass value="0.22652" />
+      <inertia ixx="0.00020005" ixy="0" ixz="0" iyy="0.00017832" iyz="0" izz="0.00013478" />
+    </inertial>
+    <visual>
+      <origin xyz="0 0 0" rpy="0 0 1.57" />
+      <geometry>
+        <mesh filename="package://robotiq_hande_gripper_description/meshes/hros_robotiq_adapter.dae" scale="0.001 0.001 0.001"/>
+      </geometry>
+      <material name="Gazebo/Black">
+        <color rgba="0.1 0.1 0.1 1" />
+      </material>
+    </visual>
+    <collision>
+      <origin xyz="0 0 0" rpy="0 0 1.57" />
+      <geometry>
+        <mesh filename="package://robotiq_hande_gripper_description/meshes/hros_robotiq_adapter.dae" scale="0.001 0.001 0.001"/>
+      </geometry>
+    </collision>
+  </link>
+  <gazebo reference="robotiq_adapter_link">
+    <material>Gazebo/Black</material>
+    <selfCollide>False</selfCollide>
+  </gazebo>
+  <joint name="base_adapter_to_base_robotiq_joint" type="fixed">
+    <origin rpy="0 1.57 0" xyz=" 0 0 0.10653"/>
+    <parent link="robotiq_adapter_link" />
+    <child link="robotiq_hande_base_link"/>
+  </joint>
+  <joint name="world_to_hande_joint" type="fixed">
+    <origin rpy="0 0 0" xyz="0 0 0.5"/>
+    <parent link="world"/>
+    <child link="robotiq_adapter_link"/>
+  </joint>
 </robot>

File: robotiq_hande_gripper_description/urdf/robotiq_hande.urdf (robot description, URDF)
Before this commit: robot robotiq_hande, 4 links, 3 joints
Links:
- added link robotiq_adapter_link, mass 0.22652; collision mesh filename=package://robotiq_hande_gripper_description/meshes/hros_rob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 scale=0.001 0.001 0.001; visual mesh filename=package://robotiq_hande_gripper_description/meshes/hros_rob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 scale=0.001 0.001 0.001
Joints:
- added joint base_adapter_to_base_robotiq_joint: type fixed, parent robotiq_adapter_link, child robotiq_hande_base_link, origin xyz= 0 0 0.10653 rpy=0 1.57 0
- joint world_to_hande_joint: child robotiq_hande_base_link -> robotiq_adapter_link; origin xyz=0 0 0.5 rpy=0 1.57 0 -> xyz=0 0 0.5 rpy=0 0 0

File: robotiq_hande_gripper_description/urdf/robotiq_hande.urdf.xacro (robot description, xacro)
@@ -86,13 +86,17 @@
       </plugin>
     </gazebo>
-    <joint name="finger1_joint" type="fixed">
+    <joint name="finger1_joint" type="prismatic">
       <origin rpy="0 0 0" xyz="0 0 0.0"/>
       <parent link="robotiq_hande_base_link"/>
       <child link="finger1"/>
+      <axis xyz="0 0 -1"/>
+      <limit effort="1000" lower="0" upper="0.024858" velocity="2.0"/>
     </joint>
-    <joint name="finger2_joint" type="fixed">
+    <joint name="finger2_joint" type="prismatic">
       <origin rpy="0 0 0" xyz="0 0 0.0"/>
       <parent link="robotiq_hande_base_link"/>
       <child link="finger2"/>
+      <axis xyz="0 0 1"/>
+      <limit effort="1000" lower="0" upper="0.024858" velocity="2.0"/>
     </joint>
   </xacro:macro>
