Commit message: changing finger  joint names

File: robotiq_hande_gripper_description/urdf/robotiq_hande.urdf.xacro (robot description, xacro)
@@ -82,9 +82,9 @@
     <gazebo>
       <plugin filename="librobotiq_linear_gripper_gazebo_plugin.so" name="robotiq_hande_gripper">
-        <left_joint>finger1_joint</left_joint>
+        <left_joint>joint_finger</left_joint>
         <right_joint>finger2_joint</right_joint>
       </plugin>
     </gazebo>
-    <joint name="finger1_joint" type="prismatic">
+    <joint name="joint_finger" type="prismatic">
       <origin rpy="0 0 0" xyz="0 0 0.0"/>
       <parent link="robotiq_hande_base_link"/>
@@ -99,4 +99,5 @@
       <axis xyz="0 0 1"/>
       <limit effort="1000" lower="0" upper="0.024858" velocity="2.0"/>
+      <mimic joint="joint_finger" multiplier="1" offset="0"/>
     </joint>
   </xacro:macro>
