Commit message: HANDE Updated URDF model

File: robotiq_hande_gripper_description/urdf/robotiq_hande.urdf (robot description, URDF)
Before this commit: robot robotiq_hande, 5 links, 4 joints
Links:
- removed link finger1
- removed link finger2
- removed link robotiq_adapter_link
- removed link robotiq_hande_base_link
- removed link world
Joints:
- removed joint base_adapter_to_base_robotiq_joint
- removed joint finger1_joint
- removed joint finger2_joint
- removed joint world_to_hande_joint

File: robotiq_hande_gripper_description/urdf/robotiq_hande.urdf.xacro (robot description, xacro)
@@ -2,4 +2,30 @@
 <robot xmlns:xacro="http://ros.org/wiki/xacro">
   <xacro:macro name="robotiq_hande"  params="prefix">
+    <link name="robotiq_adapter_link">
+      <inertial>
+        <origin xyz="8.625E-08 -4.6583E-06 0.03145" rpy="0 0 0" />
+        <mass value="0.22652" />
+        <inertia ixx="0.00020005" ixy="0" ixz="0" iyy="0.00017832" iyz="0" izz="0.00013478" />
+      </inertial>
+      <visual>
+        <origin xyz="0 0 0" rpy="0 0 1.57" />
+        <geometry>
+          <mesh filename="package://robotiq_hande_gripper_description/meshes/hros_robotiq_adapter.dae" scale="0.001 0.001 0.001"/>
+        </geometry>
+        <material name="Gazebo/Black">
+          <color rgba="0.0 0.0 0.0 1" />
+        </material>
+      </visual>
+      <collision>
+        <origin xyz="0 0 0" rpy="0 0 1.57" />
+        <geometry>
+          <mesh filename="package://robotiq_hande_gripper_description/meshes/hros_robotiq_adapter.dae" scale="0.001 0.001 0.001"/>
+        </geometry>
+      </collision>
+    </link>
+    <gazebo reference="robotiq_adapter_link">
+      <material>Gazebo/Black</material>
+      <selfCollide>False</selfCollide>
+    </gazebo>
     <link name="robotiq_hande_base_link">
       <inertial>
@@ -89,4 +115,9 @@
       </plugin>
     </gazebo>
+    <joint name="base_adapter_to_base_robotiq_joint" type="fixed">
+      <origin rpy="0 1.57 0" xyz=" 0 0 0.10653"/>
+      <parent link="robotiq_adapter_link" />
+      <child link="robotiq_hande_base_link"/>
+    </joint>
     <joint name="joint_finger" type="prismatic">
       <origin rpy="0 0 0" xyz="0 0 0.0"/>

Commit message: update dae files of the hande

File: robotiq_hande_gripper_description/urdf/robotiq_hande.urdf (robot description, URDF)
Before this commit: robot robotiq_hande, 5 links, 4 joints
Links:
- removed link robotiq_adapter_link
Joints:
- removed joint base_adapter_to_base_robotiq_joint
- removed joint world_to_hande_joint
- added joint world_to_robotiq_adapter: type fixed, parent world, child robotiq_hande_base_link, origin xyz=0 0 0.5 rpy=0 0 0
- joint finger2_joint: axis 0 0 1 -> 1 0 0; limit lower=0 upper=0.024858 effort=1000 velocity=2.0 -> lower=0 upper=0.025 effort=130 velocity=0.15; origin xyz=0 0 0.0 rpy=0 0 0 -> xyz=0 0 0.099 rpy=0 0 0
- joint joint_finger: axis 0 0 -1 -> -1 0 0; limit lower=0 upper=0.024858 effort=1000 velocity=2.0 -> lower=0 upper=0.025 effort=130 velocity=0.15; origin xyz=0 0 0.0 rpy=0 0 0 -> xyz=0 0 0.099 rpy=0 0 0

File: robotiq_hande_gripper_description/urdf/robotiq_hande.urdf.xacro (robot description, xacro)
@@ -2,30 +2,4 @@
 <robot xmlns:xacro="http://ros.org/wiki/xacro">
   <xacro:macro name="robotiq_hande"  params="prefix">
-    <link name="robotiq_adapter_link">
-      <inertial>
-        <origin xyz="8.625E-08 -4.6583E-06 0.03145" rpy="0 0 0" />
-        <mass value="0.22652" />
-        <inertia ixx="0.00020005" ixy="0" ixz="0" iyy="0.00017832" iyz="0" izz="0.00013478" />
-      </inertial>
-      <visual>
-        <origin xyz="0 0 0" rpy="0 0 1.57" />
-        <geometry>
-          <mesh filename="package://robotiq_hande_gripper_description/meshes/hros_robotiq_adapter.dae" scale="0.001 0.001 0.001"/>
-        </geometry>
-        <material name="Gazebo/Black">
-          <color rgba="0.0 0.0 0.0 1" />
-        </material>
-      </visual>
-      <collision>
-        <origin xyz="0 0 0" rpy="0 0 1.57" />
-        <geometry>
-          <mesh filename="package://robotiq_hande_gripper_description/meshes/hros_robotiq_adapter.dae" scale="0.001 0.001 0.001"/>
-        </geometry>
-      </collision>
-    </link>
-    <gazebo reference="robotiq_adapter_link">
-      <material>Gazebo/Black</material>
-      <selfCollide>False</selfCollide>
-    </gazebo>
     <link name="robotiq_hande_base_link">
       <inertial>
@@ -35,5 +9,5 @@
       </inertial>
       <visual>
-        <origin xyz="0 0 0" rpy="0 0 1.57" />
+        <origin xyz="0 0 0" rpy="0 0 0" />
         <geometry>
           <mesh filename="package://robotiq_hande_gripper_description/meshes/hand-e.dae" scale="0.001 0.001 0.001"/>
@@ -44,5 +18,5 @@
       </visual>
       <collision>
-        <origin xyz="0 0 0" rpy="0 0 1.57" />
+        <origin xyz="0 0 0" rpy="0 0 0" />
         <geometry>
           <mesh filename="package://robotiq_hande_gripper_description/meshes/hand-e.dae" scale="0.001 0.001 0.001"/>
@@ -61,5 +35,5 @@
       </inertial>
       <visual>
-        <origin rpy="0 0 1.57" xyz="0 0 0"/>
+        <origin rpy="0 0 0" xyz="0 0 0"/>
         <geometry>
           <mesh filename="package://robotiq_hande_gripper_description/meshes/finger_1.dae" scale="0.001 0.001 0.001"/>
@@ -70,5 +44,5 @@
       </visual>
       <collision>
-        <origin rpy="0 0 1.57" xyz="0 0 0"/>
+        <origin rpy="0 0 0" xyz="0 0 0"/>
         <geometry>
           <mesh filename="package://robotiq_hande_gripper_description/meshes/finger_1.dae" scale="0.001 0.001 0.001"/>
@@ -87,5 +61,5 @@
       </inertial>
       <visual>
-        <origin rpy="0 0 1.57" xyz="0 0 0"/>
+        <origin rpy="0 0 0" xyz="0 0 0"/>
         <geometry>
           <mesh filename="package://robotiq_hande_gripper_description/meshes/finger_2.dae" scale="0.001 0.001 0.001"/>
@@ -96,5 +70,5 @@
       </visual>
       <collision>
-        <origin rpy="0 0 1.57" xyz="0 0 0"/>
+        <origin rpy="0 0 0" xyz="0 0 0"/>
         <geometry>
           <mesh filename="package://robotiq_hande_gripper_description/meshes/finger_2.dae" scale="0.001 0.001 0.001"/>
@@ -106,4 +80,19 @@
       <selfCollide>True</selfCollide>
     </gazebo>
+    <joint name="joint_finger" type="prismatic">
+      <origin rpy="0 0 0" xyz="0 0 0.099"/>
+      <parent link="robotiq_hande_base_link"/>
+      <child link="finger1"/>
+      <axis xyz="-1 0 0"/>
+      <limit effort="130" lower="0" upper="0.025" velocity="0.15"/>
+    </joint>
+    <joint name="finger2_joint" type="prismatic">
+      <origin rpy="0 0 0" xyz="0 0 0.099"/>
+      <parent link="robotiq_hande_base_link"/>
+      <child link="finger2"/>
+      <axis xyz="1 0 0"/>
+      <limit effort="130" lower="0" upper="0.025" velocity="0.15"/>
+      <mimic joint="joint_finger" multiplier="1" offset="0"/>
+    </joint>
     <gazebo>
       <plugin filename="librobotiq_gripper_gazebo_plugin.so" name="hrim_actuation_gripper_000000000004">
@@ -122,24 +111,4 @@
       </plugin>
     </gazebo>
-    <joint name="base_adapter_to_base_robotiq_joint" type="fixed">
-      <origin rpy="0 1.57 0" xyz=" 0 0 0.10653"/>
-      <parent link="robotiq_adapter_link" />
-      <child link="robotiq_hande_base_link"/>
-    </joint>
-    <joint name="joint_finger" type="prismatic">
-      <origin rpy="0 0 0" xyz="0 0 0.0"/>
-      <parent link="robotiq_hande_base_link"/>
-      <child link="finger1"/>
-      <axis xyz="0 0 -1"/>
-      <limit effort="1000" lower="0" upper="0.024858" velocity="2.0"/>
-    </joint>
-    <joint name="finger2_joint" type="prismatic">
-      <origin rpy="0 0 0" xyz="0 0 0.0"/>
-      <parent link="robotiq_hande_base_link"/>
-      <child link="finger2"/>
-      <axis xyz="0 0 1"/>
-      <limit effort="1000" lower="0" upper="0.024858" velocity="2.0"/>
-      <mimic joint="joint_finger" multiplier="1" offset="0"/>
-    </joint>
   </xacro:macro>
 </robot>

File: robotiq_hande_gripper_description/urdf/robotiq_hande_world.urdf.xacro (robot description, xacro)
@@ -1,13 +1,12 @@
 <?xml version="1.0"?>
-<robot xmlns:xacro="http://ros.org/wiki/xacro"
-       name="robotiq_hande" >
-  <!-- robotiq hande_gripper -->
+<robot xmlns:xacro="http://ros.org/wiki/xacro" name="robotiq_hande" >
+  <!-- robotiq_hande_gripper -->
   <xacro:include filename="$(find robotiq_hande_gripper_description)/urdf/robotiq_hande.urdf.xacro" />
   <xacro:robotiq_hande prefix=""/>
   <link name="world" />
-  <joint name="world_to_hande_joint" type="fixed">
+  <joint name="world_to_robotiq_adapter" type="fixed">
     <origin rpy="0 0 0" xyz="0 0 0.5"/>
     <parent link="world"/>
-    <child link="robotiq_adapter_link"/>
+    <child link="robotiq_hande_base_link"/>
   </joint>
 </robot>

Commit message: fix inertial values of the hande

File: robotiq_hande_gripper_description/urdf/robotiq_hande.urdf (robot description, URDF)
Before this commit: robot robotiq_hande, 4 links, 3 joints
Links:
- removed link finger1
- removed link finger2
- added link left_finger, mass 0.03804; collision mesh filename=package://robotiq_hande_gripper_description/meshes/finger_1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 scale=0.001 0.001 0.001; visual mesh filename=package://robotiq_hande_gripper_description/meshes/finger_1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 scale=0.001 0.001 0.001
- added link right_finger, mass 0.03804; collision mesh filename=package://robotiq_hande_gripper_description/meshes/finger_2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 scale=0.001 0.001 0.001; visual mesh filename=package://robotiq_hande_gripper_description/meshes/finger_2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 scale=0.001 0.001 0.001
- link robotiq_hande_base_link: mass 0.22652 -> 0.86387
Joints:
- removed joint finger2_joint
- added joint robotiq_hande_base_to_right_finger: type prismatic, parent robotiq_hande_base_link, child right_finger, origin xyz=0 0 0.099 rpy=0 0 0, axis 1 0 0, limit lower=0 upper=0.025 effort=130 velocity=0.15, mimic joint=joint_finger multiplier=1 offset=0
- joint joint_finger: child finger1 -> left_finger

File: robotiq_hande_gripper_description/urdf/robotiq_hande.urdf.xacro (robot description, xacro)
@@ -4,7 +4,7 @@
     <link name="robotiq_hande_base_link">
       <inertial>
-        <origin xyz="8.625E-08 -4.6583E-06 0.03145" rpy="0 0 0" />
-        <mass value="0.22652" />
-        <inertia ixx="0.00020005" ixy="0" ixz="0" iyy="0.00017832" iyz="0" izz="0.00013478" />
+        <origin xyz="0 0 0.04607" rpy="0 0 0" />
+        <mass value="0.86387" />
+        <inertia ixx="1017560E-9" ixy="0" ixz="2235E-9" iyy="1028041E-9" iyz="0" izz="489810E-9" />
       </inertial>
       <visual>
@@ -28,9 +28,9 @@
       <selfCollide>True</selfCollide>
     </gazebo>
-    <link name="finger1">
+    <link name="left_finger">
       <inertial>
-        <origin rpy="0 0 0" xyz="8.625E-08 -4.6583E-06 0.03145"/>
-        <mass value="0.22652"/>
-        <inertia ixx="0.00020005" ixy="0" ixz="0" iyy="0.00017832" iyz="0" izz="0.00013478"/>
+        <origin rpy="0 0 0" xyz="0.02262 -0.00759 0.00738"/>
+        <mass value="0.03804"/>
+        <inertia ixx="13567E-9" ixy="1849E-9" ixz="3622E-9" iyy="15784E-9" iyz="3616E-9" izz="7478E-9"/>
       </inertial>
       <visual>
@@ -50,13 +50,13 @@
       </collision>
     </link>
-    <gazebo reference="finger1">
+    <gazebo reference="left_finger">
       <material>Gazebo/Grey</material>
       <selfCollide>True</selfCollide>
     </gazebo>
-    <link name="finger2">
+    <link name="right_finger">
       <inertial>
-        <origin rpy="0 0 0" xyz="8.625E-08 -4.6583E-06 0.03145"/>
-        <mass value="0.22652"/>
-        <inertia ixx="0.00020005" ixy="0" ixz="0" iyy="0.00017832" iyz="0" izz="0.00013478"/>
+        <origin rpy="0 0 0" xyz="-0.02262 0.00759 0.00738"/>
+        <mass value="0.03804"/>
+        <inertia ixx="13567E-9" ixy="1849E-9" ixz="-3622E-9" iyy="15784E-9" iyz="-3616E-9" izz="7478E-9"/>
       </inertial>
       <visual>
@@ -76,5 +76,5 @@
       </collision>
     </link>
-    <gazebo reference="finger2">
+    <gazebo reference="right_finger">
       <material>Gazebo/Grey</material>
       <selfCollide>True</selfCollide>
@@ -83,12 +83,12 @@
       <origin rpy="0 0 0" xyz="0 0 0.099"/>
       <parent link="robotiq_hande_base_link"/>
-      <child link="finger1"/>
+      <child link="left_finger"/>
       <axis xyz="-1 0 0"/>
       <limit effort="130" lower="0" upper="0.025" velocity="0.15"/>
     </joint>
-    <joint name="finger2_joint" type="prismatic">
+    <joint name="robotiq_hande_base_to_right_finger" type="prismatic">
       <origin rpy="0 0 0" xyz="0 0 0.099"/>
       <parent link="robotiq_hande_base_link"/>
-      <child link="finger2"/>
+      <child link="right_finger"/>
       <axis xyz="1 0 0"/>
       <limit effort="130" lower="0" upper="0.025" velocity="0.15"/>
@@ -99,7 +99,7 @@
         <kp>10</kp>
         <ki>3</ki>
-        <kd>5</kd>
+        <kd>9</kd>
         <joint>joint_finger</joint>
-        <joint>finger2_joint</joint>
+        <joint>robotiq_hande_base_to_right_finger</joint>
       </plugin>
       <plugin filename="libgazebo_ros_joint_state_publisher.so" name="mara_joint_state">
