Commit message: Remove left/right joint distinction from gripper plugin

File: robotiq_140_gripper_description/urdf/robotiq_140.urdf.xacro (robot description, xacro)
@@ -359,8 +359,8 @@
       </joint>
       <plugin filename="librobotiq_gripper_gazebo_plugin.so" name="robotiq_140_gripper">
-        <left_joint>left_inner_knuckle_joint</left_joint>
-        <left_joint>left_outer_knuckle_joint</left_joint>
-        <right_joint>right_inner_knuckle_joint</right_joint>
-        <right_joint>joint_finger</right_joint>
+        <joint>left_inner_knuckle_joint</joint>
+        <joint>left_outer_knuckle_joint</joint>
+        <joint>right_inner_knuckle_joint</joint>
+        <joint>joint_finger</joint>
       </plugin>
     </gazebo>

File: robotiq_85_gripper_description/urdf/robotiq_85.urdf.xacro (robot description, xacro)
@@ -323,8 +323,8 @@
       </joint>
       <plugin filename="librobotiq_gripper_gazebo_plugin.so" name="robotiq_85_gripper">
-        <left_joint>left_inner_knuckle_joint</left_joint>
-        <left_joint>left_outer_knuckle_joint</left_joint>
-        <right_joint>right_inner_knuckle_joint</right_joint>
-        <right_joint>joint_finger</right_joint>
+        <joint>left_inner_knuckle_joint</joint>
+        <joint>left_outer_knuckle_joint</joint>
+        <joint>right_inner_knuckle_joint</joint>
+        <joint>joint_finger</joint>
       </plugin>
     </gazebo>

File: robotiq_hande_gripper_description/urdf/robotiq_hande.urdf.xacro (robot description, xacro)
@@ -85,6 +85,6 @@
         <ki>3</ki>
         <kd>5</kd>
-        <left_joint>joint_finger</left_joint>
-        <right_joint>finger2_joint</right_joint>
+        <joint>joint_finger</joint>
+        <joint>finger2_joint</joint>
       </plugin>
     </gazebo>

Commit message: Updating robotiq 140

File: robotiq_140_gripper_description/urdf/robotiq_140.urdf.xacro (robot description, xacro)
@@ -2,4 +2,35 @@
 <robot xmlns:xacro="http://ros.org/wiki/xacro">
   <xacro:macro name="robotiq_gripper"  params="prefix">
+    <link name="robotiq_adapter_link">
+      <inertial>
+        <origin xyz="8.625E-08 -4.6583E-06 0.03145" rpy="0 0 0" />
+        <mass value="0.22652" />
+        <inertia ixx="0.00020005" ixy="0" ixz="0" iyy="0.00017832" iyz="0" izz="0.00013478" />
+      </inertial>
+      <visual>
+        <origin xyz="0 0 0" rpy="0 0 1.57" />
+        <geometry>
+          <mesh filename="package://robotiq_140_gripper_description/meshes/hros_robotiq_adapter.dae" scale="0.001 0.001 0.001"/>
+        </geometry>
+        <material name="Gazebo/Black">
+          <color rgba="0.0 0.0 0.0 1" />
+        </material>
+      </visual>
+      <collision>
+        <origin xyz="0 0 0" rpy="0 0 1.57" />
+        <geometry>
+          <mesh filename="package://robotiq_140_gripper_description/meshes/hros_robotiq_adapter.dae" scale="0.001 0.001 0.001"/>
+        </geometry>
+      </collision>
+    </link>
+    <gazebo reference="robotiq_adapter_link">
+      <material>Gazebo/Black</material>
+      <selfCollide>False</selfCollide>
+    </gazebo>
+    <joint name="base_adapter_to_base_robotiq_joint" type="fixed">
+      <origin rpy="0 0 0" xyz=" 0 0 0.03653"/>
+      <parent link="robotiq_adapter_link" />
+      <child link="robotiq_arg2f_base_link"/>
+    </joint>
     <link name="robotiq_arg2f_base_link">
       <inertial>

Commit message: Adding motor state publisher and changing the name of the topics

File: robotiq_140_gripper_description/urdf/robotiq_140.urdf.xacro (robot description, xacro)
@@ -389,5 +389,5 @@
         </axis>
       </joint>
-      <plugin filename="librobotiq_gripper_gazebo_plugin.so" name="robotiq_140_gripper">
+      <plugin filename="librobotiq_gripper_gazebo_plugin.so" name="hrim_actuation_gripper_000000000004">
         <joint>left_inner_knuckle_joint</joint>
         <joint>left_outer_knuckle_joint</joint>
@@ -395,4 +395,11 @@
         <joint>joint_finger</joint>
       </plugin>
+      <plugin filename="libgazebo_ros_joint_state_publisher.so" name="mara_joint_state">
+        <ros>
+          <argument>~/out:=joint_states</argument>
+        </ros>
+        <update_rate>25</update_rate>
+        <joint_name>joint_finger</joint_name>
+      </plugin>
     </gazebo>
   </xacro:macro>

File: robotiq_85_gripper_description/urdf/robotiq_85.urdf.xacro (robot description, xacro)
@@ -353,5 +353,5 @@
         </axis>
       </joint>
-      <plugin filename="librobotiq_gripper_gazebo_plugin.so" name="robotiq_85_gripper">
+      <plugin filename="librobotiq_gripper_gazebo_plugin.so" name="hrim_actuation_gripper_000000000004">
         <joint>left_inner_knuckle_joint</joint>
         <joint>left_outer_knuckle_joint</joint>
@@ -359,4 +359,11 @@
         <joint>joint_finger</joint>
       </plugin>
+      <plugin filename="libgazebo_ros_joint_state_publisher.so" name="mara_joint_state">
+        <ros>
+          <argument>~/out:=joint_states</argument>
+        </ros>
+        <update_rate>25</update_rate>
+        <joint_name>joint_finger</joint_name>
+      </plugin>
     </gazebo>
   </xacro:macro>

File: robotiq_hande_gripper_description/urdf/hande_gripper_hros_support.urdf.xacro (robot description, xacro)
@@ -6,35 +6,4 @@
   <xacro:robotiq_hande prefix=""/>
   <link name="world" />
-  <link name="robotiq_adapter_link">
-    <inertial>
-      <origin xyz="8.625E-08 -4.6583E-06 0.03145" rpy="0 0 0" />
-      <mass value="0.22652" />
-      <inertia ixx="0.00020005" ixy="0" ixz="0" iyy="0.00017832" iyz="0" izz="0.00013478" />
-    </inertial>
-    <visual>
-      <origin xyz="0 0 0" rpy="0 0 1.57" />
-      <geometry>
-        <mesh filename="package://robotiq_hande_gripper_description/meshes/hros_robotiq_adapter.dae" scale="0.001 0.001 0.001"/>
-      </geometry>
-      <material name="Gazebo/Black">
-        <color rgba="0.1 0.1 0.1 1" />
-      </material>
-    </visual>
-    <collision>
-      <origin xyz="0 0 0" rpy="0 0 1.57" />
-      <geometry>
-        <mesh filename="package://robotiq_hande_gripper_description/meshes/hros_robotiq_adapter.dae" scale="0.001 0.001 0.001"/>
-      </geometry>
-    </collision>
-  </link>
-  <gazebo reference="robotiq_adapter_link">
-    <material>Gazebo/Black</material>
-    <selfCollide>False</selfCollide>
-  </gazebo>
-  <joint name="base_adapter_to_base_robotiq_joint" type="fixed">
-    <origin rpy="0 1.57 0" xyz=" 0 0 0.10653"/>
-    <parent link="robotiq_adapter_link" />
-    <child link="robotiq_hande_base_link"/>
-  </joint>
   <joint name="world_to_hande_joint" type="fixed">
     <origin rpy="0 0 0" xyz="0 0 0.5"/>

File: robotiq_hande_gripper_description/urdf/robotiq_hande.urdf (robot description, URDF)
Before this commit: robot None, 0 links, 0 joints
Links:
- added link finger1, mass 0.22652; collision mesh filename=package://robotiq_hande_gripper_description/meshes/finger_1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 scale=0.001 0.001 0.001; visual mesh filename=package://robotiq_hande_gripper_description/meshes/finger_1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 scale=0.001 0.001 0.001
- added link finger2, mass 0.22652; collision mesh filename=package://robotiq_hande_gripper_description/meshes/finger_2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 scale=0.001 0.001 0.001; visual mesh filename=package://robotiq_hande_gripper_description/meshes/finger_2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 scale=0.001 0.001 0.001
- added link robotiq_adapter_link, mass 0.22652; collision mesh filename=package://robotiq_hande_gripper_description/meshes/hros_rob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 scale=0.001 0.001 0.001; visual mesh filename=package://robotiq_hande_gripper_description/meshes/hros_rob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 scale=0.001 0.001 0.001
- added link robotiq_hande_base_link, mass 0.22652; collision mesh filename=package://robotiq_hande_gripper_description/meshes/hand-e.d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 scale=0.001 0.001 0.001; visual mesh filename=package://robotiq_hande_gripper_description/meshes/hand-e.d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 scale=0.001 0.001 0.001
- added link world
Joints:
- added joint base_adapter_to_base_robotiq_joint: type fixed, parent robotiq_adapter_link, child robotiq_hande_base_link, origin xyz= 0 0 0.10653 rpy=0 1.57 0
- added joint finger2_joint: type prismatic, parent robotiq_hande_base_link, child finger2, origin xyz=0 0 0.0 rpy=0 0 0, axis 0 0 1, limit lower=0 upper=0.024858 effort=1000 velocity=2.0, mimic joint=joint_finger multiplier=1 offset=0
- added joint joint_finger: type prismatic, parent robotiq_hande_base_link, child finger1, origin xyz=0 0 0.0 rpy=0 0 0, axis 0 0 -1, limit lower=0 upper=0.024858 effort=1000 velocity=2.0
- added joint world_to_hande_joint: type fixed, parent world, child robotiq_adapter_link, origin xyz=0 0 0.5 rpy=0 0 0

File: robotiq_hande_gripper_description/urdf/robotiq_hande.urdf.xacro (robot description, xacro)
@@ -107,5 +107,5 @@
     </gazebo>
     <gazebo>
-      <plugin filename="librobotiq_gripper_gazebo_plugin.so" name="robotiq_hande_gripper">
+      <plugin filename="librobotiq_gripper_gazebo_plugin.so" name="hrim_actuation_gripper_000000000004">
         <kp>10</kp>
         <ki>3</ki>
@@ -113,4 +113,11 @@
         <joint>joint_finger</joint>
         <joint>finger2_joint</joint>
+      </plugin>
+      <plugin filename="libgazebo_ros_joint_state_publisher.so" name="mara_joint_state">
+        <ros>
+          <argument>~/out:=joint_states</argument>
+        </ros>
+        <update_rate>25</update_rate>
+        <joint_name>joint_finger</joint_name>
       </plugin>
     </gazebo>

Commit message: rotate inertia and make only inner self collided false

File: robotiq_140_gripper_description/urdf/robotiq_140.urdf.xacro (robot description, xacro)
@@ -26,5 +26,5 @@
     <gazebo reference="robotiq_arg2f_base_link">
       <material>Gazebo/Black</material>
-      <selfCollide>False</selfCollide>
+      <selfCollide>True</selfCollide>
     </gazebo>
     <link name="left_outer_knuckle">
@@ -32,5 +32,5 @@
         <origin xyz="0.01616 0 -0.00133" rpy="0 0 0" />
         <mass value="0.0131" />
-        <inertia ixx="325.5E-9" ixy="0" ixz="-197.94E-9" iyy="2306.36E-9" iyz="0" izz="2176E-9" />
+        <inertia ixx="325.5E-9" ixy="0" ixz="197.94E-9" iyy="2306.36E-9" iyz="0" izz="2176E-9" />
       </inertial>
       <visual>
@@ -52,5 +52,5 @@
     <gazebo reference="left_outer_knuckle">
       <material>Gazebo/Grey</material>
-      <selfCollide>False</selfCollide>
+      <selfCollide>True</selfCollide>
     </gazebo>
     <link name="right_outer_knuckle">
@@ -58,5 +58,5 @@
         <origin xyz="-0.01616 0 -0.00133" rpy="0 0 0" />
         <mass value="0.0131" />
-        <inertia ixx="325.5E-9" ixy="0" ixz="197.94E-9" iyy="2306.36E-9" iyz="0" izz="2176E-9" />
+        <inertia ixx="325.5E-9" ixy="0" ixz="-197.94E-9" iyy="2306.36E-9" iyz="0" izz="2176E-9" />
       </inertial>
       <visual>
@@ -78,5 +78,5 @@
     <gazebo reference="right_outer_knuckle">
       <material>Gazebo/Grey</material>
-      <selfCollide>False</selfCollide>
+      <selfCollide>True</selfCollide>
     </gazebo>
     <link name="left_inner_knuckle">
@@ -84,5 +84,5 @@
         <origin xyz="0.03332 0 0.0379" rpy="0 0 0" />
         <mass value="0.04476" />
-        <inertia ixx="28054E-9" ixy="0" ixz="19174E-9" iyy="39758E-9" iyz="0" izz="23453E-9" />
+        <inertia ixx="28054E-9" ixy="0" ixz="-19174E-9" iyy="39758E-9" iyz="0" izz="23453E-9" />
       </inertial>
       <visual>
@@ -110,5 +110,5 @@
         <origin xyz="-0.03332 0 0.0379" rpy="0 0 0" />
         <mass value="0.04476" />
-        <inertia ixx="28054E-9" ixy="0" ixz="-19174E-9" iyy="39758E-9" iyz="0" izz="23453E-9" />
+        <inertia ixx="28054E-9" ixy="0" ixz="19174E-9" iyy="39758E-9" iyz="0" izz="23453E-9" />
       </inertial>
       <visual>
@@ -136,5 +136,5 @@
         <origin xyz="-0.01563 0 0.02522" rpy="0 0 0" />
         <mass value="0.045" />
-        <inertia ixx="26663E-9" ixy="0" ixz="-5579E-9" iyy="28009E-9" iyz="0" izz="4368E-9" />
+        <inertia ixx="26663E-9" ixy="0" ixz="5579E-9" iyy="28009E-9" iyz="0" izz="4368E-9" />
       </inertial>
       <visual>
@@ -162,5 +162,5 @@
         <origin xyz="0.01563 0 0.02522" rpy="0 0 0" />
         <mass value="0.045" />
-        <inertia ixx="26663E-9" ixy="0" ixz="5579E-9" iyy="28009E-9" iyz="0" izz="4368E-9" />
+        <inertia ixx="26663E-9" ixy="0" ixz="-5579E-9" iyy="28009E-9" iyz="0" izz="4368E-9" />
       </inertial>
       <visual>
@@ -188,5 +188,5 @@
         <origin xyz="0.01482 0 0.03451" rpy="0 0 0" />
         <mass value="0.07637" />
-        <inertia ixx="45513E-9" ixy="0" ixz="20691E-9" iyy="52570E-9" iyz="0" izz="17804E-9" />
+        <inertia ixx="45513E-9" ixy="0" ixz="-20691E-9" iyy="52570E-9" iyz="0" izz="17804E-9" />
       </inertial>
       <visual>
@@ -208,5 +208,5 @@
     <gazebo reference="left_outer_finger">
       <material>Gazebo/Black</material>
-      <selfCollide>False</selfCollide>
+      <selfCollide>True</selfCollide>
     </gazebo>
     <link name="right_outer_finger">
@@ -214,5 +214,5 @@
         <origin xyz="-0.01482 0 0.03451" rpy="0 0 0" />
         <mass value="0.07637" />
-        <inertia ixx="45513E-9" ixy="0" ixz="-20691E-9" iyy="52570E-9" iyz="0" izz="17804E-9" />
+        <inertia ixx="45513E-9" ixy="0" ixz="20691E-9" iyy="52570E-9" iyz="0" izz="17804E-9" />
       </inertial>
       <visual>
@@ -234,5 +234,5 @@
     <gazebo reference="right_outer_finger">
       <material>Gazebo/Black</material>
-      <selfCollide>False</selfCollide>
+      <selfCollide>True</selfCollide>
     </gazebo>
     <joint name="robotiq_arg2f_base_to_left_outer_knuckle" type="revolute">
