Commit message: update URDFs robotiq 140

File: robotiq_140_gripper_description/urdf/robotiq_140_hros_support.urdf.xacro (robot description, xacro)
@@ -1,398 +1,53 @@
 <?xml version="1.0"?>
-<robot xmlns:xacro="http://ros.org/wiki/xacro">
-  <xacro:macro name="robotiq_gripper"  params="prefix">
-    <link name="robotiq_adapter_link">
-      <inertial>
-        <origin xyz="8.625E-08 -4.6583E-06 0.03145" rpy="0 0 0" />
-        <mass value="0.22652" />
-        <inertia ixx="0.00020005" ixy="0" ixz="0" iyy="0.00017832" iyz="0" izz="0.00013478" />
-      </inertial>
-      <visual>
-        <origin xyz="0 0 0" rpy="0 0 0" />
-        <geometry>
-          <mesh filename="package://robotiq_85_gripper_description/meshes/hros_robotiq_adapter.dae" scale="0.001 0.001 0.001"/>
-        </geometry>
-        <material name="Gazebo/Black">
-          <color rgba="0.1 0.1 0.1 1" />
-        </material>
-      </visual>
-      <collision>
-        <origin xyz="0 0 0" rpy="0 0 0" />
-        <geometry>
-          <mesh filename="package://robotiq_85_gripper_description/meshes/hros_robotiq_adapter.dae" scale="0.001 0.001 0.001"/>
-        </geometry>
-      </collision>
-    </link>
-    <gazebo reference="robotiq_adapter_link">
-      <material>Gazebo/Black</material>
-      <selfCollide>True</selfCollide>
-    </gazebo>
-    <link name="robotiq_arg2f_base_link">
-      <inertial>
-        <origin xyz="8.625E-08 -4.6583E-06 0.03145" rpy="0 0 0" />
-        <mass value="0.22652" />
-        <inertia ixx="0.00020005" ixy="0" ixz="0" iyy="0.00017832" iyz="0" izz="0.00013478" />
-      </inertial>
-      <visual>
-        <origin xyz="0 0 0" rpy="0 0 1.57" />
-        <geometry>
-          <mesh filename="package://robotiq_140_gripper_description/meshes/GRIPPER_base_axis.dae" scale="0.001 0.001 0.001"/>
-        </geometry>
-        <material name="Gazebo/Black">
-          <color rgba="0.1 0.1 0.1 1" />
-        </material>
-      </visual>
-      <collision>
-        <origin xyz="0 0 0" rpy="0 0 1.57" />
-        <geometry>
-          <mesh filename="package://robotiq_140_gripper_description/meshes/GRIPPER_base_axis.dae" scale="0.001 0.001 0.001"/>
-        </geometry>
-      </collision>
-    </link>
-    <gazebo reference="robotiq_arg2f_base_link">
-      <material>Gazebo/Black</material>
-      <selfCollide>True</selfCollide>
-    </gazebo>
-    <link name="left_outer_knuckle">
-      <inertial>
-        <origin xyz="0 0 0" rpy="0 0 0" />
-        <mass value="0.00853198276973456" />
-        <inertia
-            ixx="2.89328108496468E-06"
-            ixy="0"
-            ixz="0"
-            iyy="1.86719750325683E-06"
-            iyz="-1.21858577871576E-06"
-            izz="1.21905238907251E-06" />
-      </inertial>
-      <visual>
-        <origin xyz="0 0 0" rpy="0 0 0" />
-        <geometry>
-          <mesh filename="package://robotiq_140_gripper_description/meshes/robotiq_140_left_outer_knuckle.dae" />
-        </geometry>
-        <material name="">
-          <color rgba="0.792156862745098 0.819607843137255 0.933333333333333 1" />
-        </material>
-      </visual>
-      <collision>
-        <origin xyz="0 0 0" rpy="0 0 0" />
-        <geometry>
-          <mesh filename="package://robotiq_140_gripper_description/meshes/robotiq_140_left_outer_knuckle.dae" />
-        </geometry>
-      </collision>
-    </link>
-    <gazebo reference="left_outer_knuckle">
-      <material>Gazebo/Grey</material>
-      <selfCollide>True</selfCollide>
-    </gazebo>
-    <link name="right_outer_knuckle">
-      <inertial>
-        <origin xyz="0 0 0" rpy="0 0 0" />
-        <mass value="0.00853198276973456" />
-        <inertia
-            ixx="2.89328108496468E-06"
-            ixy="0"
-            ixz="0"
-            iyy="1.86719750325683E-06"
-            iyz="-1.21858577871576E-06"
-            izz="1.21905238907251E-06" />
-      </inertial>
-      <visual>
-        <origin xyz="0 0 0" rpy="0 0 0" />
-        <geometry>
-          <mesh filename="package://robotiq_140_gripper_description/meshes/robotiq_140_right_outer_knuckle.dae" />
-        </geometry>
-        <material name="">
-          <color rgba="0.792156862745098 0.819607843137255 0.933333333333333 1" />
-        </material>
-      </visual>
-      <collision>
-        <origin xyz="0 0 0" rpy="0 0 0" />
-        <geometry>
-          <mesh filename="package://robotiq_140_gripper_description/meshes/robotiq_140_right_outer_knuckle.dae" />
-        </geometry>
-      </collision>
-    </link>
-    <gazebo reference="right_outer_knuckle">
-      <material>Gazebo/Grey</material>
-      <selfCollide>True</selfCollide>
-    </gazebo>
-    <link name="left_inner_knuckle">
-      <inertial>
-        <origin xyz="0.000123011831763771 0.0507850843201817 0.00103968640075166" rpy="0 0 0" />
-        <mass value="0.0271177346495152" />
-        <inertia
-            ixx="2.61910379223783E-05"
-            ixy="-2.43616858946494E-07"
-            ixz="-6.37789906117123E-09"
-            iyy="2.8270243746167E-06"
-            iyz="-5.37200748039765E-07"
-            izz="2.83695868220296E-05" />
-      </inertial>
-      <visual>
-        <origin xyz="0 0 0" rpy="0 0 0" />
-        <geometry>
-          <mesh filename="package://robotiq_140_gripper_description/meshes/robotiq_140_left_inner_knuckle.dae" />
-        </geometry>
-        <material name="Gazebo/Black">
-          <color rgba="0.1 0.1 0.1 1" />
-        </material>
-      </visual>
-    </link>
-    <gazebo reference="left_inner_knuckle">
-      <material>Gazebo/Black</material>
-      <selfCollide>True</selfCollide>
-    </gazebo>
-    <link name="right_inner_knuckle">
-      <inertial>
-        <origin xyz="0.000123011831763771 0.0507850843201817 0.00103968640075166" rpy="0 0 0" />
-        <mass value="0.0271177346495152" />
-        <inertia
-            ixx="2.61910379223783E-05"
-            ixy="-2.43616858946494E-07"
-            ixz="-6.37789906117123E-09"
-            iyy="2.8270243746167E-06"
-            iyz="-5.37200748039765E-07"
-            izz="2.83695868220296E-05" />
-      </inertial>
-      <visual>
-        <origin xyz="0 0 0" rpy="0 0 0" />
-        <geometry>
-          <mesh filename="package://robotiq_140_gripper_description/meshes/robotiq_140_right_inner_knuckle.dae" />
-        </geometry>
-        <material name="Gazebo/Black">
-          <color rgba="0.1 0.1 0.1 1" />
-        </material>
-      </visual>
-    </link>
-    <gazebo reference="right_inner_knuckle">
-      <material>Gazebo/Black</material>
-      <selfCollide>True</selfCollide>
-    </gazebo>
-    <link name="left_inner_finger">
-      <inertial>
-        <origin xyz="0.0 0.031506174 -0.017648840" rpy="0 0 0" />
-        <mass value="0.0104003125914103" />
-        <inertia
-            ixx="6.06863499e-06"
-            ixy="0"
-            ixz="0"
-            iyy="7.46305064e-07"
-            iyz="0"
-            izz="6.21796490e-06" />
-      </inertial>
-      <visual>
-        <origin xyz="0 0 0" rpy="0 0 0" />
-        <geometry>
-          <mesh filename="package://robotiq_140_gripper_description/meshes/robotiq_140_left_inner_finger.dae" scale="0.001 0.001 0.001" />
-        </geometry>
-        <material name="Gazebo/Black">
-          <color rgba="0.1 0.1 0.1 1" />
-        </material>
-      </visual>
-      <collision>
-        <origin xyz="0 0 0" rpy="0 0 0" />
-        <geometry>
-          <mesh filename="package://robotiq_140_gripper_description/meshes/robotiq_140_left_inner_finger.dae" scale="0.001 0.001 0.001" />
-        </geometry>
-      </collision>
-    </link>
-    <gazebo reference="left_inner_finger">
-      <material>Gazebo/Black</material>
-      <selfCollide>True</selfCollide>
-    </gazebo>
-    <link name="right_inner_finger">
-      <inertial>
-        <origin xyz="0.0 0.031506174 -0.017648840" rpy="0 0 0" />
-        <mass value="0.0104003125914103" />
-        <inertia
-            ixx="6.06863499e-06"
-            ixy="0"
-            ixz="0"
-            iyy="7.46305064e-07"
-            iyz="0"
-            izz="6.21796490e-06" />
-      </inertial>
-      <visual>
-        <origin xyz="0 0 0" rpy="0 0 0" />
-        <geometry>
-          <mesh filename="package://robotiq_140_gripper_description/meshes/robotiq_140_right_inner_finger.dae" scale="0.001 0.001 0.001"/>
-        </geometry>
-        <material name="Gazebo/Black">
-          <color rgba="0.1 0.1 0.1 1" />
-        </material>
-      </visual>
-      <collision>
-        <origin xyz="0 0 0" rpy="0 0 0" />
-        <geometry>
-          <mesh filename="package://robotiq_140_gripper_description/meshes/robotiq_140_right_inner_finger.dae" scale="0.001 0.001 0.001"/>
-        </geometry>
-      </collision>
-    </link>
-    <gazebo reference="right_inner_finger">
-      <material>Gazebo/Black</material>
-      <selfCollide>True</selfCollide>
-    </gazebo>
-    <link name="left_outer_finger">
-      <inertial>
-        <origin xyz="0.00030115855001899 0.0373907951953854 -0.0208027427000385" rpy="0 0 0" />
-        <mass value="0.022614240507152" />
-        <inertia
-            ixx="1.52518312458174E-05"
-            ixy="9.76583423954399E-10"
-            ixz="-5.43838577022588E-10"
-            iyy="6.17694243867776E-06"
-            iyz="6.78636130740228E-06"
-            izz="1.16494917907219E-05" />
-      </inertial>
-      <visual>
-        <origin xyz="0 0 0" rpy="0 0 0" />
-        <geometry>
-          <mesh filename="package://robotiq_140_gripper_description/meshes/robotiq_140_left_outer_finger.dae" />
-        </geometry>
-        <material name="Gazebo/Black">
-          <color rgba="0.1 0.1 0.1 1" />
-        </material>
-      </visual>
-      <collision>
-        <origin xyz="0 0 0" rpy="0 0 0" />
-        <geometry>
-          <mesh filename="package://robotiq_140_gripper_description/meshes/robotiq_140_left_outer_finger.dae" />
-        </geometry>
-      </collision>
-    </link>
-    <gazebo reference="left_outer_finger">
-      <material>Gazebo/Black</material>
-      <selfCollide>True</selfCollide>
-    </gazebo>
-    <link name="right_outer_finger">
-      <inertial>
-        <origin xyz="0.00030115855001899 0.0373907951953854 -0.0208027427000385" rpy="0 0 0" />
-        <mass value="0.022614240507152" />
-        <inertia
-            ixx="1.52518312458174E-05"
-            ixy="9.76583423954399E-10"
-            ixz="-5.43838577022588E-10"
-            iyy="6.17694243867776E-06"
-            iyz="6.78636130740228E-06"
-            izz="1.16494917907219E-05" />
-      </inertial>
-      <visual>
-        <origin xyz="0 0 0" rpy="0 0 0" />
-        <geometry>
-          <mesh filename="package://robotiq_140_gripper_description/meshes/robotiq_140_right_outer_finger.dae" />
-        </geometry>
-        <material name="Gazebo/Black">
-          <color rgba="0.1 0.1 0.1 1" />
-        </material>
-      </visual>
-      <collision>
-        <origin xyz="0 0 0" rpy="0 0 0" />
-        <geometry>
-          <mesh filename="package://robotiq_140_gripper_description/meshes/robotiq_140_right_outer_finger.dae" />
-        </geometry>
-      </collision>
-    </link>
-    <gazebo reference="right_outer_finger">
-      <material>Gazebo/Black</material>
-      <selfCollide>True</selfCollide>
-    </gazebo>
-    <joint name="base_adapter_to_base_robotiq_joint" type="fixed">
-      <origin rpy="0 0 0" xyz=" 0 0 0.03653"/>
-      <parent link="robotiq_adapter_link" />
-      <child link="robotiq_arg2f_base_link"/>
-    </joint>
-    <joint name="left_outer_knuckle_joint" type="revolute">
-      <origin xyz="0 -0.030601 0.054905" rpy="2.31 0 0" />
-      <parent link="robotiq_arg2f_base_link" />
-      <child link="left_outer_knuckle" />
-      <axis xyz="-1 0 0" />
-      <limit lower="0" upper="0.78"  velocity="2.0" effort="1000" />
-    </joint>
-    <joint name="right_outer_knuckle_joint" type="revolute">
-      <origin xyz="0 0.030601 0.054905" rpy="2.31 0 3.14159265359" />
-      <parent link="robotiq_arg2f_base_link" />
-      <child link="right_outer_knuckle" />
-      <axis xyz="-1 0 0" />
-      <limit lower="0" upper="0.78" velocity="2.0" effort="1000" />
-    </joint>
-    <joint name="left_inner_knuckle_joint" type="revolute">
-      <origin xyz="0 -0.0127 0.06142" rpy="2.29 0 0" />
-      <parent link="robotiq_arg2f_base_link" />
-      <child link="left_inner_knuckle" />
-      <axis xyz="-1 0 0" />
-      <limit lower="0" upper="0.78" velocity="2.0" effort="1000" />
-    </joint>
-    <joint name="right_inner_knuckle_joint" type="revolute">
-      <origin xyz="0 0.0127 0.06142" rpy="2.29 0 -3.14159265359" />
-      <parent link="robotiq_arg2f_base_link" />
-      <child link="right_inner_knuckle" />
-      <axis xyz="-1 0 0" />
-      <limit lower="0" upper="0.78" velocity="2.0" effort="1000" />
-    </joint>
-    <joint name="left_outer_finger_joint" type="revolute">
-      <origin xyz="0 0.01821998610742 0.0260018192872234" rpy="0 0 0" />
-      <parent link="left_outer_knuckle" />
-      <child link="left_outer_finger" />
-      <axis xyz="-1 0 0" />
-      <limit lower="-0.875" upper="-0.0075" velocity="2.0" effort="1000" />
-    </joint>
-    <joint name="right_outer_finger_joint" type="revolute">
-      <origin xyz="0 0.01821998610742 0.0260018192872234" rpy="0 0 0" />
-      <parent link="right_outer_knuckle" />
-      <child link="right_outer_finger" />
-      <axis xyz="-1 0 0" />
-      <limit lower="-0.875" upper="-0.0075" velocity="2.0" effort="1000" />
-    </joint>
-    <joint name="left_inner_finger_joint" type="revolute">
-      <origin xyz="0 0.0817554015893473 -0.0282203446692936" rpy="-.725 0 0" />
-      <parent link="left_outer_finger" />
-      <child link="left_inner_finger" />
-      <axis xyz="1 0 0" />
-      <limit lower="-0.875" upper="0.8757" velocity="2.0" effort="1000" />
-    </joint>
-    <joint name="right_inner_finger_joint" type="revolute">
-      <origin xyz="0 0.0817554015893473 -0.0282203446692936" rpy="-.725 0 0" />
-      <parent link="right_outer_finger" />
-      <child link="right_inner_finger" />
-      <axis xyz="1 0 0" />
-      <limit lower="-0.875" upper="0.8757" velocity="2.0" effort="1000" />
-    </joint>
-    <gazebo>
-      <joint name="left_inner_finger_knuckle_joint" type="revolute">
-        <pose frame="">0 0.006 -0.018 0 0 0</pose>
-        <parent>${prefix}::left_inner_knuckle</parent>
-        <child>${prefix}::left_inner_finger</child>
-        <axis>
-          <xyz>1 0 0</xyz>
-          <limit>
-            <lower>-0.8</lower>
-            <upper>0.8</upper>
-            <velocity>2.0</velocity>
-            <effort>1000</effort>
-          </limit>
-        </axis>
-      </joint>
-      <joint name="right_inner_finger_knuckle_joint" type="revolute">
-        <pose frame="">0 0.006 -0.018 0 0 0</pose>
-        <parent>${prefix}::right_inner_knuckle</parent>
-        <child>${prefix}::right_inner_finger</child>
-        <axis>
-          <xyz>-1 0 0</xyz>
-          <limit>
-            <lower>-0.8</lower>
-            <upper>0.8</upper>
-            <velocity>2.0</velocity>
-            <effort>1000</effort>
-          </limit>
-        </axis>
-      </joint>
-      <plugin filename="librobotiq_gripper_gazebo_plugin.so" name="hros_actuation_gripper_000000000004">
-        <left_joint>left_inner_knuckle_joint</left_joint>
-        <left_joint>left_outer_knuckle_joint</left_joint>
-        <right_joint>right_inner_knuckle_joint</right_joint>
-        <right_joint>right_outer_knuckle_joint</right_joint>
-      </plugin>
-    </gazebo>
-  </xacro:macro>
+<robot xmlns:xacro="http://ros.org/wiki/xacro"
+       name="robotiq_gripper" >
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