Commit message: update S140 dae files

File: robotiq_140_gripper_description/urdf/robotiq_140.urdf (robot description, URDF)
Before this commit: robot robotiq_gripper, 11 links, 10 joints
Links:
- removed link robotiq_adapter_link
- link left_inner_knuckle: geometry visual mesh filename=package://robotiq_140_gripper_description/meshes/robotiq_14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 scale=0.001 0.001 0.001
- link left_outer_finger: geometry collision mesh filename=package://robotiq_140_gripper_description/meshes/robotiq_14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 scale=0.001 0.001 0.001; visual mesh filename=package://robotiq_140_gripper_description/meshes/robotiq_14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 scale=0.001 0.001 0.001
- link left_outer_knuckle: geometry collision mesh filename=package://robotiq_140_gripper_description/meshes/robotiq_14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 scale=0.001 0.001 0.001; visual mesh filename=package://robotiq_140_gripper_description/meshes/robotiq_14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 scale=0.001 0.001 0.001
- link right_inner_knuckle: geometry visual mesh filename=package://robotiq_140_gripper_description/meshes/robotiq_14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 scale=0.001 0.001 0.001
- link right_outer_finger: geometry collision mesh filename=package://robotiq_140_gripper_description/meshes/robotiq_14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 scale=0.001 0.001 0.001; visual mesh filename=package://robotiq_140_gripper_description/meshes/robotiq_14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 scale=0.001 0.001 0.001
- link right_outer_knuckle: geometry collision mesh filename=package://robotiq_140_gripper_description/meshes/robotiq_14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 scale=0.001 0.001 0.001; visual mesh filename=package://robotiq_140_gripper_description/meshes/robotiq_14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 scale=0.001 0.001 0.001
Joints:
- removed joint base_adapter_to_base_robotiq_joint
- removed joint left_inner_finger_joint
- removed joint left_inner_knuckle_joint
- removed joint left_outer_finger_joint
- removed joint left_outer_knuckle_joint
- removed joint right_inner_finger_joint
- removed joint right_inner_knuckle_joint
- removed joint right_outer_finger_joint
- removed joint world_to_hande_joint
- added joint left_outer_finger_to_inner: type revolute, parent left_outer_finger, child left_inner_finger, origin xyz=0.03543 0 0.0789 rpy=0 0 0, axis 0 -1 0, limit lower=0 upper=0.78574722925 effort=1000 velocity=2.0, mimic joint=joint_finger multiplier=1 offset=0
- added joint left_outer_knuckle_to_finger: type fixed, parent left_outer_knuckle, child left_outer_finger, origin xyz=0.03142 0 -0.00453 rpy=0 0 0
- added joint right_outer_finger_to_inner: type revolute, parent right_outer_finger, child right_inner_finger, origin xyz=-0.03543 0 0.0789 rpy=0 0 0, axis 0 1 0, limit lower=0 upper=0.78574722925 effort=1000 velocity=2.0, mimic joint=joint_finger multiplier=1 offset=0
- added joint right_outer_knuckle_to_finger: type fixed, parent right_outer_knuckle, child right_outer_finger, origin xyz=-0.03142 0 -0.00453 rpy=0 0 0
- added joint robotiq_arg2f_base_to_left_inner_knuckle: type revolute, parent robotiq_arg2f_base_link, child left_inner_knuckle, origin xyz=0.0127 0 0.06118 rpy=0 0 0, axis 0 -1 0, limit lower=0 upper=0.78574722925 effort=1000 velocity=2.0, mimic joint=joint_finger multiplier=1 offset=0
- added joint robotiq_arg2f_base_to_left_outer_knuckle: type revolute, parent robotiq_arg2f_base_link, child left_outer_knuckle, origin xyz=0.0306 0 0.05466 rpy=0 0 0, axis 0 -1 0, limit lower=0 upper=0.78574722925 effort=1000 velocity=2.0, mimic joint=joint_finger multiplier=1 offset=0
- added joint robotiq_arg2f_base_to_right_inner_knuckle: type revolute, parent robotiq_arg2f_base_link, child right_inner_knuckle, origin xyz=-0.0127 0 0.06118 rpy=0 0 0, axis 0 1 0, limit lower=0 upper=0.78574722925 effort=1000 velocity=2.0, mimic joint=joint_finger multiplier=1 offset=0
- added joint world_to_robotiq_adapter: type fixed, parent world, child robotiq_arg2f_base_link, origin xyz=0 0 0.5 rpy=0 0 0
- joint joint_finger: axis -1 0 0 -> 0 1 0; limit lower=0 upper=0.775 effort=1000 velocity=2.0 -> lower=0 upper=0.78574722925 effort=1000 velocity=2.0; origin xyz=0 0.030601 0.054905 rpy=2.31 0 3.14159265359 -> xyz=-0.0306 0 0.05466 rpy=0 0 0

File: robotiq_140_gripper_description/urdf/robotiq_140.urdf.xacro (robot description, xacro)
@@ -2,5 +2,5 @@
 <robot xmlns:xacro="http://ros.org/wiki/xacro">
   <xacro:macro name="robotiq_gripper"  params="prefix">
-    <link name="robotiq_adapter_link">
+    <link name="robotiq_arg2f_base_link">
       <inertial>
         <origin xyz="8.625E-08 -4.6583E-06 0.03145" rpy="0 0 0" />
@@ -9,36 +9,5 @@
       </inertial>
       <visual>
-        <origin xyz="0 0 0" rpy="0 0 1.57" />
-        <geometry>
-          <mesh filename="package://robotiq_140_gripper_description/meshes/hros_robotiq_adapter.dae" scale="0.001 0.001 0.001"/>
-        </geometry>
-        <material name="Gazebo/Black">
-          <color rgba="0.0 0.0 0.0 1" />
-        </material>
-      </visual>
-      <collision>
-        <origin xyz="0 0 0" rpy="0 0 1.57" />
-        <geometry>
-          <mesh filename="package://robotiq_140_gripper_description/meshes/hros_robotiq_adapter.dae" scale="0.001 0.001 0.001"/>
-        </geometry>
-      </collision>
-    </link>
-    <gazebo reference="robotiq_adapter_link">
-      <material>Gazebo/Black</material>
-      <selfCollide>False</selfCollide>
-    </gazebo>
-    <joint name="base_adapter_to_base_robotiq_joint" type="fixed">
-      <origin rpy="0 0 0" xyz=" 0 0 0.03653"/>
-      <parent link="robotiq_adapter_link" />
-      <child link="robotiq_arg2f_base_link"/>
-    </joint>
-    <link name="robotiq_arg2f_base_link">
-      <inertial>
-        <origin xyz="8.625E-08 -4.6583E-06 0.03145" rpy="0 0 0" />
-        <mass value="0.22652" />
-        <inertia ixx="0.00020005" ixy="0" ixz="0" iyy="0.00017832" iyz="0" izz="0.00013478" />
-      </inertial>
-      <visual>
-        <origin xyz="0 0 0" rpy="0 0 1.57" />
+        <origin xyz="0 0 0" rpy="0 0 0" />
         <geometry>
           <mesh filename="package://robotiq_140_gripper_description/meshes/GRIPPER_base_axis.dae" scale="0.001 0.001 0.001"/>
@@ -49,5 +18,5 @@
       </visual>
       <collision>
-        <origin xyz="0 0 0" rpy="0 0 1.57" />
+        <origin xyz="0 0 0" rpy="0 0 0" />
         <geometry>
           <mesh filename="package://robotiq_140_gripper_description/meshes/GRIPPER_base_axis.dae" scale="0.001 0.001 0.001"/>
@@ -74,5 +43,5 @@
         <origin xyz="0 0 0" rpy="0 0 0" />
         <geometry>
-          <mesh filename="package://robotiq_140_gripper_description/meshes/robotiq_140_left_outer_knuckle.dae" />
+          <mesh filename="package://robotiq_140_gripper_description/meshes/robotiq_140_left_outer_knuckle.dae" scale="0.001 0.001 0.001"/>
         </geometry>
         <material name="">
@@ -83,5 +52,5 @@
         <origin xyz="0 0 0" rpy="0 0 0" />
         <geometry>
-          <mesh filename="package://robotiq_140_gripper_description/meshes/robotiq_140_left_outer_knuckle.dae" />
+          <mesh filename="package://robotiq_140_gripper_description/meshes/robotiq_140_left_outer_knuckle.dae" scale="0.001 0.001 0.001"/>
         </geometry>
       </collision>
@@ -106,5 +75,5 @@
         <origin xyz="0 0 0" rpy="0 0 0" />
         <geometry>
-          <mesh filename="package://robotiq_140_gripper_description/meshes/robotiq_140_right_outer_knuckle.dae" />
+          <mesh filename="package://robotiq_140_gripper_description/meshes/robotiq_140_right_outer_knuckle.dae" scale="0.001 0.001 0.001"/>
         </geometry>
         <material name="">
@@ -115,5 +84,5 @@
         <origin xyz="0 0 0" rpy="0 0 0" />
         <geometry>
-          <mesh filename="package://robotiq_140_gripper_description/meshes/robotiq_140_right_outer_knuckle.dae" />
+          <mesh filename="package://robotiq_140_gripper_description/meshes/robotiq_140_right_outer_knuckle.dae" scale="0.001 0.001 0.001"/>
         </geometry>
       </collision>
@@ -138,5 +107,5 @@
         <origin xyz="0 0 0" rpy="0 0 0" />
         <geometry>
-          <mesh filename="package://robotiq_140_gripper_description/meshes/robotiq_140_left_inner_knuckle.dae" />
+          <mesh filename="package://robotiq_140_gripper_description/meshes/robotiq_140_left_inner_knuckle.dae" scale="0.001 0.001 0.001"/>
         </geometry>
         <material name="Gazebo/Black">
@@ -164,5 +133,5 @@
         <origin xyz="0 0 0" rpy="0 0 0" />
         <geometry>
-          <mesh filename="package://robotiq_140_gripper_description/meshes/robotiq_140_right_inner_knuckle.dae" />
+          <mesh filename="package://robotiq_140_gripper_description/meshes/robotiq_140_right_inner_knuckle.dae" scale="0.001 0.001 0.001"/>
         </geometry>
         <material name="Gazebo/Black">
@@ -254,14 +223,14 @@
         <origin xyz="0 0 0" rpy="0 0 0" />
         <geometry>
-          <mesh filename="package://robotiq_140_gripper_description/meshes/robotiq_140_left_outer_finger.dae" />
-        </geometry>
-        <material name="Gazebo/Black">
-          <color rgba="0.1 0.1 0.1 1" />
-        </material>
-      </visual>
-      <collision>
-        <origin xyz="0 0 0" rpy="0 0 0" />
-        <geometry>
-          <mesh filename="package://robotiq_140_gripper_description/meshes/robotiq_140_left_outer_finger.dae" />
+          <mesh filename="package://robotiq_140_gripper_description/meshes/robotiq_140_left_outer_finger.dae" scale="0.001 0.001 0.001"/>
+        </geometry>
+        <material name="Gazebo/Black">
+          <color rgba="0.1 0.1 0.1 1" />
+        </material>
+      </visual>
+      <collision>
+        <origin xyz="0 0 0" rpy="0 0 0" />
+        <geometry>
+          <mesh filename="package://robotiq_140_gripper_description/meshes/robotiq_140_left_outer_finger.dae" scale="0.001 0.001 0.001"/>
         </geometry>
       </collision>
@@ -286,14 +255,14 @@
         <origin xyz="0 0 0" rpy="0 0 0" />
         <geometry>
-          <mesh filename="package://robotiq_140_gripper_description/meshes/robotiq_140_right_outer_finger.dae" />
-        </geometry>
-        <material name="Gazebo/Black">
-          <color rgba="0.1 0.1 0.1 1" />
-        </material>
-      </visual>
-      <collision>
-        <origin xyz="0 0 0" rpy="0 0 0" />
-        <geometry>
-          <mesh filename="package://robotiq_140_gripper_description/meshes/robotiq_140_right_outer_finger.dae" />
+          <mesh filename="package://robotiq_140_gripper_description/meshes/robotiq_140_right_outer_finger.dae" scale="0.001 0.001 0.001"/>
+        </geometry>
+        <material name="Gazebo/Black">
+          <color rgba="0.1 0.1 0.1 1" />
+        </material>
+      </visual>
+      <collision>
+        <origin xyz="0 0 0" rpy="0 0 0" />
+        <geometry>
+          <mesh filename="package://robotiq_140_gripper_description/meshes/robotiq_140_right_outer_finger.dae" scale="0.001 0.001 0.001"/>
         </geometry>
       </collision>
@@ -303,71 +272,71 @@
       <selfCollide>False</selfCollide>
     </gazebo>
-    <joint name="left_outer_knuckle_joint" type="revolute">
-      <origin xyz="0 -0.030601 0.054905" rpy="2.31 0 0" />
+    <joint name="robotiq_arg2f_base_to_left_outer_knuckle" type="revolute">
+      <origin xyz="0.0306 0 0.05466" rpy="0 0 0" />
       <parent link="robotiq_arg2f_base_link" />
       <child link="left_outer_knuckle" />
-      <axis xyz="-1 0 0" />
-      <limit lower="0" upper="0.775"  velocity="2.0" effort="1000" />
+      <axis xyz="0 -1 0" />
+      <limit lower="0" upper="0.78574722925"  velocity="2.0" effort="1000" />
       <mimic joint="joint_finger" multiplier="1" offset="0"/>
     </joint>
     <joint name="joint_finger" type="revolute">
-      <origin xyz="0 0.030601 0.054905" rpy="2.31 0 3.14159265359" />
+      <origin xyz="-0.0306 0 0.05466" rpy="0 0 0" />
       <parent link="robotiq_arg2f_base_link" />
       <child link="right_outer_knuckle" />
-      <axis xyz="-1 0 0" />
-      <limit lower="0" upper="0.775" velocity="2.0" effort="1000" />
-    </joint>
-    <joint name="left_inner_knuckle_joint" type="revolute">
-      <origin xyz="0 -0.0127 0.06142" rpy="2.29 0 0" />
+      <axis xyz="0 1 0" />
+      <limit lower="0" upper="0.78574722925" velocity="2.0" effort="1000" />
+    </joint>
+    <joint name="robotiq_arg2f_base_to_left_inner_knuckle" type="revolute">
+      <origin xyz="0.0127 0 0.06118" rpy="0 0 0" />
       <parent link="robotiq_arg2f_base_link" />
       <child link="left_inner_knuckle" />
-      <axis xyz="-1 0 0" />
-      <limit lower="0" upper="0.78" velocity="2.0" effort="1000" />
-      <mimic joint="joint_finger" multiplier="1" offset="0"/>
-    </joint>
-    <joint name="right_inner_knuckle_joint" type="revolute">
-      <origin xyz="0 0.0127 0.06142" rpy="2.29 0 -3.14159265359" />
+      <axis xyz="0 -1 0" />
+      <limit lower="0" upper="0.78574722925" velocity="2.0" effort="1000" />
+      <mimic joint="joint_finger" multiplier="1" offset="0"/>
+    </joint>
+    <joint name="robotiq_arg2f_base_to_right_inner_knuckle" type="revolute">
+      <origin xyz="-0.0127 0 0.06118" rpy="0 0 0" />
       <parent link="robotiq_arg2f_base_link" />
       <child link="right_inner_knuckle" />
-      <axis xyz="-1 0 0" />
-      <limit lower="0" upper="0.78" velocity="2.0" effort="1000" />
-      <mimic joint="joint_finger" multiplier="1" offset="0"/>
-    </joint>
-    <joint name="left_outer_finger_joint" type="fixed">
-      <origin xyz="0 0.01821998610742 0.0260018192872234" rpy="0 0 0" />
+      <axis xyz="0 1 0" />
+      <limit lower="0" upper="0.78574722925" velocity="2.0" effort="1000" />
+      <mimic joint="joint_finger" multiplier="1" offset="0"/>
+    </joint>
+    <joint name="left_outer_knuckle_to_finger" type="fixed">
+      <origin xyz="0.03142 0 -0.00453" rpy="0 0 0" />
       <parent link="left_outer_knuckle" />
       <child link="left_outer_finger" />
     </joint>
-    <joint name="right_outer_finger_joint" type="fixed">
-      <origin xyz="0 0.01821998610742 0.0260018192872234" rpy="0 0 0" />
+    <joint name="right_outer_knuckle_to_finger" type="fixed">
+      <origin xyz="-0.03142 0 -0.00453" rpy="0 0 0" />
       <parent link="right_outer_knuckle" />
       <child link="right_outer_finger" />
     </joint>
-    <joint name="left_inner_finger_joint" type="revolute">
-      <origin xyz="0 0.0817554015893473 -0.0282203446692936" rpy="-.725 0 0" />
+    <joint name="left_outer_finger_to_inner" type="revolute">
+      <origin xyz="0.03543 0 0.0789" rpy="0 0 0" />
       <parent link="left_outer_finger" />
       <child link="left_inner_finger" />
-      <axis xyz="1 0 0" />
-      <limit lower="0" upper="0.8757" velocity="2.0" effort="1000" />
-      <mimic joint="joint_finger" multiplier="1" offset="0"/>
-    </joint>
-    <joint name="right_inner_finger_joint" type="revolute">
-      <origin xyz="0 0.0817554015893473 -0.0282203446692936" rpy="-.725 0 0" />
+      <axis xyz="0 -1 0" />
+      <limit lower="0" upper="0.78574722925" velocity="2.0" effort="1000" />
+      <mimic joint="joint_finger" multiplier="1" offset="0"/>
+    </joint>
+    <joint name="right_outer_finger_to_inner" type="revolute">
+      <origin xyz="-0.03543 0 0.0789" rpy="0 0 0" />
       <parent link="right_outer_finger" />
       <child link="right_inner_finger" />
-      <axis xyz="1 0 0" />
-      <limit lower="0" upper="0.8757" velocity="2.0" effort="1000" />
+      <axis xyz="0 1 0" />
+      <limit lower="0" upper="0.78574722925" velocity="2.0" effort="1000" />
       <mimic joint="joint_finger" multiplier="1" offset="0"/>
     </joint>
     <gazebo>
-      <joint name="left_inner_finger_knuckle_joint" type="revolute">
-        <pose frame="">0 0.006 -0.018 0 0 0</pose>
+      <joint name="left_inner_knuckle_to_finger" type="revolute">
+        <pose frame="">0.06686 0 0.07436 0 0 0</pose>
         <parent>${prefix}::left_inner_knuckle</parent>
         <child>${prefix}::left_inner_finger</child>
         <axis>
-          <xyz>1 0 0</xyz>
+          <xyz>0 -1 0</xyz>
           <limit>
-            <lower>-0.8</lower>
-            <upper>0.8</upper>
+            <lower>0</lower>
+            <upper>0.78574722925</upper>
             <velocity>2.0</velocity>
             <effort>1000</effort>
@@ -375,13 +344,13 @@
         </axis>
       </joint>
-      <joint name="right_inner_finger_knuckle_joint" type="revolute">
-        <pose frame="">0 0.006 -0.018 0 0 0</pose>
+      <joint name="right_inner_knuckle_to_finger" type="revolute">
+        <pose frame="">-0.06686 0 0.07436 0 0 0</pose>
         <parent>${prefix}::right_inner_knuckle</parent>
         <child>${prefix}::right_inner_finger</child>
         <axis>
-          <xyz>-1 0 0</xyz>
+          <xyz>0 1 0</xyz>
           <limit>
-            <lower>-0.8</lower>
-            <upper>0.8</upper>
+            <lower>0</lower>
+            <upper>0.78574722925</upper>
             <velocity>2.0</velocity>
             <effort>1000</effort>
@@ -390,7 +359,7 @@
       </joint>
       <plugin filename="librobotiq_gripper_gazebo_plugin.so" name="hrim_actuation_gripper_000000000004">
-        <joint>left_inner_knuckle_joint</joint>
-        <joint>left_outer_knuckle_joint</joint>
-        <joint>right_inner_knuckle_joint</joint>
+        <joint>robotiq_arg2f_base_to_left_inner_knuckle</joint>
+        <joint>robotiq_arg2f_base_to_left_outer_knuckle</joint>
+        <joint>robotiq_arg2f_base_to_right_inner_knuckle</joint>
         <joint>joint_finger</joint>
       </plugin>

Commit message: fix joints and axes

File: robotiq_140_gripper_description/urdf/robotiq_140.urdf (robot description, URDF)
Before this commit: robot robotiq_gripper, 10 links, 9 joints
Joints:
- joint left_outer_finger_to_inner: axis 0 -1 0 -> 0 1 0
- joint right_outer_finger_to_inner: axis 0 1 0 -> 0 -1 0

File: robotiq_140_gripper_description/urdf/robotiq_140.urdf.xacro (robot description, xacro)
@@ -317,5 +317,5 @@
       <parent link="left_outer_finger" />
       <child link="left_inner_finger" />
-      <axis xyz="0 -1 0" />
+      <axis xyz="0 1 0" />
       <limit lower="0" upper="0.78574722925" velocity="2.0" effort="1000" />
       <mimic joint="joint_finger" multiplier="1" offset="0"/>
@@ -325,5 +325,5 @@
       <parent link="right_outer_finger" />
       <child link="right_inner_finger" />
-      <axis xyz="0 1 0" />
+      <axis xyz="0 -1 0" />
       <limit lower="0" upper="0.78574722925" velocity="2.0" effort="1000" />
       <mimic joint="joint_finger" multiplier="1" offset="0"/>
@@ -331,9 +331,9 @@
     <gazebo>
       <joint name="left_inner_knuckle_to_finger" type="revolute">
-        <pose frame="">0.06686 0 0.07436 0 0 0</pose>
+        <pose frame="">-0.0179 0 0.00652 0 0 0</pose>
         <parent>${prefix}::left_inner_knuckle</parent>
         <child>${prefix}::left_inner_finger</child>
         <axis>
-          <xyz>0 -1 0</xyz>
+          <xyz>0 1 0</xyz>
           <limit>
             <lower>0</lower>
@@ -345,9 +345,9 @@
       </joint>
       <joint name="right_inner_knuckle_to_finger" type="revolute">
-        <pose frame="">-0.06686 0 0.07436 0 0 0</pose>
+        <pose frame="">0.0179 0 0.00652 0 0 0</pose>
         <parent>${prefix}::right_inner_knuckle</parent>
         <child>${prefix}::right_inner_finger</child>
         <axis>
-          <xyz>0 1 0</xyz>
+          <xyz>0 -1 0</xyz>
           <limit>
             <lower>0</lower>

Commit message: make vel and effort of S140 same to real

File: robotiq_140_gripper_description/urdf/robotiq_140.urdf (robot description, URDF)
Before this commit: robot robotiq_gripper, 10 links, 9 joints
Joints:
- joint joint_finger: limit lower=0 upper=0.78574722925 effort=1000 velocity=2.0 -> lower=0 upper=0.78574722925 effort=18.65 velocity=3.54
- joint left_outer_finger_to_inner: limit lower=0 upper=0.78574722925 effort=1000 velocity=2.0 -> lower=0 upper=0.78574722925 effort=18.65 velocity=3.54
- joint right_outer_finger_to_inner: limit lower=0 upper=0.78574722925 effort=1000 velocity=2.0 -> lower=0 upper=0.78574722925 effort=18.65 velocity=3.54
- joint robotiq_arg2f_base_to_left_inner_knuckle: limit lower=0 upper=0.78574722925 effort=1000 velocity=2.0 -> lower=0 upper=0.78574722925 effort=18.65 velocity=3.54
- joint robotiq_arg2f_base_to_left_outer_knuckle: limit lower=0 upper=0.78574722925 effort=1000 velocity=2.0 -> lower=0 upper=0.78574722925 effort=18.65 velocity=2.0
- joint robotiq_arg2f_base_to_right_inner_knuckle: limit lower=0 upper=0.78574722925 effort=1000 velocity=2.0 -> lower=0 upper=0.78574722925 effort=18.65 velocity=3.54

File: robotiq_140_gripper_description/urdf/robotiq_140.urdf.xacro (robot description, xacro)
@@ -277,5 +277,5 @@
       <child link="left_outer_knuckle" />
       <axis xyz="0 -1 0" />
-      <limit lower="0" upper="0.78574722925"  velocity="2.0" effort="1000" />
+      <limit lower="0" upper="0.78574722925"  velocity="2.0" effort="18.65" />
       <mimic joint="joint_finger" multiplier="1" offset="0"/>
     </joint>
@@ -285,5 +285,5 @@
       <child link="right_outer_knuckle" />
       <axis xyz="0 1 0" />
-      <limit lower="0" upper="0.78574722925" velocity="2.0" effort="1000" />
+      <limit lower="0" upper="0.78574722925" velocity="3.54" effort="18.65" />
     </joint>
     <joint name="robotiq_arg2f_base_to_left_inner_knuckle" type="revolute">
@@ -292,5 +292,5 @@
       <child link="left_inner_knuckle" />
       <axis xyz="0 -1 0" />
-      <limit lower="0" upper="0.78574722925" velocity="2.0" effort="1000" />
+      <limit lower="0" upper="0.78574722925" velocity="3.54" effort="18.65" />
       <mimic joint="joint_finger" multiplier="1" offset="0"/>
     </joint>
@@ -300,5 +300,5 @@
       <child link="right_inner_knuckle" />
       <axis xyz="0 1 0" />
-      <limit lower="0" upper="0.78574722925" velocity="2.0" effort="1000" />
+      <limit lower="0" upper="0.78574722925" velocity="3.54" effort="18.65" />
       <mimic joint="joint_finger" multiplier="1" offset="0"/>
     </joint>
@@ -318,5 +318,5 @@
       <child link="left_inner_finger" />
       <axis xyz="0 1 0" />
-      <limit lower="0" upper="0.78574722925" velocity="2.0" effort="1000" />
+      <limit lower="0" upper="0.78574722925" velocity="3.54" effort="18.65" />
       <mimic joint="joint_finger" multiplier="1" offset="0"/>
     </joint>
@@ -326,5 +326,5 @@
       <child link="right_inner_finger" />
       <axis xyz="0 -1 0" />
-      <limit lower="0" upper="0.78574722925" velocity="2.0" effort="1000" />
+      <limit lower="0" upper="0.78574722925" velocity="3.54" effort="18.65" />
       <mimic joint="joint_finger" multiplier="1" offset="0"/>
     </joint>
@@ -339,6 +339,6 @@
             <lower>0</lower>
             <upper>0.78574722925</upper>
-            <velocity>2.0</velocity>
-            <effort>1000</effort>
+            <velocity>3.54</velocity>
+            <effort>18.65</effort>
           </limit>
         </axis>
@@ -353,6 +353,6 @@
             <lower>0</lower>
             <upper>0.78574722925</upper>
-            <velocity>2.0</velocity>
-            <effort>1000</effort>
+            <velocity>3.54</velocity>
+            <effort>18.65</effort>
           </limit>
         </axis>
