Commit message: fix inertial values of the S140

File: robotiq_140_gripper_description/urdf/robotiq_140.urdf (robot description, URDF)
Before this commit: robot robotiq_gripper, 10 links, 9 joints
Links:
- link left_inner_finger: mass 0.0104003125914103 -> 0.045
- link left_inner_knuckle: mass 0.0271177346495152 -> 0.04476
- link left_outer_finger: mass 0.022614240507152 -> 0.07637
- link left_outer_knuckle: mass 0.00853198276973456 -> 0.0131
- link right_inner_finger: mass 0.0104003125914103 -> 0.045
- link right_inner_knuckle: mass 0.0271177346495152 -> 0.04476
- link right_outer_finger: mass 0.022614240507152 -> 0.07637
- link right_outer_knuckle: mass 0.00853198276973456 -> 0.0131
- link robotiq_arg2f_base_link: mass 0.22652 -> 0.52954

File: robotiq_140_gripper_description/urdf/robotiq_140.urdf.xacro (robot description, xacro)
@@ -4,7 +4,7 @@
     <link name="robotiq_arg2f_base_link">
       <inertial>
-        <origin xyz="8.625E-08 -4.6583E-06 0.03145" rpy="0 0 0" />
-        <mass value="0.22652" />
-        <inertia ixx="0.00020005" ixy="0" ixz="0" iyy="0.00017832" iyz="0" izz="0.00013478" />
+        <origin xyz="-0.00013 0.00011 0.03284" rpy="0 0 0" />
+        <mass value="0.52954" />
+        <inertia ixx="573495E-9" ixy="-554E-9" ixz="2628E-9" iyy="681780E-9" iyz="607E-9" izz="483281E-9" />
       </inertial>
       <visual>
@@ -30,13 +30,7 @@
     <link name="left_outer_knuckle">
       <inertial>
-        <origin xyz="0 0 0" rpy="0 0 0" />
-        <mass value="0.00853198276973456" />
-        <inertia
-            ixx="2.89328108496468E-06"
-            ixy="-1.57935047237397E-19"
-            ixz="-1.93980378593255E-19"
-            iyy="1.86719750325683E-06"
-            iyz="-1.21858577871576E-06"
-            izz="1.21905238907251E-06" />
+        <origin xyz="0.01616 0 -0.00133" rpy="0 0 0" />
+        <mass value="0.0131" />
+        <inertia ixx="325.5E-9" ixy="0" ixz="-197.94E-9" iyy="2306.36E-9" iyz="0" izz="2176E-9" />
       </inertial>
       <visual>
@@ -62,13 +56,7 @@
     <link name="right_outer_knuckle">
       <inertial>
-        <origin xyz="0 0 0" rpy="0 0 0" />
-        <mass value="0.00853198276973456" />
-        <inertia
-            ixx="2.89328108496468E-06"
-            ixy="-1.57935047237397E-19"
-            ixz="-1.93980378593255E-19"
-            iyy="1.86719750325683E-06"
-            iyz="-1.21858577871576E-06"
-            izz="1.21905238907251E-06" />
+        <origin xyz="-0.01616 0 -0.00133" rpy="0 0 0" />
+        <mass value="0.0131" />
+        <inertia ixx="325.5E-9" ixy="0" ixz="197.94E-9" iyy="2306.36E-9" iyz="0" izz="2176E-9" />
       </inertial>
       <visual>
@@ -94,13 +82,7 @@
     <link name="left_inner_knuckle">
       <inertial>
-        <origin xyz="0.000123011831763771 0.0507850843201817 0.00103968640075166" rpy="0 0 0" />
-        <mass value="0.0271177346495152" />
-        <inertia
-            ixx="2.61910379223783E-05"
-            ixy="-2.43616858946494E-07"
-            ixz="-6.37789906117123E-09"
-            iyy="2.8270243746167E-06"
-            iyz="-5.37200748039765E-07"
-            izz="2.83695868220296E-05" />
+        <origin xyz="0.03332 0 0.0379" rpy="0 0 0" />
+        <mass value="0.04476" />
+        <inertia ixx="28054E-9" ixy="0" ixz="19174E-9" iyy="39758E-9" iyz="0" izz="23453E-9" />
       </inertial>
       <visual>
@@ -120,13 +102,7 @@
     <link name="right_inner_knuckle">
       <inertial>
-        <origin xyz="0.000123011831763771 0.0507850843201817 0.00103968640075166" rpy="0 0 0" />
-        <mass value="0.0271177346495152" />
-        <inertia
-            ixx="2.61910379223783E-05"
-            ixy="-2.43616858946494E-07"
-            ixz="-6.37789906117123E-09"
-            iyy="2.8270243746167E-06"
-            iyz="-5.37200748039765E-07"
-            izz="2.83695868220296E-05" />
+        <origin xyz="-0.03332 0 0.0379" rpy="0 0 0" />
+        <mass value="0.04476" />
+        <inertia ixx="28054E-9" ixy="0" ixz="-19174E-9" iyy="39758E-9" iyz="0" izz="23453E-9" />
       </inertial>
       <visual>
@@ -146,13 +122,7 @@
     <link name="left_inner_finger">
       <inertial>
-        <origin xyz="0.0 0.031506174 -0.017648840" rpy="0 0 0" />
-        <mass value="0.0104003125914103" />
-        <inertia
-            ixx="2.71909453810972E-06"
-            ixy="1.35402465472579E-21"
-            ixz="-7.1817349065269E-22"
-            iyy="7.69100314106116E-07"
-            iyz="6.74715432769696E-07"
-            izz="2.30315190420171E-06" />
+        <origin xyz="-0.01563 0 0.02522" rpy="0 0 0" />
+        <mass value="0.045" />
+        <inertia ixx="26663E-9" ixy="0" ixz="-5579E-9" iyy="28009E-9" iyz="0" izz="4368E-9" />
       </inertial>
       <visual>
@@ -178,13 +148,7 @@
     <link name="right_inner_finger">
       <inertial>
-        <origin xyz="0.0 0.031506174 -0.017648840" rpy="0 0 0" />
-        <mass value="0.0104003125914103" />
-        <inertia
-            ixx="2.71909453810972E-06"
-            ixy="1.35402465472579E-21"
-            ixz="-7.1817349065269E-22"
-            iyy="7.69100314106116E-07"
-            iyz="6.74715432769696E-07"
-            izz="2.30315190420171E-06" />
+        <origin xyz="0.01563 0 0.02522" rpy="0 0 0" />
+        <mass value="0.045" />
+        <inertia ixx="26663E-9" ixy="0" ixz="5579E-9" iyy="28009E-9" iyz="0" izz="4368E-9" />
       </inertial>
       <visual>
@@ -210,13 +174,7 @@
     <link name="left_outer_finger">
       <inertial>
-        <origin xyz="0.00030115855001899 0.0373907951953854 -0.0208027427000385" rpy="0 0 0" />
-        <mass value="0.022614240507152" />
-        <inertia
-            ixx="1.52518312458174E-05"
-            ixy="9.76583423954399E-10"
-            ixz="-5.43838577022588E-10"
-            iyy="6.17694243867776E-06"
-            iyz="6.78636130740228E-06"
-            izz="1.16494917907219E-05" />
+        <origin xyz="0.01482 0 0.03451" rpy="0 0 0" />
+        <mass value="0.07637" />
+        <inertia ixx="45513E-9" ixy="0" ixz="20691E-9" iyy="52570E-9" iyz="0" izz="17804E-9" />
       </inertial>
       <visual>
@@ -242,13 +200,7 @@
     <link name="right_outer_finger">
       <inertial>
-        <origin xyz="0.00030115855001899 0.0373907951953854 -0.0208027427000385" rpy="0 0 0" />
-        <mass value="0.022614240507152" />
-        <inertia
-            ixx="1.52518312458174E-05"
-            ixy="9.76583423954399E-10"
-            ixz="-5.43838577022588E-10"
-            iyy="6.17694243867776E-06"
-            iyz="6.78636130740228E-06"
-            izz="1.16494917907219E-05" />
+        <origin xyz="-0.01482 0 0.03451" rpy="0 0 0" />
+        <mass value="0.07637" />
+        <inertia ixx="45513E-9" ixy="0" ixz="-20691E-9" iyy="52570E-9" iyz="0" izz="17804E-9" />
       </inertial>
       <visual>
@@ -359,5 +311,5 @@
       </joint>
       <plugin filename="librobotiq_gripper_gazebo_plugin.so" name="hrim_actuation_gripper_000000000004">
-        <kp>1</kp>
+        <kp>1000</kp>
         <ki>0.1</ki>
         <kd>0.01</kd>

Commit message: add missing collision tags in S140

File: robotiq_140_gripper_description/urdf/robotiq_140.urdf (robot description, URDF)
Before this commit: robot robotiq_gripper, 10 links, 9 joints
Links:
- link left_inner_knuckle: geometry collision mesh filename=package://robotiq_140_gripper_description/meshes/robotiq_14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 scale=0.001 0.001 0.001; visual mesh filename=package://robotiq_140_gripper_description/meshes/robotiq_14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 scale=0.001 0.001 0.001
- link right_inner_knuckle: geometry collision mesh filename=package://robotiq_140_gripper_description/meshes/robotiq_14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 scale=0.001 0.001 0.001; visual mesh filename=package://robotiq_140_gripper_description/meshes/robotiq_14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 scale=0.001 0.001 0.001

File: robotiq_140_gripper_description/urdf/robotiq_140.urdf.xacro (robot description, xacro)
@@ -95,4 +95,10 @@
         </material>
       </visual>
+      <collision>
+        <origin xyz="0 0 0" rpy="0 0 0" />
+        <geometry>
+          <mesh filename="package://robotiq_140_gripper_description/meshes/robotiq_140_left_inner_knuckle.dae" scale="0.001 0.001 0.001"/>
+        </geometry>
+      </collision>
     </link>
     <gazebo reference="left_inner_knuckle">
@@ -115,4 +121,10 @@
         </material>
       </visual>
+      <collision>
+        <origin xyz="0 0 0" rpy="0 0 0" />
+        <geometry>
+          <mesh filename="package://robotiq_140_gripper_description/meshes/robotiq_140_right_inner_knuckle.dae" scale="0.001 0.001 0.001"/>
+        </geometry>
+      </collision>
     </link>
     <gazebo reference="right_inner_knuckle">
