Commit message: enable multiple S140

File: robotiq_140_gripper_description/urdf/robotiq_140.urdf (robot description, URDF)
Before this commit: robot robotiq_gripper, 10 links, 9 joints
Links:
- removed link left_inner_finger
- removed link left_inner_knuckle
- removed link left_outer_finger
- removed link left_outer_knuckle
- removed link right_inner_finger
- removed link right_inner_knuckle
- removed link right_outer_finger
- removed link right_outer_knuckle
- removed link robotiq_arg2f_base_link
- added link robotiq_140left_inner_finger, mass 0.045; collision mesh filename=package://robotiq_140_gripper_description/meshes/robotiq_14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 scale=0.001 0.001 0.001; visual mesh filename=package://robotiq_140_gripper_description/meshes/robotiq_14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 scale=0.001 0.001 0.001
- added link robotiq_140left_inner_knuckle, mass 0.04476; collision mesh filename=package://robotiq_140_gripper_description/meshes/robotiq_14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 scale=0.001 0.001 0.001; visual mesh filename=package://robotiq_140_gripper_description/meshes/robotiq_14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 scale=0.001 0.001 0.001
- added link robotiq_140left_outer_finger, mass 0.07637; collision mesh filename=package://robotiq_140_gripper_description/meshes/robotiq_14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 scale=0.001 0.001 0.001; visual mesh filename=package://robotiq_140_gripper_description/meshes/robotiq_14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 scale=0.001 0.001 0.001
- added link robotiq_140left_outer_knuckle, mass 0.0131; collision mesh filename=package://robotiq_140_gripper_description/meshes/robotiq_14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 scale=0.001 0.001 0.001; visual mesh filename=package://robotiq_140_gripper_description/meshes/robotiq_14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 scale=0.001 0.001 0.001
- added link robotiq_140right_inner_finger, mass 0.045; collision mesh filename=package://robotiq_140_gripper_description/meshes/robotiq_14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 scale=0.001 0.001 0.001; visual mesh filename=package://robotiq_140_gripper_description/meshes/robotiq_14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 scale=0.001 0.001 0.001
- added link robotiq_140right_inner_knuckle, mass 0.04476; collision mesh filename=package://robotiq_140_gripper_description/meshes/robotiq_14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 scale=0.001 0.001 0.001; visual mesh filename=package://robotiq_140_gripper_description/meshes/robotiq_14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 scale=0.001 0.001 0.001
- added link robotiq_140right_outer_finger, mass 0.07637; collision mesh filename=package://robotiq_140_gripper_description/meshes/robotiq_14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 scale=0.001 0.001 0.001; visual mesh filename=package://robotiq_140_gripper_description/meshes/robotiq_14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 scale=0.001 0.001 0.001
- added link robotiq_140right_outer_knuckle, mass 0.0131; collision mesh filename=package://robotiq_140_gripper_description/meshes/robotiq_14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 scale=0.001 0.001 0.001; visual mesh filename=package://robotiq_140_gripper_description/meshes/robotiq_14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 scale=0.001 0.001 0.001
- added link robotiq_140robotiq_arg2f_base_link, mass 0.52954; collision mesh filename=package://robotiq_140_gripper_description/meshes/GRIPPER_ba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 scale=0.001 0.001 0.001; visual mesh filename=package://robotiq_140_gripper_description/meshes/GRIPPER_ba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 scale=0.001 0.001 0.001
Joints:
- removed joint joint_finger
- removed joint left_outer_finger_to_inner
- removed joint left_outer_knuckle_to_finger
- removed joint right_outer_finger_to_inner
- removed joint right_outer_knuckle_to_finger
- removed joint robotiq_arg2f_base_to_left_inner_knuckle
- removed joint robotiq_arg2f_base_to_left_outer_knuckle
- removed joint robotiq_arg2f_base_to_right_inner_knuckle
- added joint robotiq_140joint_finger: type revolute, parent robotiq_140robotiq_arg2f_base_link, child robotiq_140right_outer_knuckle, origin xyz=-0.0306 0 0.05466 rpy=0 0 0, axis 0 1 0, limit lower=0 upper=0.78574722925 effort=18.65 velocity=3.54
- added joint robotiq_140left_outer_finger_to_inner: type revolute, parent robotiq_140left_outer_finger, child robotiq_140left_inner_finger, origin xyz=0.03543 0 0.0789 rpy=0 0 0, axis 0 1 0, limit lower=0 upper=0.78574722925 effort=18.65 velocity=3.54, mimic joint=robotiq_140joint_finger multiplier=1 offset=0
- added joint robotiq_140left_outer_knuckle_to_finger: type fixed, parent robotiq_140left_outer_knuckle, child robotiq_140left_outer_finger, origin xyz=0.03142 0 -0.00453 rpy=0 0 0
- added joint robotiq_140right_outer_finger_to_inner: type revolute, parent robotiq_140right_outer_finger, child robotiq_140right_inner_finger, origin xyz=-0.03543 0 0.0789 rpy=0 0 0, axis 0 -1 0, limit lower=0 upper=0.78574722925 effort=18.65 velocity=3.54, mimic joint=robotiq_140joint_finger multiplier=1 offset=0
- added joint robotiq_140right_outer_knuckle_to_finger: type fixed, parent robotiq_140right_outer_knuckle, child robotiq_140right_outer_finger, origin xyz=-0.03142 0 -0.00453 rpy=0 0 0
- added joint robotiq_arg2f_base_to_robotiq_140left_inner_knuckle: type revolute, parent robotiq_140robotiq_arg2f_base_link, child robotiq_140left_inner_knuckle, origin xyz=0.0127 0 0.06118 rpy=0 0 0, axis 0 -1 0, limit lower=0 upper=0.78574722925 effort=18.65 velocity=3.54, mimic joint=robotiq_140joint_finger multiplier=1 offset=0
- added joint robotiq_arg2f_base_to_robotiq_140left_outer_knuckle: type revolute, parent robotiq_140robotiq_arg2f_base_link, child robotiq_140left_outer_knuckle, origin xyz=0.0306 0 0.05466 rpy=0 0 0, axis 0 -1 0, limit lower=0 upper=0.78574722925 effort=18.65 velocity=2.0, mimic joint=robotiq_140joint_finger multiplier=1 offset=0
- added joint robotiq_arg2f_base_to_robotiq_140right_inner_knuckle: type revolute, parent robotiq_140robotiq_arg2f_base_link, child robotiq_140right_inner_knuckle, origin xyz=-0.0127 0 0.06118 rpy=0 0 0, axis 0 1 0, limit lower=0 upper=0.78574722925 effort=18.65 velocity=3.54, mimic joint=robotiq_140joint_finger multiplier=1 offset=0

File: robotiq_140_gripper_description/urdf/robotiq_140.urdf.xacro (robot description, xacro)
@@ -1,6 +1,6 @@
 <?xml version="1.0"?>
 <robot xmlns:xacro="http://ros.org/wiki/xacro">
-  <xacro:macro name="robotiq_gripper"  params="prefix">
-    <link name="robotiq_arg2f_base_link">
+  <xacro:macro name="robotiq_gripper"  params="prefix MAC">
+    <link name="${prefix}robotiq_arg2f_base_link">
       <inertial>
         <origin xyz="-0.00013 0.00011 0.03284" rpy="0 0 0" />
@@ -24,9 +24,9 @@
       </collision>
     </link>
-    <gazebo reference="robotiq_arg2f_base_link">
-      <material>Gazebo/Black</material>
-      <selfCollide>True</selfCollide>
-    </gazebo>
-    <link name="left_outer_knuckle">
+    <gazebo reference="${prefix}robotiq_arg2f_base_link">
+      <material>Gazebo/Black</material>
+      <selfCollide>True</selfCollide>
+    </gazebo>
+    <link name="${prefix}left_outer_knuckle">
       <inertial>
         <origin xyz="0.01616 0 -0.00133" rpy="0 0 0" />
@@ -50,9 +50,9 @@
       </collision>
     </link>
-    <gazebo reference="left_outer_knuckle">
+    <gazebo reference="${prefix}left_outer_knuckle">
       <material>Gazebo/Grey</material>
       <selfCollide>True</selfCollide>
     </gazebo>
-    <link name="right_outer_knuckle">
+    <link name="${prefix}right_outer_knuckle">
       <inertial>
         <origin xyz="-0.01616 0 -0.00133" rpy="0 0 0" />
@@ -76,9 +76,9 @@
       </collision>
     </link>
-    <gazebo reference="right_outer_knuckle">
+    <gazebo reference="${prefix}right_outer_knuckle">
       <material>Gazebo/Grey</material>
       <selfCollide>True</selfCollide>
     </gazebo>
-    <link name="left_inner_knuckle">
+    <link name="${prefix}left_inner_knuckle">
       <inertial>
         <origin xyz="0.03332 0 0.0379" rpy="0 0 0" />
@@ -102,9 +102,9 @@
       </collision>
     </link>
-    <gazebo reference="left_inner_knuckle">
+    <gazebo reference="${prefix}left_inner_knuckle">
       <material>Gazebo/Black</material>
       <selfCollide>False</selfCollide>
     </gazebo>
-    <link name="right_inner_knuckle">
+    <link name="${prefix}right_inner_knuckle">
       <inertial>
         <origin xyz="-0.03332 0 0.0379" rpy="0 0 0" />
@@ -128,9 +128,9 @@
       </collision>
     </link>
-    <gazebo reference="right_inner_knuckle">
+    <gazebo reference="${prefix}right_inner_knuckle">
       <material>Gazebo/Black</material>
       <selfCollide>False</selfCollide>
     </gazebo>
-    <link name="left_inner_finger">
+    <link name="${prefix}left_inner_finger">
       <inertial>
         <origin xyz="-0.01563 0 0.02522" rpy="0 0 0" />
@@ -154,9 +154,9 @@
       </collision>
     </link>
-    <gazebo reference="left_inner_finger">
+    <gazebo reference="${prefix}left_inner_finger">
       <material>Gazebo/Black</material>
       <selfCollide>False</selfCollide>
     </gazebo>
-    <link name="right_inner_finger">
+    <link name="${prefix}right_inner_finger">
       <inertial>
         <origin xyz="0.01563 0 0.02522" rpy="0 0 0" />
@@ -180,9 +180,9 @@
       </collision>
     </link>
-    <gazebo reference="right_inner_finger">
+    <gazebo reference="${prefix}right_inner_finger">
       <material>Gazebo/Black</material>
       <selfCollide>False</selfCollide>
     </gazebo>
-    <link name="left_outer_finger">
+    <link name="${prefix}left_outer_finger">
       <inertial>
         <origin xyz="0.01482 0 0.03451" rpy="0 0 0" />
@@ -206,9 +206,9 @@
       </collision>
     </link>
-    <gazebo reference="left_outer_finger">
-      <material>Gazebo/Black</material>
-      <selfCollide>True</selfCollide>
-    </gazebo>
-    <link name="right_outer_finger">
+    <gazebo reference="${prefix}left_outer_finger">
+      <material>Gazebo/Black</material>
+      <selfCollide>True</selfCollide>
+    </gazebo>
+    <link name="${prefix}right_outer_finger">
       <inertial>
         <origin xyz="-0.01482 0 0.03451" rpy="0 0 0" />
@@ -232,70 +232,70 @@
       </collision>
     </link>
-    <gazebo reference="right_outer_finger">
-      <material>Gazebo/Black</material>
-      <selfCollide>True</selfCollide>
-    </gazebo>
-    <joint name="robotiq_arg2f_base_to_left_outer_knuckle" type="revolute">
+    <gazebo reference="${prefix}right_outer_finger">
+      <material>Gazebo/Black</material>
+      <selfCollide>True</selfCollide>
+    </gazebo>
+    <joint name="robotiq_arg2f_base_to_${prefix}left_outer_knuckle" type="revolute">
       <origin xyz="0.0306 0 0.05466" rpy="0 0 0" />
-      <parent link="robotiq_arg2f_base_link" />
-      <child link="left_outer_knuckle" />
+      <parent link="${prefix}robotiq_arg2f_base_link" />
+      <child link="${prefix}left_outer_knuckle" />
       <axis xyz="0 -1 0" />
       <limit lower="0" upper="0.78574722925"  velocity="2.0" effort="18.65" />
-      <mimic joint="joint_finger" multiplier="1" offset="0"/>
-    </joint>
-    <joint name="joint_finger" type="revolute">
+      <mimic joint="${prefix}joint_finger" multiplier="1" offset="0"/>
+    </joint>
+    <joint name="${prefix}joint_finger" type="revolute">
       <origin xyz="-0.0306 0 0.05466" rpy="0 0 0" />
-      <parent link="robotiq_arg2f_base_link" />
-      <child link="right_outer_knuckle" />
+      <parent link="${prefix}robotiq_arg2f_base_link" />
+      <child link="${prefix}right_outer_knuckle" />
       <axis xyz="0 1 0" />
       <limit lower="0" upper="0.78574722925" velocity="3.54" effort="18.65" />
     </joint>
-    <joint name="robotiq_arg2f_base_to_left_inner_knuckle" type="revolute">
+    <joint name="robotiq_arg2f_base_to_${prefix}left_inner_knuckle" type="revolute">
       <origin xyz="0.0127 0 0.06118" rpy="0 0 0" />
-      <parent link="robotiq_arg2f_base_link" />
-      <child link="left_inner_knuckle" />
+      <parent link="${prefix}robotiq_arg2f_base_link" />
+      <child link="${prefix}left_inner_knuckle" />
       <axis xyz="0 -1 0" />
       <limit lower="0" upper="0.78574722925" velocity="3.54" effort="18.65" />
-      <mimic joint="joint_finger" multiplier="1" offset="0"/>
-    </joint>
-    <joint name="robotiq_arg2f_base_to_right_inner_knuckle" type="revolute">
+      <mimic joint="${prefix}joint_finger" multiplier="1" offset="0"/>
+    </joint>
+    <joint name="robotiq_arg2f_base_to_${prefix}right_inner_knuckle" type="revolute">
       <origin xyz="-0.0127 0 0.06118" rpy="0 0 0" />
-      <parent link="robotiq_arg2f_base_link" />
-      <child link="right_inner_knuckle" />
+      <parent link="${prefix}robotiq_arg2f_base_link" />
+      <child link="${prefix}right_inner_knuckle" />
       <axis xyz="0 1 0" />
       <limit lower="0" upper="0.78574722925" velocity="3.54" effort="18.65" />
-      <mimic joint="joint_finger" multiplier="1" offset="0"/>
-    </joint>
-    <joint name="left_outer_knuckle_to_finger" type="fixed">
+      <mimic joint="${prefix}joint_finger" multiplier="1" offset="0"/>
+    </joint>
+    <joint name="${prefix}left_outer_knuckle_to_finger" type="fixed">
       <origin xyz="0.03142 0 -0.00453" rpy="0 0 0" />
-      <parent link="left_outer_knuckle" />
-      <child link="left_outer_finger" />
-    </joint>
-    <joint name="right_outer_knuckle_to_finger" type="fixed">
+      <parent link="${prefix}left_outer_knuckle" />
+      <child link="${prefix}left_outer_finger" />
+    </joint>
+    <joint name="${prefix}right_outer_knuckle_to_finger" type="fixed">
       <origin xyz="-0.03142 0 -0.00453" rpy="0 0 0" />
-      <parent link="right_outer_knuckle" />
-      <child link="right_outer_finger" />
-    </joint>
-    <joint name="left_outer_finger_to_inner" type="revolute">
+      <parent link="${prefix}right_outer_knuckle" />
+      <child link="${prefix}right_outer_finger" />
+    </joint>
+    <joint name="${prefix}left_outer_finger_to_inner" type="revolute">
       <origin xyz="0.03543 0 0.0789" rpy="0 0 0" />
-      <parent link="left_outer_finger" />
-      <child link="left_inner_finger" />
+      <parent link="${prefix}left_outer_finger" />
+      <child link="${prefix}left_inner_finger" />
       <axis xyz="0 1 0" />
       <limit lower="0" upper="0.78574722925" velocity="3.54" effort="18.65" />
-      <mimic joint="joint_finger" multiplier="1" offset="0"/>
-    </joint>
-    <joint name="right_outer_finger_to_inner" type="revolute">
+      <mimic joint="${prefix}joint_finger" multiplier="1" offset="0"/>
+    </joint>
+    <joint name="${prefix}right_outer_finger_to_inner" type="revolute">
       <origin xyz="-0.03543 0 0.0789" rpy="0 0 0" />
-      <parent link="right_outer_finger" />
-      <child link="right_inner_finger" />
+      <parent link="${prefix}right_outer_finger" />
+      <child link="${prefix}right_inner_finger" />
       <axis xyz="0 -1 0" />
       <limit lower="0" upper="0.78574722925" velocity="3.54" effort="18.65" />
-      <mimic joint="joint_finger" multiplier="1" offset="0"/>
+      <mimic joint="${prefix}joint_finger" multiplier="1" offset="0"/>
     </joint>
     <gazebo>
-      <joint name="left_inner_knuckle_to_finger" type="revolute">
+      <joint name="${prefix}left_inner_knuckle_to_finger" type="revolute">
         <pose frame="">-0.0179 0 0.00652 0 0 0</pose>
-        <parent>${prefix}::left_inner_knuckle</parent>
-        <child>${prefix}::left_inner_finger</child>
+        <parent>${prefix}left_inner_knuckle</parent>
+        <child>${prefix}left_inner_finger</child>
         <axis>
           <xyz>0 1 0</xyz>
@@ -308,8 +308,8 @@
         </axis>
       </joint>
-      <joint name="right_inner_knuckle_to_finger" type="revolute">
+      <joint name="${prefix}right_inner_knuckle_to_finger" type="revolute">
         <pose frame="">0.0179 0 0.00652 0 0 0</pose>
-        <parent>${prefix}::right_inner_knuckle</parent>
-        <child>${prefix}::right_inner_finger</child>
+        <parent>${prefix}right_inner_knuckle</parent>
+        <child>${prefix}right_inner_finger</child>
         <axis>
           <xyz>0 -1 0</xyz>
@@ -322,19 +322,12 @@
         </axis>
       </joint>
-      <plugin filename="librobotiq_gripper_gazebo_plugin.so" name="hrim_actuation_gripper_000000000004">
-        <kp>500</kp>
+      <plugin filename="librobotiq_gripper_gazebo_plugin.so" name="hrim_actuator_gripper${MAC}">
+        <kp>600</kp>
         <ki>0.1</ki>
         <kd>0.01</kd>
-        <joint>robotiq_arg2f_base_to_left_inner_knuckle</joint>
-        <joint>robotiq_arg2f_base_to_left_outer_knuckle</joint>
-        <joint>robotiq_arg2f_base_to_right_inner_knuckle</joint>
-        <joint>joint_finger</joint>
-      </plugin>
-      <plugin filename="libgazebo_ros_joint_state_publisher.so" name="mara_joint_state">
-        <ros>
-          <argument>~/out:=joint_states</argument>
-        </ros>
-        <update_rate>25</update_rate>
-        <joint_name>joint_finger</joint_name>
+        <joint>robotiq_arg2f_base_to_${prefix}left_inner_knuckle</joint>
+        <joint>robotiq_arg2f_base_to_${prefix}left_outer_knuckle</joint>
+        <joint>robotiq_arg2f_base_to_${prefix}right_inner_knuckle</joint>
+        <joint>${prefix}joint_finger</joint>
       </plugin>
     </gazebo>

File: robotiq_140_gripper_description/urdf/robotiq_140_world.urdf.xacro (robot description, xacro)
@@ -2,5 +2,5 @@
 <robot xmlns:xacro="http://ros.org/wiki/xacro" name="robotiq_gripper" >
   <xacro:include filename="$(find robotiq_140_gripper_description)/urdf/robotiq_140.urdf.xacro" />
-  <xacro:robotiq_gripper prefix="robotiq_140"/>
+  <xacro:robotiq_gripper prefix="robotiq_140" MAC="_000000000004"/>
   <link name="world" />
   <joint name="world_to_robotiq_adapter" type="fixed">
