Commit message: fix libgazebo_ros_joint_state_publisher plugin

File: robotiq_140_gripper_description/urdf/robotiq_140.urdf (robot description, URDF)
Before this commit: robot robotiq_gripper, 10 links, 9 joints
Links:
- removed link robotiq_140left_inner_finger
- removed link robotiq_140left_inner_knuckle
- removed link robotiq_140left_outer_finger
- removed link robotiq_140left_outer_knuckle
- removed link robotiq_140right_inner_finger
- removed link robotiq_140right_inner_knuckle
- removed link robotiq_140right_outer_finger
- removed link robotiq_140right_outer_knuckle
- removed link robotiq_140robotiq_arg2f_base_link
- added link robotiq_140_left_inner_finger, mass 0.045; collision mesh filename=package://robotiq_140_gripper_description/meshes/robotiq_14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 scale=0.001 0.001 0.001; visual mesh filename=package://robotiq_140_gripper_description/meshes/robotiq_14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 scale=0.001 0.001 0.001
- added link robotiq_140_left_inner_knuckle, mass 0.04476; collision mesh filename=package://robotiq_140_gripper_description/meshes/robotiq_14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 scale=0.001 0.001 0.001; visual mesh filename=package://robotiq_140_gripper_description/meshes/robotiq_14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 scale=0.001 0.001 0.001
- added link robotiq_140_left_outer_finger, mass 0.07637; collision mesh filename=package://robotiq_140_gripper_description/meshes/robotiq_14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 scale=0.001 0.001 0.001; visual mesh filename=package://robotiq_140_gripper_description/meshes/robotiq_14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 scale=0.001 0.001 0.001
- added link robotiq_140_left_outer_knuckle, mass 0.0131; collision mesh filename=package://robotiq_140_gripper_description/meshes/robotiq_14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 scale=0.001 0.001 0.001; visual mesh filename=package://robotiq_140_gripper_description/meshes/robotiq_14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 scale=0.001 0.001 0.001
- added link robotiq_140_right_inner_finger, mass 0.045; collision mesh filename=package://robotiq_140_gripper_description/meshes/robotiq_14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 scale=0.001 0.001 0.001; visual mesh filename=package://robotiq_140_gripper_description/meshes/robotiq_14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 scale=0.001 0.001 0.001
- added link robotiq_140_right_inner_knuckle, mass 0.04476; collision mesh filename=package://robotiq_140_gripper_description/meshes/robotiq_14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 scale=0.001 0.001 0.001; visual mesh filename=package://robotiq_140_gripper_description/meshes/robotiq_14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 scale=0.001 0.001 0.001
- added link robotiq_140_right_outer_finger, mass 0.07637; collision mesh filename=package://robotiq_140_gripper_description/meshes/robotiq_14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 scale=0.001 0.001 0.001; visual mesh filename=package://robotiq_140_gripper_description/meshes/robotiq_14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 scale=0.001 0.001 0.001
- added link robotiq_140_right_outer_knuckle, mass 0.0131; collision mesh filename=package://robotiq_140_gripper_description/meshes/robotiq_14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 scale=0.001 0.001 0.001; visual mesh filename=package://robotiq_140_gripper_description/meshes/robotiq_14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 scale=0.001 0.001 0.001
- added link robotiq_140_robotiq_arg2f_base_link, mass 0.52954; collision mesh filename=package://robotiq_140_gripper_description/meshes/GRIPPER_ba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 scale=0.001 0.001 0.001; visual mesh filename=package://robotiq_140_gripper_description/meshes/GRIPPER_ba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 scale=0.001 0.001 0.001
Joints:
- removed joint robotiq_140joint_finger
- removed joint robotiq_140left_outer_finger_to_inner
- removed joint robotiq_140left_outer_knuckle_to_finger
- removed joint robotiq_140right_outer_finger_to_inner
- removed joint robotiq_140right_outer_knuckle_to_finger
- removed joint robotiq_arg2f_base_to_robotiq_140left_inner_knuckle
- removed joint robotiq_arg2f_base_to_robotiq_140left_outer_knuckle
- removed joint robotiq_arg2f_base_to_robotiq_140right_inner_knuckle
- added joint robotiq_140_joint_finger: type revolute, parent robotiq_140_robotiq_arg2f_base_link, child robotiq_140_right_outer_knuckle, origin xyz=-0.0306 0 0.05466 rpy=0 0 0, axis 0 1 0, limit lower=0 upper=0.78574722925 effort=18.65 velocity=3.54
- added joint robotiq_140_left_outer_finger_to_inner: type revolute, parent robotiq_140_left_outer_finger, child robotiq_140_left_inner_finger, origin xyz=0.03543 0 0.0789 rpy=0 0 0, axis 0 1 0, limit lower=0 upper=0.78574722925 effort=18.65 velocity=3.54, mimic joint=robotiq_140_joint_finger multiplier=1 offset=0
- added joint robotiq_140_left_outer_knuckle_to_finger: type fixed, parent robotiq_140_left_outer_knuckle, child robotiq_140_left_outer_finger, origin xyz=0.03142 0 -0.00453 rpy=0 0 0
- added joint robotiq_140_right_outer_finger_to_inner: type revolute, parent robotiq_140_right_outer_finger, child robotiq_140_right_inner_finger, origin xyz=-0.03543 0 0.0789 rpy=0 0 0, axis 0 -1 0, limit lower=0 upper=0.78574722925 effort=18.65 velocity=3.54, mimic joint=robotiq_140_joint_finger multiplier=1 offset=0
- added joint robotiq_140_right_outer_knuckle_to_finger: type fixed, parent robotiq_140_right_outer_knuckle, child robotiq_140_right_outer_finger, origin xyz=-0.03142 0 -0.00453 rpy=0 0 0
- added joint robotiq_arg2f_base_to_robotiq_140_left_inner_knuckle: type revolute, parent robotiq_140_robotiq_arg2f_base_link, child robotiq_140_left_inner_knuckle, origin xyz=0.0127 0 0.06118 rpy=0 0 0, axis 0 -1 0, limit lower=0 upper=0.78574722925 effort=18.65 velocity=3.54, mimic joint=robotiq_140_joint_finger multiplier=1 offset=0
- added joint robotiq_arg2f_base_to_robotiq_140_left_outer_knuckle: type revolute, parent robotiq_140_robotiq_arg2f_base_link, child robotiq_140_left_outer_knuckle, origin xyz=0.0306 0 0.05466 rpy=0 0 0, axis 0 -1 0, limit lower=0 upper=0.78574722925 effort=18.65 velocity=2.0, mimic joint=robotiq_140_joint_finger multiplier=1 offset=0
- added joint robotiq_arg2f_base_to_robotiq_140_right_inner_knuckle: type revolute, parent robotiq_140_robotiq_arg2f_base_link, child robotiq_140_right_inner_knuckle, origin xyz=-0.0127 0 0.06118 rpy=0 0 0, axis 0 1 0, limit lower=0 upper=0.78574722925 effort=18.65 velocity=3.54, mimic joint=robotiq_140_joint_finger multiplier=1 offset=0
- joint world_to_robotiq_adapter: child robotiq_arg2f_base_link -> robotiq_140_robotiq_arg2f_base_link

File: robotiq_140_gripper_description/urdf/robotiq_140.urdf.xacro (robot description, xacro)
@@ -331,4 +331,11 @@
         <joint>${prefix}joint_finger</joint>
       </plugin>
+      <plugin filename="libgazebo_ros_joint_state_publisher.so" name="${prefix}joint_state">
+        <ros>
+          <argument>~/out:=${prefix}joint_states</argument>
+        </ros>
+        <update_rate>25</update_rate>
+        <joint_name>${prefix}joint_finger</joint_name>
+      </plugin>
     </gazebo>
   </xacro:macro>

File: robotiq_140_gripper_description/urdf/robotiq_140_world.urdf.xacro (robot description, xacro)
@@ -2,10 +2,10 @@
 <robot xmlns:xacro="http://ros.org/wiki/xacro" name="robotiq_gripper" >
   <xacro:include filename="$(find robotiq_140_gripper_description)/urdf/robotiq_140.urdf.xacro" />
-  <xacro:robotiq_gripper prefix="robotiq_140" MAC="_000000000004"/>
+  <xacro:robotiq_gripper prefix="robotiq_140_" MAC="_000000000004"/>
   <link name="world" />
   <joint name="world_to_robotiq_adapter" type="fixed">
     <origin rpy="0 0 0" xyz="0 0 0.5"/>
     <parent link="world"/>
-    <child link="robotiq_arg2f_base_link"/>
+    <child link="robotiq_140_robotiq_arg2f_base_link"/>
   </joint>
 </robot>

File: robotiq_85_gripper_description/urdf/robotiq_85.urdf (robot description, URDF)
Before this commit: robot robotiq_85, 10 links, 9 joints
Links:
- removed link robotiq85left_inner_finger
- removed link robotiq85left_inner_knuckle
- removed link robotiq85left_outer_finger
- removed link robotiq85left_outer_knuckle
- removed link robotiq85right_inner_finger
- removed link robotiq85right_inner_knuckle
- removed link robotiq85right_outer_finger
- removed link robotiq85right_outer_knuckle
- removed link robotiq85robotiq_arg2f_base_link
- added link robotiq_85_left_inner_finger, mass 0.037; collision mesh filename=package://robotiq_85_gripper_description/meshes/2-F-85_4_l.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 scale=0.001 0.001 0.001; visual mesh filename=package://robotiq_85_gripper_description/meshes/2-F-85_4_l.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 scale=0.001 0.001 0.001
- added link robotiq_85_left_inner_knuckle, mass 0.02731; collision mesh filename=package://robotiq_85_gripper_description/meshes/2-F-85_2_l.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 scale=0.001 0.001 0.001; visual mesh filename=package://robotiq_85_gripper_description/meshes/2-F-85_2_l.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 scale=0.001 0.001 0.001
- added link robotiq_85_left_outer_finger, mass 0.03848; collision mesh filename=package://robotiq_85_gripper_description/meshes/2-F-85_3_l.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 scale=0.001 0.001 0.001; visual mesh filename=package://robotiq_85_gripper_description/meshes/2-F-85_3_l.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 scale=0.001 0.001 0.001
- added link robotiq_85_left_outer_knuckle, mass 0.01252; collision mesh filename=package://robotiq_85_gripper_description/meshes/2-F-85_1_l.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 scale=0.001 0.001 0.001; visual mesh filename=package://robotiq_85_gripper_description/meshes/2-F-85_1_l.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 scale=0.001 0.001 0.001
- added link robotiq_85_right_inner_finger, mass 0.037; collision mesh filename=package://robotiq_85_gripper_description/meshes/2-F-85_4_r.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 scale=0.001 0.001 0.001; visual mesh filename=package://robotiq_85_gripper_description/meshes/2-F-85_4_r.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 scale=0.001 0.001 0.001
- added link robotiq_85_right_inner_knuckle, mass 0.02731; collision mesh filename=package://robotiq_85_gripper_description/meshes/2-F-85_2_r.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 scale=0.001 0.001 0.001; visual mesh filename=package://robotiq_85_gripper_description/meshes/2-F-85_2_r.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 scale=0.001 0.001 0.001
- added link robotiq_85_right_outer_finger, mass 0.03848; collision mesh filename=package://robotiq_85_gripper_description/meshes/2-F-85_3_r.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 scale=0.001 0.001 0.001; visual mesh filename=package://robotiq_85_gripper_description/meshes/2-F-85_3_r.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 scale=0.001 0.001 0.001
- added link robotiq_85_right_outer_knuckle, mass 0.01252; collision mesh filename=package://robotiq_85_gripper_description/meshes/2-F-85_1_r.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 scale=0.001 0.001 0.001; visual mesh filename=package://robotiq_85_gripper_description/meshes/2-F-85_1_r.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 scale=0.001 0.001 0.001
- added link robotiq_85_robotiq_arg2f_base_link, mass 0.55938; collision mesh filename=package://robotiq_85_gripper_description/meshes/base_grippe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 scale=0.001 0.001 0.001; visual mesh filename=package://robotiq_85_gripper_description/meshes/base_grippe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 scale=0.001 0.001 0.001
Joints:
- removed joint robotiq85joint_finger
- removed joint robotiq85left_outer_finger_to_inner
- removed joint robotiq85left_outer_knuckle_to_finger
- removed joint robotiq85right_outer_finger_to_inner
- removed joint robotiq85right_outer_knuckle_to_finger
- removed joint robotiq85robotiq_arg2f_base_link_to_robotiq85left_inner_knuckle
- removed joint robotiq85robotiq_arg2f_base_link_to_robotiq85left_outer_knuckle
- removed joint robotiq85robotiq_arg2f_base_link_to_robotiq85right_inner_knuckle
- added joint robotiq_85_joint_finger: type revolute, parent robotiq_85_robotiq_arg2f_base_link, child robotiq_85_right_outer_knuckle, origin xyz=-0.0306 0 0.05466 rpy=0 0 0, axis 0 1 0, limit lower=0 upper=0.82589 effort=21.03 velocity=3.87
- added joint robotiq_85_left_outer_finger_to_inner: type revolute, parent robotiq_85_left_outer_finger, child robotiq_85_left_inner_finger, origin xyz=0.00678 0 0.04703 rpy=0 0 0, axis 0 1 0, limit lower=0 upper=0.82589 effort=21.03 velocity=3.87, mimic joint=robotiq_85_joint_finger multiplier=1 offset=0
- added joint robotiq_85_left_outer_knuckle_to_finger: type fixed, parent robotiq_85_left_outer_knuckle, child robotiq_85_left_outer_finger, origin xyz=0.03142 0 -0.00453 rpy=0 0 0
- added joint robotiq_85_right_outer_finger_to_inner: type revolute, parent robotiq_85_right_outer_finger, child robotiq_85_right_inner_finger, origin xyz=-0.00678 0 0.04703 rpy=0 0 0, axis 0 -1 0, limit lower=0 upper=0.82589 effort=21.03 velocity=3.87, mimic joint=robotiq_85_joint_finger multiplier=1 offset=0
- added joint robotiq_85_right_outer_knuckle_to_finger: type fixed, parent robotiq_85_right_outer_knuckle, child robotiq_85_right_outer_finger, origin xyz=-0.03142 0 -0.00453 rpy=0 0 0
- added joint robotiq_85_robotiq_arg2f_base_link_to_robotiq_85_left_inner_knuckle: type revolute, parent robotiq_85_robotiq_arg2f_base_link, child robotiq_85_left_inner_knuckle, origin xyz=0.0127 0 0.06118 rpy=0 0 0, axis 0 -1 0, limit lower=0 upper=0.82589 effort=21.03 velocity=3.87, mimic joint=robotiq_85_joint_finger multiplier=1 offset=0
- added joint robotiq_85_robotiq_arg2f_base_link_to_robotiq_85_left_outer_knuckle: type revolute, parent robotiq_85_robotiq_arg2f_base_link, child robotiq_85_left_outer_knuckle, origin xyz=0.0306 0 0.05466 rpy=0 0 0, axis 0 -1 0, limit lower=0 upper=0.82589 effort=21.03 velocity=3.87, mimic joint=robotiq_85_joint_finger multiplier=1 offset=0
- added joint robotiq_85_robotiq_arg2f_base_link_to_robotiq_85_right_inner_knuckle: type revolute, parent robotiq_85_robotiq_arg2f_base_link, child robotiq_85_right_inner_knuckle, origin xyz=-0.0127 0 0.06118 rpy=0 0 0, axis 0 1 0, limit lower=0 upper=0.82589 effort=21.03 velocity=3.87, mimic joint=robotiq_85_joint_finger multiplier=1 offset=0
- joint world_to_robotiq_arg2f_base: child robotiq_arg2f_base_link -> robotiq_85_robotiq_arg2f_base_link

File: robotiq_85_gripper_description/urdf/robotiq_85.urdf.xacro (robot description, xacro)
@@ -331,7 +331,7 @@
         <joint>${prefix}joint_finger</joint>
       </plugin>
-      <plugin filename="libgazebo_ros_joint_state_publisher.so" name="mara_joint_state">
+      <plugin filename="libgazebo_ros_joint_state_publisher.so" name="${prefix}joint_state">
         <ros>
-          <argument>~/out:=joint_states</argument>
+          <argument>~/out:=${prefix}joint_states</argument>
         </ros>
         <update_rate>25</update_rate>

File: robotiq_85_gripper_description/urdf/robotiq_85_world.urdf.xacro (robot description, xacro)
@@ -2,10 +2,10 @@
 <robot xmlns:xacro="http://ros.org/wiki/xacro" name="robotiq_85" >
   <xacro:include filename="$(find robotiq_85_gripper_description)/urdf/robotiq_85.urdf.xacro" />
-  <xacro:robotiq_85 prefix="robotiq85" MAC="_000000000004"/>
+  <xacro:robotiq_85 prefix="robotiq_85_" MAC="_000000000004"/>
   <link name="world" />
   <joint name="world_to_robotiq_arg2f_base" type="fixed">
     <origin rpy="0 0 0" xyz="0 0 0.5"/>
     <parent link="world"/>
-    <child link="robotiq_arg2f_base_link"/>
+    <child link="robotiq_85_robotiq_arg2f_base_link"/>
   </joint>
 </robot>

File: robotiq_hande_gripper_description/urdf/robotiq_hande.urdf (robot description, URDF)
Before this commit: robot robotiq_hande, 4 links, 3 joints
Links:
- removed link handeleft_finger
- removed link handeright_finger
- removed link handerobotiq_hande_base_link
- added link hande_left_finger, mass 0.03804; collision mesh filename=package://robotiq_hande_gripper_description/meshes/finger_1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 scale=0.001 0.001 0.001; visual mesh filename=package://robotiq_hande_gripper_description/meshes/finger_1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 scale=0.001 0.001 0.001
- added link hande_right_finger, mass 0.03804; collision mesh filename=package://robotiq_hande_gripper_description/meshes/finger_2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 scale=0.001 0.001 0.001; visual mesh filename=package://robotiq_hande_gripper_description/meshes/finger_2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 scale=0.001 0.001 0.001
- added link hande_robotiq_hande_base_link, mass 0.86387; collision mesh filename=package://robotiq_hande_gripper_description/meshes/hand-e.d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 scale=0.001 0.001 0.001; visual mesh filename=package://robotiq_hande_gripper_description/meshes/hand-e.d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 scale=0.001 0.001 0.001
Joints:
- removed joint handejoint_finger
- removed joint robotiq_hande_base_to_handeright_finger
- added joint hande_joint_finger: type prismatic, parent hande_robotiq_hande_base_link, child hande_left_finger, origin xyz=0 0 0.099 rpy=0 0 0, axis -1 0 0, limit lower=0 upper=0.025 effort=130 velocity=0.15
- added joint robotiq_hande_base_to_hande_right_finger: type prismatic, parent hande_robotiq_hande_base_link, child hande_right_finger, origin xyz=0 0 0.099 rpy=0 0 0, axis 1 0 0, limit lower=0 upper=0.025 effort=130 velocity=0.15, mimic joint=hande_joint_finger multiplier=1 offset=0
- joint world_to_robotiq_adapter: child robotiq_hande_base_link -> hande_robotiq_hande_base_link

File: robotiq_hande_gripper_description/urdf/robotiq_hande.urdf.xacro (robot description, xacro)
@@ -103,7 +103,7 @@
         <joint>robotiq_hande_base_to_${prefix}right_finger</joint>
       </plugin>
-      <plugin filename="libgazebo_ros_joint_state_publisher.so" name="mara_joint_state">
+      <plugin filename="libgazebo_ros_joint_state_publisher.so" name="${prefix}joint_state">
         <ros>
-          <argument>~/out:=joint_states</argument>
+          <argument>~/out:=${prefix}joint_states</argument>
         </ros>
         <update_rate>25</update_rate>

File: robotiq_hande_gripper_description/urdf/robotiq_hande_world.urdf.xacro (robot description, xacro)
@@ -3,10 +3,10 @@
   <!-- robotiq_hande_gripper -->
   <xacro:include filename="$(find robotiq_hande_gripper_description)/urdf/robotiq_hande.urdf.xacro" />
-  <xacro:robotiq_hande prefix="hande" MAC="_000000000004"/>
+  <xacro:robotiq_hande prefix="hande_" MAC="_000000000004"/>
   <link name="world" />
   <joint name="world_to_robotiq_adapter" type="fixed">
     <origin rpy="0 0 0" xyz="0 0 0.5"/>
     <parent link="world"/>
-    <child link="robotiq_hande_base_link"/>
+    <child link="hande_robotiq_hande_base_link"/>
   </joint>
 </robot>
