Commit message: Updating robotiq 85

File: robotiq_85_gripper_description/urdf/robotiq_85.urdf.xacro (robot description, xacro)
@@ -2,4 +2,35 @@
 <robot xmlns:xacro="http://ros.org/wiki/xacro">
   <xacro:macro name="robotiq_85"  params="prefix">
+    <link name="robotiq_adapter_link">
+      <inertial>
+        <origin xyz="8.625E-08 -4.6583E-06 0.03145" rpy="0 0 0" />
+        <mass value="0.22652" />
+        <inertia ixx="0.00020005" ixy="0" ixz="0" iyy="0.00017832" iyz="0" izz="0.00013478" />
+      </inertial>
+      <visual>
+        <origin xyz="0 0 0" rpy="0 0 1.57" />
+        <geometry>
+          <mesh filename="package://robotiq_85_gripper_description/meshes/hros_robotiq_adapter.dae" scale="0.001 0.001 0.001"/>
+        </geometry>
+        <material name="Gazebo/Black">
+          <color rgba="0.0 0.0 0.0 1" />
+        </material>
+      </visual>
+      <collision>
+        <origin xyz="0 0 0" rpy="0 0 1.57" />
+        <geometry>
+          <mesh filename="package://robotiq_85_gripper_description/meshes/hros_robotiq_adapter.dae" scale="0.001 0.001 0.001"/>
+        </geometry>
+      </collision>
+    </link>
+    <gazebo reference="robotiq_adapter_link">
+      <material>Gazebo/Black</material>
+      <selfCollide>False</selfCollide>
+    </gazebo>
+    <joint name="base_adapter_to_base_robotiq_joint" type="fixed">
+      <origin rpy="0 0 0" xyz=" 0 0 0.03653"/>
+      <parent link="robotiq_adapter_link" />
+      <child link="robotiq_arg2f_base"/>
+    </joint>
     <link name="robotiq_arg2f_base">
       <inertial>

Commit message: fix upper limit

File: robotiq_85_gripper_description/urdf/robotiq_85.urdf.xacro (robot description, xacro)
@@ -241,5 +241,5 @@
       <child link="left_outer_knuckle" />
       <axis xyz="0 -1 0" />
-      <limit lower="0.0" upper="0.78" velocity="2.0" effort="1000" />
+      <limit lower="0" upper="0.82589" velocity="3.87" effort="21.03" />
       <mimic joint="joint_finger" multiplier="1" offset="0"/>
     </joint>
@@ -249,5 +249,5 @@
       <child link="right_outer_knuckle" />
       <axis xyz="0 1 0" />
-      <limit lower="0" upper="0.78" velocity="2.0" effort="1000" />
+      <limit lower="0" upper="0.82589" velocity="3.87" effort="21.03" />
     </joint>
     <joint name="robotiq_arg2f_base_link_to_left_inner_knuckle" type="revolute">
@@ -256,5 +256,5 @@
       <child link="left_inner_knuckle" />
       <axis xyz="0 -1 0" />
-      <limit lower="0" upper="0.8757" velocity="2.0" effort="1000" />
+      <limit lower="0" upper="0.82589" velocity="3.87" effort="21.03" />
       <mimic joint="joint_finger" multiplier="1" offset="0"/>
     </joint>
@@ -264,5 +264,5 @@
       <child link="right_inner_knuckle" />
       <axis xyz="0 1 0" />
-      <limit lower="0" upper="0.8757" velocity="2.0" effort="1000" />
+      <limit lower="0" upper="0.82589" velocity="3.87" effort="21.03" />
       <mimic joint="joint_finger" multiplier="1" offset="0"/>
     </joint>
@@ -272,5 +272,5 @@
       <child link="left_inner_finger" />
       <axis xyz="0 1 0" />
-      <limit lower="0" upper="0.775" velocity="2.0" effort="1000" />
+      <limit lower="0" upper="0.82589" velocity="3.87" effort="21.03" />
       <mimic joint="joint_finger" multiplier="1" offset="0"/>
     </joint>
@@ -280,5 +280,5 @@
       <child link="right_inner_finger" />
       <axis xyz="0 -1 0" />
-      <limit lower="0" upper="0.775" velocity="2.0" effort="1000" />
+      <limit lower="0" upper="0.82589" velocity="3.87" effort="21.03" />
       <mimic joint="joint_finger" multiplier="1" offset="0"/>
     </joint>
@@ -301,8 +301,8 @@
           <xyz>0 1 0</xyz>
           <limit>
-            <lower>-0.8</lower>
-            <upper>0.8</upper>
-            <velocity>2.0</velocity>
-            <effort>1000</effort>
+            <lower>0</lower>
+            <upper>0.82589</upper>
+            <velocity>3.87</velocity>
+            <effort>21.03</effort>
           </limit>
         </axis>
@@ -315,8 +315,8 @@
           <xyz>0 -1 0</xyz>
           <limit>
-            <lower>-0.8</lower>
-            <upper>0.8</upper>
-            <velocity>2.0</velocity>
-            <effort>1000</effort>
+            <lower>0</lower>
+            <upper>0.82589</upper>
+            <velocity>3.87</velocity>
+            <effort>21.03</effort>
           </limit>
         </axis>

Commit message: fix S85 right_inner inertia and make only inner self collide false

File: robotiq_85_gripper_description/urdf/robotiq_85.urdf.xacro (robot description, xacro)
@@ -26,5 +26,5 @@
     <gazebo reference="robotiq_arg2f_base_link">
       <material>Gazebo/Black</material>
-      <selfCollide>False</selfCollide>
+      <selfCollide>True</selfCollide>
     </gazebo>
     <link name="left_outer_knuckle">
@@ -52,5 +52,5 @@
     <gazebo reference="left_outer_knuckle">
       <material>Gazebo/Grey</material>
-      <selfCollide>False</selfCollide>
+      <selfCollide>True</selfCollide>
     </gazebo>
     <link name="right_outer_knuckle">
@@ -78,5 +78,5 @@
     <gazebo reference="right_outer_knuckle">
       <material>Gazebo/Grey</material>
-      <selfCollide>False</selfCollide>
+      <selfCollide>True</selfCollide>
     </gazebo>
     <link name="left_outer_finger">
@@ -104,5 +104,5 @@
     <gazebo reference="left_outer_finger">
       <material>Gazebo/Black</material>
-      <selfCollide>False</selfCollide>
+      <selfCollide>True</selfCollide>
     </gazebo>
     <link name="right_outer_finger">
@@ -130,5 +130,5 @@
     <gazebo reference="right_outer_finger">
       <material>Gazebo/Black</material>
-      <selfCollide>False</selfCollide>
+      <selfCollide>True</selfCollide>
     </gazebo>
     <link name="left_inner_knuckle">
@@ -162,5 +162,5 @@
         <origin xyz="-0.01952 0 0.022" rpy="0 0 0" />
         <mass value="0.02731" />
-        <inertia ixx="8621.3E-9" ixy="0" ixz="-3646.49E-9" iyy="8004.28E-9" iyz="0" izz="7704.42E-9" />
+        <inertia ixx="8621.3E-9" ixy="0" ixz="3646.49E-9" iyy="8004.28E-9" iyz="0" izz="7704.42E-9" />
       </inertial>
       <visual>
@@ -214,5 +214,5 @@
         <origin xyz="0.01409 0 0.01569" rpy="0 0 0" />
         <mass value="0.037" />
-        <inertia ixx="12446.57E-9" ixy="0" ixz="4167.81E-9" iyy="14201.18E-9" iyz="0" izz="4979.86E-9" />
+        <inertia ixx="12446.57E-9" ixy="0" ixz="-4167.81E-9" iyy="14201.18E-9" iyz="0" izz="4979.86E-9" />
       </inertial>
       <visual>
