Commit message: update URDFs robotiq 85

File: robotiq_85_gripper_description/urdf/robotiq_85.urdf (robot description, URDF)
Before this commit: robot robotiq_85, 11 links, 10 joints
Links:
- removed link robotiq_85_base_link
- removed link robotiq_85_left_finger_link
- removed link robotiq_85_left_inner_finger_link
- removed link robotiq_85_left_inner_knuckle_link
- removed link robotiq_85_left_outer_knuckle_link
- removed link robotiq_85_right_finger_link
- removed link robotiq_85_right_inner_finger_link
- removed link robotiq_85_right_inner_knuckle_link
- removed link robotiq_85_right_outer_knuckle_link
- added link left_inner_finger, mass 0.22652; collision mesh filename=package://robotiq_85_gripper_description/meshes/2-F-85_4_l.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 scale=0.001 0.001 0.001; visual mesh filename=package://robotiq_85_gripper_description/meshes/2-F-85_4_l.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 scale=0.001 0.001 0.001
- added link left_inner_knuckle, mass 0.22652; collision mesh filename=package://robotiq_85_gripper_description/meshes/2-F-85_2_l.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 scale=0.001 0.001 0.001; visual mesh filename=package://robotiq_85_gripper_description/meshes/2-F-85_2_l.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 scale=0.001 0.001 0.001
- added link left_outer_finger, mass 0.22652; collision mesh filename=package://robotiq_85_gripper_description/meshes/2-F-85_3_l.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 scale=0.001 0.001 0.001; visual mesh filename=package://robotiq_85_gripper_description/meshes/2-F-85_3_l.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 scale=0.001 0.001 0.001
- added link left_outer_knuckle, mass 0.22652; collision mesh filename=package://robotiq_85_gripper_description/meshes/2-F-85_1_l.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 scale=0.001 0.001 0.001; visual mesh filename=package://robotiq_85_gripper_description/meshes/2-F-85_1_l.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 scale=0.001 0.001 0.001
- added link right_inner_finger, mass 0.22652; collision mesh filename=package://robotiq_85_gripper_description/meshes/2-F-85_4_r.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 scale=0.001 0.001 0.001; visual mesh filename=package://robotiq_85_gripper_description/meshes/2-F-85_4_r.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 scale=0.001 0.001 0.001
- added link right_inner_knuckle, mass 0.22652; collision mesh filename=package://robotiq_85_gripper_description/meshes/2-F-85_2_r.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 scale=0.001 0.001 0.001; visual mesh filename=package://robotiq_85_gripper_description/meshes/2-F-85_2_r.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 scale=0.001 0.001 0.001
- added link right_outer_finger, mass 0.22652; collision mesh filename=package://robotiq_85_gripper_description/meshes/2-F-85_3_r.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 scale=0.001 0.001 0.001; visual mesh filename=package://robotiq_85_gripper_description/meshes/2-F-85_3_r.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 scale=0.001 0.001 0.001
- added link right_outer_knuckle, mass 0.22652; collision mesh filename=package://robotiq_85_gripper_description/meshes/2-F-85_1_r.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 scale=0.001 0.001 0.001; visual mesh filename=package://robotiq_85_gripper_description/meshes/2-F-85_1_r.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 scale=0.001 0.001 0.001
- added link robotiq_arg2f_base, mass 0.22652; collision mesh filename=package://robotiq_85_gripper_description/meshes/base_grippe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 scale=0.001 0.001 0.001; visual mesh filename=package://robotiq_85_gripper_description/meshes/base_grippe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 scale=0.001 0.001 0.001
- link robotiq_adapter_link: geometry collision mesh filename=package://robotiq_140_gripper_description/meshes/hros_robot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 scale=0.001 0.001 0.001; visual mesh filename=package://robotiq_140_gripper_description/meshes/hros_robot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 scale=0.001 0.001 0.001
Joints:
- removed joint left_finger_joint
- removed joint right_finger_joint
- removed joint right_outer_knuckle_joint
- added joint joint_finger: type revolute, parent robotiq_arg2f_base, child right_outer_knuckle, origin xyz=0.0306 0 0.05490 rpy=0 0 3.1416, axis 0 1 0, limit lower=0 upper=0.78 effort=1000 velocity=2.0
- added joint left_outer_finger_joint: type fixed, parent left_outer_knuckle, child left_outer_finger, origin xyz=-0.03156 0 -0.003758 rpy=0 0 0
- added joint right_outer_finger_joint: type fixed, parent right_outer_knuckle, child right_outer_finger, origin xyz=-0.03156 0 -0.003758 rpy=0 0 0
- joint base_adapter_to_base_robotiq_joint: child robotiq_85_base_link -> robotiq_arg2f_base
- joint left_inner_finger_joint: axis 0 1 0 -> 0 -1 0; child robotiq_85_left_inner_finger_link -> left_inner_finger; limit lower=0 upper=0.8757 effort=1000 velocity=2.0 -> lower=0 upper=0.775 effort=1000 velocity=2.0; mimic (none) -> joint=joint_finger multiplier=1 offset=0; origin xyz=-0.0127 0 0.06142 rpy=0 0 0 -> xyz=-0.005625 0 0.04718 rpy=0 0.0 0; parent robotiq_85_base_link -> left_outer_finger
- joint left_inner_knuckle_joint: child robotiq_85_left_inner_knuckle_link -> left_inner_knuckle; limit lower=0.0 upper=0.794 effort=1000 velocity=2.0 -> lower=0 upper=0.8757 effort=1000 velocity=2.0; mimic (none) -> joint=joint_finger multiplier=1 offset=0; origin xyz=-0.0306 0 0.05490 rpy=0 0 0 -> xyz=-0.0127 0 0.06142 rpy=0 0 0; parent robotiq_85_base_link -> robotiq_arg2f_base
- joint left_outer_knuckle_joint: axis 0 -1 0 -> 0 1 0; child robotiq_85_left_outer_knuckle_link -> left_outer_knuckle; limit lower=0 upper=0.8757 effort=1000 velocity=2.0 -> lower=0.0 upper=0.78 effort=1000 velocity=2.0; mimic (none) -> joint=joint_finger multiplier=1 offset=0; origin xyz=-0.03156 0 -0.003758 rpy=0 0 0 -> xyz=-0.0306 0 0.05490 rpy=0 0 0; parent robotiq_85_left_inner_knuckle_link -> robotiq_arg2f_base
- joint right_inner_finger_joint: axis 0 1 0 -> 0 -1 0; child robotiq_85_right_inner_finger_link -> right_inner_finger; limit lower=0 upper=0.8757 effort=1000 velocity=2.0 -> lower=0 upper=0.775 effort=1000 velocity=2.0; mimic (none) -> joint=joint_finger multiplier=1 offset=0; origin xyz=0.0127 0 0.06142 rpy=0 0 3.1416 -> xyz=-0.005625 0 0.04718 rpy=0 0 0; parent robotiq_85_base_link -> right_outer_finger
- joint right_inner_knuckle_joint: child robotiq_85_right_inner_knuckle_link -> right_inner_knuckle; limit lower=0 upper=0.794 effort=1000 velocity=2.0 -> lower=0 upper=0.8757 effort=1000 velocity=2.0; mimic (none) -> joint=joint_finger multiplier=1 offset=0; origin xyz=0.0306 0 0.05490 rpy=0 0 3.1416 -> xyz=0.0127 0 0.06142 rpy=0 0 3.1416; parent robotiq_85_base_link -> robotiq_arg2f_base

File: robotiq_85_gripper_description/urdf/robotiq_85.urdf.xacro (robot description, xacro)
@@ -2,5 +2,5 @@
 <robot xmlns:xacro="http://ros.org/wiki/xacro">
   <xacro:macro name="robotiq_85"  params="prefix">
-    <link name="robotiq_85_base_link">
+    <link name="robotiq_arg2f_base">
       <inertial>
         <origin xyz="8.625E-08 -4.6583E-06 0.03145" rpy="0 0 0" />
@@ -24,9 +24,9 @@
       </collision>
     </link>
-    <gazebo reference="robotiq_85_base_link">
-      <material>Gazebo/Black</material>
-      <selfCollide>True</selfCollide>
-    </gazebo>
-    <link name="robotiq_85_left_inner_knuckle_link">
+    <gazebo reference="robotiq_arg2f_base">
+      <material>Gazebo/Black</material>
+      <selfCollide>True</selfCollide>
+    </gazebo>
+    <link name="left_outer_knuckle">
       <inertial>
         <origin xyz="8.625E-08 -4.6583E-06 0.03145" rpy="0 0 0" />
@@ -50,9 +50,9 @@
       </collision>
     </link>
-    <gazebo reference="robotiq_85_left_inner_knuckle_link">
+    <gazebo reference="left_outer_knuckle">
       <material>Gazebo/Grey</material>
       <selfCollide>True</selfCollide>
     </gazebo>
-    <link name="robotiq_85_right_inner_knuckle_link">
+    <link name="right_outer_knuckle">
       <inertial>
         <origin xyz="8.625E-08 -4.6583E-06 0.03145" rpy="0 0 0" />
@@ -76,9 +76,9 @@
       </collision>
     </link>
-    <gazebo reference="robotiq_85_right_inner_knuckle_link">
+    <gazebo reference="right_outer_knuckle">
       <material>Gazebo/Grey</material>
       <selfCollide>True</selfCollide>
     </gazebo>
-    <link name="robotiq_85_left_outer_knuckle_link">
+    <link name="left_outer_finger">
       <inertial>
         <origin xyz="8.625E-08 -4.6583E-06 0.03145" rpy="0 0 0" />
@@ -102,9 +102,9 @@
       </collision>
     </link>
-    <gazebo reference="robotiq_85_left_outer_knuckle_link">
-      <material>Gazebo/Black</material>
-      <selfCollide>True</selfCollide>
-    </gazebo>
-    <link name="robotiq_85_right_outer_knuckle_link">
+    <gazebo reference="left_outer_finger">
+      <material>Gazebo/Black</material>
+      <selfCollide>True</selfCollide>
+    </gazebo>
+    <link name="right_outer_finger">
       <inertial>
         <origin xyz="8.625E-08 -4.6583E-06 0.03145" rpy="0 0 0" />
@@ -128,9 +128,9 @@
       </collision>
     </link>
-    <gazebo reference="robotiq_85_right_outer_knuckle_link">
-      <material>Gazebo/Black</material>
-      <selfCollide>True</selfCollide>
-    </gazebo>
-    <link name="robotiq_85_left_inner_finger_link">
+    <gazebo reference="right_outer_finger">
+      <material>Gazebo/Black</material>
+      <selfCollide>True</selfCollide>
+    </gazebo>
+    <link name="left_inner_knuckle">
       <inertial>
         <origin xyz="8.625E-08 -4.6583E-06 0.03145" rpy="0 0 0" />
@@ -154,9 +154,9 @@
       </collision>
     </link>
-    <gazebo reference="robotiq_85_left_inner_finger_link">
-      <material>Gazebo/Black</material>
-      <selfCollide>True</selfCollide>
-    </gazebo>
-    <link name="robotiq_85_right_inner_finger_link">
+    <gazebo reference="left_inner_knuckle">
+      <material>Gazebo/Black</material>
+      <selfCollide>True</selfCollide>
+    </gazebo>
+    <link name="right_inner_knuckle">
       <inertial>
         <origin xyz="8.625E-08 -4.6583E-06 0.03145" rpy="0 0 0" />
@@ -180,9 +180,9 @@
       </collision>
     </link>
-    <gazebo reference="robotiq_85_right_inner_finger_link">
-      <material>Gazebo/Black</material>
-      <selfCollide>True</selfCollide>
-    </gazebo>
-    <link name="robotiq_85_left_finger_link">
+    <gazebo reference="right_inner_knuckle">
+      <material>Gazebo/Black</material>
+      <selfCollide>True</selfCollide>
+    </gazebo>
+    <link name="left_inner_finger">
       <inertial>
         <origin xyz="8.625E-08 -4.6583E-06 0.03145" rpy="0 0 0" />
@@ -206,9 +206,9 @@
       </collision>
     </link>
-    <gazebo reference="robotiq_85_left_finger_link">
-      <material>Gazebo/Black</material>
-      <selfCollide>True</selfCollide>
-    </gazebo>
-    <link name="robotiq_85_right_finger_link">
+    <gazebo reference="left_inner_finger">
+      <material>Gazebo/Black</material>
+      <selfCollide>True</selfCollide>
+    </gazebo>
+    <link name="right_inner_finger">
       <inertial>
         <origin xyz="8.625E-08 -4.6583E-06 0.03145" rpy="0 0 0" />
@@ -232,79 +232,74 @@
       </collision>
     </link>
-    <gazebo reference="robotiq_85_right_finger_link">
-      <material>Gazebo/Black</material>
-      <selfCollide>True</selfCollide>
-    </gazebo>
+    <gazebo reference="right_inner_finger">
+      <material>Gazebo/Black</material>
+      <selfCollide>True</selfCollide>
+    </gazebo>
+    <joint name="left_outer_knuckle_joint" type="revolute">
+      <origin xyz="-0.0306 0 0.05490" rpy="0 0 0" />
+      <parent link="robotiq_arg2f_base" />
+      <child link="left_outer_knuckle" />
+      <axis xyz="0 1 0" />
+      <limit lower="0.0" upper="0.78" velocity="2.0" effort="1000" />
+      <mimic joint="joint_finger" multiplier="1" offset="0"/>
+    </joint>
+    <joint name="joint_finger" type="revolute">
+      <origin xyz="0.0306 0 0.05490" rpy="0 0 3.1416" />
+      <parent link="robotiq_arg2f_base" />
+      <child link="right_outer_knuckle" />
+      <axis xyz="0 1 0" />
+      <limit lower="0" upper="0.78" velocity="2.0" effort="1000" />
+    </joint>
     <joint name="left_inner_knuckle_joint" type="revolute">
-      <origin xyz="-0.0306 0 0.05490" rpy="0 0 0" />
-      <parent link="robotiq_85_base_link" />
-      <child link="robotiq_85_left_inner_knuckle_link" />
-      <axis xyz="0 1 0" />
-      <limit lower="0.0" upper="0.794" velocity="2.0" effort="1000" />
-    </joint>
-    <joint name="right_inner_knuckle_joint" type="revolute">
-      <origin xyz="0.0306 0 0.05490" rpy="0 0 3.1416" />
-      <parent link="robotiq_85_base_link" />
-      <child link="robotiq_85_right_inner_knuckle_link" />
-      <axis xyz="0 1 0" />
-      <limit lower="0" upper="0.794" velocity="2.0" effort="1000" />
-    </joint>
-    <joint name="left_outer_knuckle_joint" type="revolute">
-      <origin xyz="-0.03156 0 -0.003758" rpy="0 0 0" />
-      <parent link="robotiq_85_left_inner_knuckle_link" />
-      <child link="robotiq_85_left_outer_knuckle_link" />
-      <axis xyz="0 -1 0" />
-      <limit lower="0" upper="0.8757" velocity="2.0" effort="1000" />
-    </joint>
-    <joint name="right_outer_knuckle_joint" type="revolute">
-      <origin xyz="-0.03156 0 -0.003758" rpy="0 0 0" />
-      <parent link="robotiq_85_right_inner_knuckle_link" />
-      <child link="robotiq_85_right_outer_knuckle_link" />
-      <axis xyz="0 -1 0" />
-      <limit lower="0" upper="0.8757" velocity="2.0" effort="1000" />
-    </joint>
-    <joint name="left_inner_finger_joint" type="revolute">
       <origin xyz="-0.0127 0 0.06142" rpy="0 0 0" />
-      <parent link="robotiq_85_base_link" />
-      <child link="robotiq_85_left_inner_finger_link" />
+      <parent link="robotiq_arg2f_base" />
+      <child link="left_inner_knuckle" />
       <axis xyz="0 1 0" />
       <limit lower="0" upper="0.8757" velocity="2.0" effort="1000" />
-    </joint>
-    <joint name="right_inner_finger_joint" type="revolute">
+      <mimic joint="joint_finger" multiplier="1" offset="0"/>
+    </joint>
+    <joint name="right_inner_knuckle_joint" type="revolute">
       <origin xyz="0.0127 0 0.06142" rpy="0 0 3.1416" />
-      <parent link="robotiq_85_base_link" />
-      <child link="robotiq_85_right_inner_finger_link" />
+      <parent link="robotiq_arg2f_base" />
+      <child link="right_inner_knuckle" />
       <axis xyz="0 1 0" />
       <limit lower="0" upper="0.8757" velocity="2.0" effort="1000" />
-    </joint>
-    <joint name="left_finger_joint" type="revolute">
+      <mimic joint="joint_finger" multiplier="1" offset="0"/>
+    </joint>
+    <joint name="left_inner_finger_joint" type="revolute">
       <origin xyz="-0.005625 0 0.04718" rpy="0 0.0 0" />
-      <parent link="robotiq_85_left_outer_knuckle_link" />
-      <child link="robotiq_85_left_finger_link" />
+      <parent link="left_outer_finger" />
+      <child link="left_inner_finger" />
       <axis xyz="0 -1 0" />
-      <limit lower="-0.1" upper="0.8757" velocity="2.0" effort="1000" />
-    </joint>
-    <joint name="right_finger_joint" type="revolute">
+      <limit lower="0" upper="0.775" velocity="2.0" effort="1000" />
+      <mimic joint="joint_finger" multiplier="1" offset="0"/>
+    </joint>
+    <joint name="right_inner_finger_joint" type="revolute">
       <origin xyz="-0.005625 0 0.04718" rpy="0 0 0" />
-      <parent link="robotiq_85_right_outer_knuckle_link" />
-      <child link="robotiq_85_right_finger_link" />
-      <axis xyz="0 -1 0"/>
-      <limit lower="-0.1" upper="0.8757" velocity="2.0" effort="1000" />
+      <parent link="right_outer_finger" />
+      <child link="right_inner_finger" />
+      <axis xyz="0 -1 0" />
+      <limit lower="0" upper="0.775" velocity="2.0" effort="1000" />
+      <mimic joint="joint_finger" multiplier="1" offset="0"/>
+    </joint>
+    <joint name="left_outer_finger_joint" type="fixed">
+      <origin xyz="-0.03156 0 -0.003758" rpy="0 0 0" />
+      <parent link="left_outer_knuckle" />
+      <child link="left_outer_finger" />
+    </joint>
+    <joint name="right_outer_finger_joint" type="fixed">
+      <origin xyz="-0.03156 0 -0.003758" rpy="0 0 0" />
+      <parent link="right_outer_knuckle" />
+      <child link="right_outer_finger" />
     </joint>
     <gazebo>
-      <plugin filename="librobotiq_angular_gripper_gazebo_plugin.so" name="robotiq_85_gripper">
-        <left_joint>left_inner_knuckle_joint</left_joint>
-        <left_joint>left_inner_finger_joint</left_joint>
-        <right_joint>right_inner_knuckle_joint</right_joint>
-        <right_joint>right_inner_finger_joint</right_joint>
-      </plugin>
       <joint name="left_finger_joint2" type="revolute">
         <pose frame="">0.017901 0 0.00651469 0 0 0</pose>
-        <parent>${prefix}::robotiq_85_left_inner_finger_link</parent>
-        <child>${prefix}::robotiq_85_left_finger_link</child>
+        <parent>${prefix}::left_inner_knuckle</parent>
+        <child>${prefix}::left_inner_finger</child>
         <axis>
           <xyz>0 -1 0</xyz>
           <limit>
-            <lower>-0.1</lower>
+            <lower>-0.8</lower>
             <upper>0.8</upper>
             <velocity>2.0</velocity>
@@ -315,10 +310,10 @@
       <joint name="right_finger_joint2" type="revolute">
         <pose frame="">0.017901 0 0.00651469 0 0 0</pose>
-        <parent>${prefix}::robotiq_85_right_inner_finger_link</parent>
-        <child>${prefix}::robotiq_85_right_finger_link</child>
+        <parent>${prefix}::right_inner_knuckle</parent>
+        <child>${prefix}::right_inner_finger</child>
         <axis>
           <xyz>0 1 0</xyz>
           <limit>
-            <lower>-0.1</lower>
+            <lower>-0.8</lower>
             <upper>0.8</upper>
             <velocity>2.0</velocity>
@@ -327,4 +322,10 @@
         </axis>
       </joint>
+      <plugin filename="librobotiq_angular_gripper_gazebo_plugin.so" name="robotiq_85_gripper">
+        <left_joint>left_inner_knuckle_joint</left_joint>
+        <left_joint>left_outer_knuckle_joint</left_joint>
+        <right_joint>right_inner_knuckle_joint</right_joint>
+        <right_joint>joint_finger</right_joint>
+      </plugin>
     </gazebo>
   </xacro:macro>
