Commit message: update URDFs robotiq 85

File: robotiq_85_gripper_description/urdf/robotiq_85_hros_support.urdf.xacro (robot description, xacro)
@@ -1,362 +1,53 @@
 <?xml version="1.0"?>
-<robot xmlns:xacro="http://ros.org/wiki/xacro">
-  <xacro:macro name="robotiq_85"  params="prefix">
-    <link name="robotiq_adapter_link">
-      <inertial>
-        <origin xyz="8.625E-08 -4.6583E-06 0.03145" rpy="0 0 0" />
-        <mass value="0.22652" />
-        <inertia ixx="0.00020005" ixy="0" ixz="0" iyy="0.00017832" iyz="0" izz="0.00013478" />
-      </inertial>
-      <visual>
-        <origin xyz="0 0 0" rpy="0 0 0" />
-        <geometry>
-          <mesh filename="package://robotiq_85_gripper_description/meshes/hros_robotiq_adapter.dae" scale="0.001 0.001 0.001"/>
-        </geometry>
-        <material name="Gazebo/Black">
-          <color rgba="0.1 0.1 0.1 1" />
-        </material>
-      </visual>
-      <collision>
-        <origin xyz="0 0 0" rpy="0 0 0" />
-        <geometry>
-          <mesh filename="package://robotiq_85_gripper_description/meshes/hros_robotiq_adapter.dae" scale="0.001 0.001 0.001"/>
-        </geometry>
-      </collision>
-    </link>
-    <gazebo reference="robotiq_adapter_link">
-      <material>Gazebo/Black</material>
-      <selfCollide>True</selfCollide>
-    </gazebo>
-    <link name="robotiq_85_base_link">
-      <inertial>
-        <origin xyz="8.625E-08 -4.6583E-06 0.03145" rpy="0 0 0" />
-        <mass value="0.22652" />
-        <inertia ixx="0.00020005" ixy="0" ixz="0" iyy="0.00017832" iyz="0" izz="0.00013478" />
-      </inertial>
-      <visual>
-        <origin xyz="0 0 0" rpy="0 0 0" />
-        <geometry>
-          <mesh filename="package://robotiq_85_gripper_description/meshes/base_gripper.dae" scale="0.001 0.001 0.001"/>
-        </geometry>
-        <material name="Gazebo/Black">
-          <color rgba="0.1 0.1 0.1 1" />
-        </material>
-      </visual>
-      <collision>
-        <origin xyz="0 0 0" rpy="0 0 0" />
-        <geometry>
-          <mesh filename="package://robotiq_85_gripper_description/meshes/base_gripper.dae" scale="0.001 0.001 0.001"/>
-        </geometry>
-      </collision>
-    </link>
-    <gazebo reference="robotiq_85_base_link">
-      <material>Gazebo/Black</material>
-      <selfCollide>True</selfCollide>
-    </gazebo>
-    <link name="robotiq_85_left_inner_knuckle_link">
-      <inertial>
-        <origin xyz="8.625E-08 -4.6583E-06 0.03145" rpy="0 0 0" />
-        <mass value="0.22652" />
-        <inertia ixx="0.00020005" ixy="0" ixz="0" iyy="0.00017832" iyz="0" izz="0.00013478" />
-      </inertial>
-      <visual>
-        <origin xyz="0 0 0" rpy="0 0 0" />
-        <geometry>
-          <mesh filename="package://robotiq_85_gripper_description/meshes/2-F-85_1_l.dae" scale="0.001 0.001 0.001"/>
-        </geometry>
-        <material name="Gazebo/Grey">
-          <color rgba="0.1 0.1 0.1 1" />
-        </material>
-      </visual>
-      <collision>
-        <origin xyz="0 0 0" rpy="0 0 0" />
-        <geometry>
-          <mesh filename="package://robotiq_85_gripper_description/meshes/2-F-85_1_l.dae" scale="0.001 0.001 0.001"/>
-        </geometry>
-      </collision>
-    </link>
-    <gazebo reference="robotiq_85_left_inner_knuckle_link">
-      <material>Gazebo/Grey</material>
-      <selfCollide>True</selfCollide>
-    </gazebo>
-    <link name="robotiq_85_right_inner_knuckle_link">
-      <inertial>
-        <origin xyz="8.625E-08 -4.6583E-06 0.03145" rpy="0 0 0" />
-        <mass value="0.22652" />
-        <inertia ixx="0.00020005" ixy="0" ixz="0" iyy="0.00017832" iyz="0" izz="0.00013478" />
-      </inertial>
-      <visual>
-        <origin xyz="0 0 0" rpy="0 0 0" />
-        <geometry>
-          <mesh filename="package://robotiq_85_gripper_description/meshes/2-F-85_1_r.dae" scale="0.001 0.001 0.001"/>
-        </geometry>
-        <material name="Gazebo/Grey">
-          <color rgba="0.1 0.1 0.1 1" />
-        </material>
-      </visual>
-      <collision>
-        <origin xyz="0 0 0" rpy="0 0 0" />
-        <geometry>
-          <mesh filename="package://robotiq_85_gripper_description/meshes/2-F-85_1_r.dae" scale="0.001 0.001 0.001"/>
-        </geometry>
-      </collision>
-    </link>
-    <gazebo reference="robotiq_85_right_inner_knuckle_link">
-      <material>Gazebo/Grey</material>
-      <selfCollide>True</selfCollide>
-    </gazebo>
-    <link name="robotiq_85_left_outer_knuckle_link">
-      <inertial>
-        <origin xyz="8.625E-08 -4.6583E-06 0.03145" rpy="0 0 0" />
-        <mass value="0.22652" />
-        <inertia ixx="0.00020005" ixy="0" ixz="0" iyy="0.00017832" iyz="0" izz="0.00013478" />
-      </inertial>
-      <visual>
-        <origin xyz="0 0 0" rpy="0 0 0" />
-        <geometry>
-          <mesh filename="package://robotiq_85_gripper_description/meshes/2-F-85_3_l.dae" scale="0.001 0.001 0.001"/>
-        </geometry>
-        <material name="Gazebo/Black">
-          <color rgba="0.1 0.1 0.1 1" />
-        </material>
-      </visual>
-      <collision>
-        <origin xyz="0 0 0" rpy="0 0 0" />
-        <geometry>
-          <mesh filename="package://robotiq_85_gripper_description/meshes/2-F-85_3_l.dae" scale="0.001 0.001 0.001"/>
-        </geometry>
-      </collision>
-    </link>
-    <gazebo reference="robotiq_85_left_outer_knuckle_link">
-      <material>Gazebo/Black</material>
-      <selfCollide>True</selfCollide>
-    </gazebo>
-    <link name="robotiq_85_right_outer_knuckle_link">
-      <inertial>
-        <origin xyz="8.625E-08 -4.6583E-06 0.03145" rpy="0 0 0" />
-        <mass value="0.22652" />
-        <inertia ixx="0.00020005" ixy="0" ixz="0" iyy="0.00017832" iyz="0" izz="0.00013478" />
-      </inertial>
-      <visual>
-        <origin xyz="0 0 0" rpy="0 0 0" />
-        <geometry>
-          <mesh filename="package://robotiq_85_gripper_description/meshes/2-F-85_3_r.dae" scale="0.001 0.001 0.001"/>
-        </geometry>
-        <material name="Gazebo/Black">
-          <color rgba="0.1 0.1 0.1 1" />
-        </material>
-      </visual>
-      <collision>
-        <origin xyz="0 0 0" rpy="0 0 0" />
-        <geometry>
-          <mesh filename="package://robotiq_85_gripper_description/meshes/2-F-85_3_r.dae" scale="0.001 0.001 0.001"/>
-        </geometry>
-      </collision>
-    </link>
-    <gazebo reference="robotiq_85_right_outer_knuckle_link">
-      <material>Gazebo/Black</material>
-      <selfCollide>True</selfCollide>
-    </gazebo>
-    <link name="robotiq_85_left_inner_finger_link">
-      <inertial>
-        <origin xyz="8.625E-08 -4.6583E-06 0.03145" rpy="0 0 0" />
-        <mass value="0.22652" />
-        <inertia ixx="0.00020005" ixy="0" ixz="0" iyy="0.00017832" iyz="0" izz="0.00013478" />
-      </inertial>
-      <visual>
-        <origin xyz="0 0 0" rpy="0 0 0" />
-        <geometry>
-          <mesh filename="package://robotiq_85_gripper_description/meshes/2-F-85_2_l.dae" scale="0.001 0.001 0.001"/>
-        </geometry>
-        <material name="Gazebo/Black">
-          <color rgba="0.1 0.1 0.1 1" />
-        </material>
-      </visual>
-      <collision>
-        <origin xyz="0 0 0" rpy="0 0 0" />
-        <geometry>
-          <mesh filename="package://robotiq_85_gripper_description/meshes/2-F-85_2_l.dae" scale="0.001 0.001 0.001"/>
-        </geometry>
-      </collision>
-    </link>
-    <gazebo reference="robotiq_85_left_inner_finger_link">
-      <material>Gazebo/Black</material>
-      <selfCollide>True</selfCollide>
-    </gazebo>
-    <link name="robotiq_85_right_inner_finger_link">
-      <inertial>
-        <origin xyz="8.625E-08 -4.6583E-06 0.03145" rpy="0 0 0" />
-        <mass value="0.22652" />
-        <inertia ixx="0.00020005" ixy="0" ixz="0" iyy="0.00017832" iyz="0" izz="0.00013478" />
-      </inertial>
-      <visual>
-        <origin xyz="0 0 0" rpy="0 0 0" />
-        <geometry>
-          <mesh filename="package://robotiq_85_gripper_description/meshes/2-F-85_2_r.dae" scale="0.001 0.001 0.001"/>
-        </geometry>
-        <material name="Gazebo/Black">
-          <color rgba="0.1 0.1 0.1 1" />
-        </material>
-      </visual>
-      <collision>
-        <origin xyz="0 0 0" rpy="0 0 0" />
-        <geometry>
-          <mesh filename="package://robotiq_85_gripper_description/meshes/2-F-85_2_r.dae" scale="0.001 0.001 0.001"/>
-        </geometry>
-      </collision>
-    </link>
-    <gazebo reference="robotiq_85_right_inner_finger_link">
-      <material>Gazebo/Black</material>
-      <selfCollide>True</selfCollide>
-    </gazebo>
-    <link name="robotiq_85_left_finger_link">
-      <inertial>
-        <origin xyz="8.625E-08 -4.6583E-06 0.03145" rpy="0 0 0" />
-        <mass value="0.22652" />
-        <inertia ixx="0.00020005" ixy="0" ixz="0" iyy="0.00017832" iyz="0" izz="0.00013478" />
-      </inertial>
-      <visual>
-        <origin xyz="0 0 0" rpy="0 0 0" />
-        <geometry>
-          <mesh filename="package://robotiq_85_gripper_description/meshes/2-F-85_4_l.dae" scale="0.001 0.001 0.001"/>
-        </geometry>
-        <material name="Gazebo/Black">
-          <color rgba="0.1 0.1 0.1 1" />
-        </material>
-      </visual>
-      <collision>
-        <origin xyz="0 0 0" rpy="0 0 0" />
-        <geometry>
-          <mesh filename="package://robotiq_85_gripper_description/meshes/2-F-85_4_l.dae" scale="0.001 0.001 0.001"/>
-        </geometry>
-      </collision>
-    </link>
-    <gazebo reference="robotiq_85_left_finger_link">
-      <material>Gazebo/Black</material>
-      <selfCollide>True</selfCollide>
-    </gazebo>
-    <link name="robotiq_85_right_finger_link">
-      <inertial>
-        <origin xyz="8.625E-08 -4.6583E-06 0.03145" rpy="0 0 0" />
-        <mass value="0.22652" />
-        <inertia ixx="0.00020005" ixy="0" ixz="0" iyy="0.00017832" iyz="0" izz="0.00013478" />
-      </inertial>
-      <visual>
-        <origin xyz="0 0 0" rpy="0 0 0" />
-        <geometry>
-          <mesh filename="package://robotiq_85_gripper_description/meshes/2-F-85_4_r.dae" scale="0.001 0.001 0.001"/>
-        </geometry>
-        <material name="Gazebo/Black">
-          <color rgba="0.1 0.1 0.1 1" />
-        </material>
-      </visual>
-      <collision>
-        <origin xyz="0 0 0" rpy="0 0 0" />
-        <geometry>
-          <mesh filename="package://robotiq_85_gripper_description/meshes/2-F-85_4_r.dae" scale="0.001 0.001 0.001"/>
-        </geometry>
-      </collision>
-    </link>
-    <gazebo reference="robotiq_85_right_finger_link">
-      <material>Gazebo/Black</material>
-      <selfCollide>True</selfCollide>
-    </gazebo>
-    <joint name="base_adapter_to_base_robotiq_joint" type="fixed">
-      <origin rpy="0 0 0" xyz=" 0 0 0.03653"/>
-      <parent link="robotiq_adapter_link" />
-      <child link="robotiq_85_base_link"/>
-    </joint>
-    <joint name="left_inner_knuckle_joint" type="revolute">
-      <origin xyz="-0.0306 0 0.05490" rpy="0 0 0" />
-      <parent link="robotiq_85_base_link" />
-      <child link="robotiq_85_left_inner_knuckle_link" />
-      <axis xyz="0 1 0" />
-      <limit lower="0.0" upper="0.794" velocity="2.0" effort="1000" />
-    </joint>
-    <joint name="right_inner_knuckle_joint" type="revolute">
-      <origin xyz="0.0306 0 0.05490" rpy="0 0 3.1416" />
-      <parent link="robotiq_85_base_link" />
-      <child link="robotiq_85_right_inner_knuckle_link" />
-      <axis xyz="0 1 0" />
-      <limit lower="0" upper="0.794" velocity="2.0" effort="1000" />
-    </joint>
-    <joint name="left_outer_knuckle_joint" type="revolute">
-      <origin xyz="-0.03156 0 -0.003758" rpy="0 0 0" />
-      <parent link="robotiq_85_left_inner_knuckle_link" />
-      <child link="robotiq_85_left_outer_knuckle_link" />
-      <axis xyz="0 -1 0" />
-      <limit lower="0" upper="0.8757" velocity="2.0" effort="1000" />
-    </joint>
-    <joint name="right_outer_knuckle_joint" type="revolute">
-      <origin xyz="-0.03156 0 -0.003758" rpy="0 0 0" />
-      <parent link="robotiq_85_right_inner_knuckle_link" />
-      <child link="robotiq_85_right_outer_knuckle_link" />
-      <axis xyz="0 -1 0" />
-      <limit lower="0" upper="0.8757" velocity="2.0" effort="1000" />
-    </joint>
-    <joint name="left_inner_finger_joint" type="revolute">
-      <origin xyz="-0.0127 0 0.06142" rpy="0 0 0" />
-      <parent link="robotiq_85_base_link" />
-      <child link="robotiq_85_left_inner_finger_link" />
-      <axis xyz="0 1 0" />
-      <limit lower="0" upper="0.8757" velocity="2.0" effort="1000" />
-    </joint>
-    <joint name="right_inner_finger_joint" type="revolute">
-      <origin xyz="0.0127 0 0.06142" rpy="0 0 3.1416" />
-      <parent link="robotiq_85_base_link" />
-      <child link="robotiq_85_right_inner_finger_link" />
-      <axis xyz="0 1 0" />
-      <limit lower="0" upper="0.8757" velocity="2.0" effort="1000" />
-    </joint>
-    <joint name="left_finger_joint" type="revolute">
-      <origin xyz="-0.005625 0 0.04718" rpy="0 0.0 0" />
-      <parent link="robotiq_85_left_outer_knuckle_link" />
-      <child link="robotiq_85_left_finger_link" />
-      <axis xyz="0 -1 0" />
-      <limit lower="-0.1" upper="0.8757" velocity="2.0" effort="1000" />
-    </joint>
-    <joint name="right_finger_joint" type="revolute">
-      <origin xyz="-0.005625 0 0.04718" rpy="0 0 0" />
-      <parent link="robotiq_85_right_outer_knuckle_link" />
-      <child link="robotiq_85_right_finger_link" />
-      <axis xyz="0 -1 0"/>
-      <limit lower="-0.1" upper="0.8757" velocity="2.0" effort="1000" />
-    </joint>
-    <gazebo>
-      <plugin filename="librobotiq_gripper_gazebo_plugin.so" name="hros_actuation_gripper_000000000004">
-        <left_joint>left_inner_knuckle_joint</left_joint>
-        <left_joint>left_inner_finger_joint</left_joint>
-        <right_joint>right_inner_knuckle_joint</right_joint>
-        <right_joint>right_inner_finger_joint</right_joint>
-      </plugin>
-      <joint name="left_finger_joint2" type="revolute">
-        <pose frame="">0.017901 0 0.00651469 0 0 0</pose>
-        <parent>${prefix}::robotiq_85_left_inner_finger_link</parent>
-        <child>${prefix}::robotiq_85_left_finger_link</child>
-        <axis>
-          <xyz>0 -1 0</xyz>
-          <limit>
-            <lower>-0.1</lower>
-            <upper>0.8</upper>
-            <velocity>2.0</velocity>
-            <effort>1000</effort>
-          </limit>
-        </axis>
-      </joint>
-      <joint name="right_finger_joint2" type="revolute">
-        <pose frame="">0.017901 0 0.00651469 0 0 0</pose>
-        <parent>${prefix}::robotiq_85_right_inner_finger_link</parent>
-        <child>${prefix}::robotiq_85_right_finger_link</child>
-        <axis>
-          <xyz>0 1 0</xyz>
-          <limit>
-            <lower>-0.1</lower>
-            <upper>0.8</upper>
-            <velocity>2.0</velocity>
-            <effort>1000</effort>
-          </limit>
-        </axis>
-      </joint>
-    </gazebo>
-  </xacro:macro>
+<robot xmlns:xacro="http://ros.org/wiki/xacro"
+       name="robotiq_85" >
+  <!-- robotiq hande_gripper -->
+  <xacro:include filename="$(find robotiq_85_gripper_description)/urdf/robotiq_85.urdf.xacro" />
+  <xacro:robotiq_85 prefix="robotiq85"/>
+  <link name="world" />
+  <link name="robotiq_adapter_link">
+    <inertial>
+      <origin xyz="8.625E-08 -4.6583E-06 0.03145" rpy="0 0 0" />
+      <mass value="0.22652" />
+      <inertia ixx="0.00020005" ixy="0" ixz="0" iyy="0.00017832" iyz="0" izz="0.00013478" />
+    </inertial>
+    <visual>
+      <origin xyz="0 0 0" rpy="0 0 1.57" />
+      <geometry>
+        <mesh filename="package://robotiq_140_gripper_description/meshes/hros_robotiq_adapter.dae" scale="0.001 0.001 0.001"/>
+      </geometry>
+      <material name="Gazebo/Black">
+        <color rgba="0.1 0.1 0.1 1" />
+      </material>
+    </visual>
+    <collision>
+      <origin xyz="0 0 0" rpy="0 0 1.57" />
+      <geometry>
+        <mesh filename="package://robotiq_140_gripper_description/meshes/hros_robotiq_adapter.dae" scale="0.001 0.001 0.001"/>
+      </geometry>
+    </collision>
+  </link>
+  <gazebo reference="robotiq_adapter_link">
+    <material>Gazebo/Black</material>
+    <selfCollide>False</selfCollide>
+  </gazebo>
+  <joint name="base_adapter_to_base_robotiq_joint" type="fixed">
+    <origin rpy="0 0 0" xyz=" 0 0 0.03653"/>
+    <parent link="robotiq_adapter_link" />
+    <child link="robotiq_arg2f_base"/>
+  </joint>
+  <joint name="world_to_hande_joint" type="fixed">
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
Commit message: fix robotiq_adapter_link orientation to match real

File: robotiq_85_gripper_description/urdf/robotiq_85.urdf (robot description, URDF)
Before this commit: robot robotiq_85, 11 links, 10 joints
Links:
- link robotiq_adapter_link: geometry collision mesh filename=package://robotiq_85_gripper_description/meshes/hros_roboti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 scale=0.001 0.001 0.001; visual mesh filename=package://robotiq_85_gripper_description/meshes/hros_roboti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 scale=0.001 0.001 0.001

File: robotiq_85_gripper_description/urdf/robotiq_85.urdf.xacro (robot description, xacro)
@@ -9,5 +9,5 @@
       </inertial>
       <visual>
-        <origin xyz="0 0 0" rpy="0 0 1.57" />
+        <origin xyz="0 0 0" rpy="0 0 0" />
         <geometry>
           <mesh filename="package://robotiq_85_gripper_description/meshes/hros_robotiq_adapter.dae" scale="0.001 0.001 0.001"/>
@@ -18,5 +18,5 @@
       </visual>
       <collision>
-        <origin xyz="0 0 0" rpy="0 0 1.57" />
+        <origin xyz="0 0 0" rpy="0 0 0" />
         <geometry>
           <mesh filename="package://robotiq_85_gripper_description/meshes/hros_robotiq_adapter.dae" scale="0.001 0.001 0.001"/>

File: robotiq_85_gripper_description/urdf/robotiq_85_hros_support.urdf.xacro (robot description, xacro)
@@ -1,40 +1,8 @@
 <?xml version="1.0"?>
-<robot xmlns:xacro="http://ros.org/wiki/xacro"
-       name="robotiq_85" >
+<robot xmlns:xacro="http://ros.org/wiki/xacro" name="robotiq_85" >
   <!-- robotiq hande_gripper -->
   <xacro:include filename="$(find robotiq_85_gripper_description)/urdf/robotiq_85.urdf.xacro" />
   <xacro:robotiq_85 prefix="robotiq85"/>
   <link name="world" />
-  <link name="robotiq_adapter_link">
-    <inertial>
-      <origin xyz="8.625E-08 -4.6583E-06 0.03145" rpy="0 0 0" />
-      <mass value="0.22652" />
-      <inertia ixx="0.00020005" ixy="0" ixz="0" iyy="0.00017832" iyz="0" izz="0.00013478" />
-    </inertial>
-    <visual>
-      <origin xyz="0 0 0" rpy="0 0 1.57" />
-      <geometry>
-        <mesh filename="package://robotiq_140_gripper_description/meshes/hros_robotiq_adapter.dae" scale="0.001 0.001 0.001"/>
-      </geometry>
-      <material name="Gazebo/Black">
-        <color rgba="0.1 0.1 0.1 1" />
-      </material>
-    </visual>
-    <collision>
-      <origin xyz="0 0 0" rpy="0 0 1.57" />
-      <geometry>
-        <mesh filename="package://robotiq_140_gripper_description/meshes/hros_robotiq_adapter.dae" scale="0.001 0.001 0.001"/>
-      </geometry>
-    </collision>
-  </link>
-  <gazebo reference="robotiq_adapter_link">
-    <material>Gazebo/Black</material>
-    <selfCollide>False</selfCollide>
-  </gazebo>
-  <joint name="base_adapter_to_base_robotiq_joint" type="fixed">
-    <origin rpy="0 0 0" xyz=" 0 0 0.03653"/>
-    <parent link="robotiq_adapter_link" />
-    <child link="robotiq_arg2f_base"/>
-  </joint>
   <joint name="world_to_hande_joint" type="fixed">
     <origin rpy="0 0 0" xyz="0 0 0.5"/>

File: robotiq_hande_gripper_description/urdf/robotiq_hande.urdf.xacro (robot description, xacro)
@@ -9,5 +9,5 @@
       </inertial>
       <visual>
-        <origin xyz="0 0 0" rpy="0 0 1.57" />
+        <origin xyz="0 0 0" rpy="0 0 0" />
         <geometry>
           <mesh filename="package://robotiq_hande_gripper_description/meshes/hros_robotiq_adapter.dae" scale="0.001 0.001 0.001"/>
@@ -18,5 +18,5 @@
       </visual>
       <collision>
-        <origin xyz="0 0 0" rpy="0 0 1.57" />
+        <origin xyz="0 0 0" rpy="0 0 0" />
         <geometry>
           <mesh filename="package://robotiq_hande_gripper_description/meshes/hros_robotiq_adapter.dae" scale="0.001 0.001 0.001"/>
