Commit message: update dae files

File: robotiq_85_gripper_description/urdf/robotiq_85.urdf (robot description, URDF)
Before this commit: robot robotiq_85, 11 links, 10 joints
Links:
- removed link robotiq_adapter_link
- removed link robotiq_arg2f_base
- added link robotiq_arg2f_base_link, mass 0.22652; collision mesh filename=package://robotiq_85_gripper_description/meshes/base_grippe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 scale=0.001 0.001 0.001; visual mesh filename=package://robotiq_85_gripper_description/meshes/base_grippe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 scale=0.001 0.001 0.001
Joints:
- removed joint base_adapter_to_base_robotiq_joint
- removed joint left_inner_finger_joint
- removed joint left_inner_knuckle_joint
- removed joint left_outer_finger_joint
- removed joint left_outer_knuckle_joint
- removed joint right_inner_finger_joint
- removed joint right_inner_knuckle_joint
- removed joint right_outer_finger_joint
- removed joint world_to_hande_joint
- added joint left_outer_finger_to_inner: type revolute, parent left_outer_finger, child left_inner_finger, origin xyz=0.00678 0 0.04703 rpy=0 0 0, axis 0 1 0, limit lower=0 upper=0.775 effort=1000 velocity=2.0, mimic joint=joint_finger multiplier=1 offset=0
- added joint left_outer_knuckle_to_finger: type fixed, parent left_outer_knuckle, child left_outer_finger, origin xyz=0.03142 0 -0.00453 rpy=0 0 0
- added joint right_outer_finger_to_inner: type revolute, parent right_outer_finger, child right_inner_finger, origin xyz=-0.00678 0 0.04703 rpy=0 0 0, axis 0 -1 0, limit lower=0 upper=0.775 effort=1000 velocity=2.0, mimic joint=joint_finger multiplier=1 offset=0
- added joint right_outer_knuckle_to_finger: type fixed, parent right_outer_knuckle, child right_outer_finger, origin xyz=-0.03142 0 -0.00453 rpy=0 0 0
- added joint robotiq_arg2f_base_link_to_left_inner_knuckle: type revolute, parent robotiq_arg2f_base_link, child left_inner_knuckle, origin xyz=0.0127 0 0.06118 rpy=0 0 0, axis 0 -1 0, limit lower=0 upper=0.8757 effort=1000 velocity=2.0, mimic joint=joint_finger multiplier=1 offset=0
- added joint robotiq_arg2f_base_link_to_left_outer_knuckle: type revolute, parent robotiq_arg2f_base_link, child left_outer_knuckle, origin xyz=0.0306 0 0.05466 rpy=0 0 0, axis 0 -1 0, limit lower=0.0 upper=0.78 effort=1000 velocity=2.0, mimic joint=joint_finger multiplier=1 offset=0
- added joint robotiq_arg2f_base_link_to_right_inner_knuckle: type revolute, parent robotiq_arg2f_base_link, child right_inner_knuckle, origin xyz=-0.0127 0 0.06118 rpy=0 0 0, axis 0 1 0, limit lower=0 upper=0.8757 effort=1000 velocity=2.0, mimic joint=joint_finger multiplier=1 offset=0
- added joint world_to_robotiq_arg2f_base: type fixed, parent world, child robotiq_arg2f_base_link, origin xyz=0 0 0.5 rpy=0 0 0
- joint joint_finger: origin xyz=0.0306 0 0.05490 rpy=0 0 3.1416 -> xyz=-0.0306 0 0.05466 rpy=0 0 0; parent robotiq_arg2f_base -> robotiq_arg2f_base_link

File: robotiq_85_gripper_description/urdf/robotiq_85.urdf.xacro (robot description, xacro)
@@ -2,36 +2,5 @@
 <robot xmlns:xacro="http://ros.org/wiki/xacro">
   <xacro:macro name="robotiq_85"  params="prefix">
-    <link name="robotiq_adapter_link">
-      <inertial>
-        <origin xyz="8.625E-08 -4.6583E-06 0.03145" rpy="0 0 0" />
-        <mass value="0.22652" />
-        <inertia ixx="0.00020005" ixy="0" ixz="0" iyy="0.00017832" iyz="0" izz="0.00013478" />
-      </inertial>
-      <visual>
-        <origin xyz="0 0 0" rpy="0 0 1.57" />
-        <geometry>
-          <mesh filename="package://robotiq_85_gripper_description/meshes/hros_robotiq_adapter.dae" scale="0.001 0.001 0.001"/>
-        </geometry>
-        <material name="Gazebo/Black">
-          <color rgba="0.0 0.0 0.0 1" />
-        </material>
-      </visual>
-      <collision>
-        <origin xyz="0 0 0" rpy="0 0 1.57" />
-        <geometry>
-          <mesh filename="package://robotiq_85_gripper_description/meshes/hros_robotiq_adapter.dae" scale="0.001 0.001 0.001"/>
-        </geometry>
-      </collision>
-    </link>
-    <gazebo reference="robotiq_adapter_link">
-      <material>Gazebo/Black</material>
-      <selfCollide>False</selfCollide>
-    </gazebo>
-    <joint name="base_adapter_to_base_robotiq_joint" type="fixed">
-      <origin rpy="0 0 0" xyz=" 0 0 0.03653"/>
-      <parent link="robotiq_adapter_link" />
-      <child link="robotiq_arg2f_base"/>
-    </joint>
-    <link name="robotiq_arg2f_base">
+    <link name="robotiq_arg2f_base_link">
       <inertial>
         <origin xyz="8.625E-08 -4.6583E-06 0.03145" rpy="0 0 0" />
@@ -55,5 +24,5 @@
       </collision>
     </link>
-    <gazebo reference="robotiq_arg2f_base">
+    <gazebo reference="robotiq_arg2f_base_link">
       <material>Gazebo/Black</material>
       <selfCollide>True</selfCollide>
@@ -267,30 +236,30 @@
       <selfCollide>True</selfCollide>
     </gazebo>
-    <joint name="left_outer_knuckle_joint" type="revolute">
-      <origin xyz="-0.0306 0 0.05490" rpy="0 0 0" />
-      <parent link="robotiq_arg2f_base" />
+    <joint name="robotiq_arg2f_base_link_to_left_outer_knuckle" type="revolute">
+      <origin xyz="0.0306 0 0.05466" rpy="0 0 0" />
+      <parent link="robotiq_arg2f_base_link" />
       <child link="left_outer_knuckle" />
-      <axis xyz="0 1 0" />
+      <axis xyz="0 -1 0" />
       <limit lower="0.0" upper="0.78" velocity="2.0" effort="1000" />
       <mimic joint="joint_finger" multiplier="1" offset="0"/>
     </joint>
     <joint name="joint_finger" type="revolute">
-      <origin xyz="0.0306 0 0.05490" rpy="0 0 3.1416" />
-      <parent link="robotiq_arg2f_base" />
+      <origin xyz="-0.0306 0 0.05466" rpy="0 0 0" />
+      <parent link="robotiq_arg2f_base_link" />
       <child link="right_outer_knuckle" />
       <axis xyz="0 1 0" />
       <limit lower="0" upper="0.78" velocity="2.0" effort="1000" />
     </joint>
-    <joint name="left_inner_knuckle_joint" type="revolute">
-      <origin xyz="-0.0127 0 0.06142" rpy="0 0 0" />
-      <parent link="robotiq_arg2f_base" />
+    <joint name="robotiq_arg2f_base_link_to_left_inner_knuckle" type="revolute">
+      <origin xyz="0.0127 0 0.06118" rpy="0 0 0" />
+      <parent link="robotiq_arg2f_base_link" />
       <child link="left_inner_knuckle" />
-      <axis xyz="0 1 0" />
+      <axis xyz="0 -1 0" />
       <limit lower="0" upper="0.8757" velocity="2.0" effort="1000" />
       <mimic joint="joint_finger" multiplier="1" offset="0"/>
     </joint>
-    <joint name="right_inner_knuckle_joint" type="revolute">
-      <origin xyz="0.0127 0 0.06142" rpy="0 0 3.1416" />
-      <parent link="robotiq_arg2f_base" />
+    <joint name="robotiq_arg2f_base_link_to_right_inner_knuckle" type="revolute">
+      <origin xyz="-0.0127 0 0.06118" rpy="0 0 0" />
+      <parent link="robotiq_arg2f_base_link" />
       <child link="right_inner_knuckle" />
       <axis xyz="0 1 0" />
@@ -298,14 +267,14 @@
       <mimic joint="joint_finger" multiplier="1" offset="0"/>
     </joint>
-    <joint name="left_inner_finger_joint" type="revolute">
-      <origin xyz="-0.005625 0 0.04718" rpy="0 0.0 0" />
+    <joint name="left_outer_finger_to_inner" type="revolute">
+      <origin xyz="0.00678 0 0.04703" rpy="0 0 0" />
       <parent link="left_outer_finger" />
       <child link="left_inner_finger" />
-      <axis xyz="0 -1 0" />
+      <axis xyz="0 1 0" />
       <limit lower="0" upper="0.775" velocity="2.0" effort="1000" />
       <mimic joint="joint_finger" multiplier="1" offset="0"/>
     </joint>
-    <joint name="right_inner_finger_joint" type="revolute">
-      <origin xyz="-0.005625 0 0.04718" rpy="0 0 0" />
+    <joint name="right_outer_finger_to_inner" type="revolute">
+      <origin xyz="-0.00678 0 0.04703" rpy="0 0 0" />
       <parent link="right_outer_finger" />
       <child link="right_inner_finger" />
@@ -314,19 +283,33 @@
       <mimic joint="joint_finger" multiplier="1" offset="0"/>
     </joint>
-    <joint name="left_outer_finger_joint" type="fixed">
-      <origin xyz="-0.03156 0 -0.003758" rpy="0 0 0" />
+    <joint name="left_outer_knuckle_to_finger" type="fixed">
+      <origin xyz="0.03142 0 -0.00453" rpy="0 0 0" />
       <parent link="left_outer_knuckle" />
       <child link="left_outer_finger" />
     </joint>
-    <joint name="right_outer_finger_joint" type="fixed">
-      <origin xyz="-0.03156 0 -0.003758" rpy="0 0 0" />
+    <joint name="right_outer_knuckle_to_finger" type="fixed">
+      <origin xyz="-0.03142 0 -0.00453" rpy="0 0 0" />
       <parent link="right_outer_knuckle" />
       <child link="right_outer_finger" />
     </joint>
     <gazebo>
-      <joint name="left_finger_joint2" type="revolute">
-        <pose frame="">0.017901 0 0.00651469 0 0 0</pose>
+      <joint name="left_inner_knuckle_to_finger" type="revolute">
+        <pose frame="">-0.0179 0 0.00652 0 0 0</pose>
         <parent>${prefix}::left_inner_knuckle</parent>
         <child>${prefix}::left_inner_finger</child>
+        <axis>
+          <xyz>0 1 0</xyz>
+          <limit>
+            <lower>-0.8</lower>
+            <upper>0.8</upper>
+            <velocity>2.0</velocity>
+            <effort>1000</effort>
+          </limit>
+        </axis>
+      </joint>
+      <joint name="right_inner_knuckle_to_finger" type="revolute">
+        <pose frame="">0.0179 0 0.00652 0 0 0</pose>
+        <parent>${prefix}::right_inner_knuckle</parent>
+        <child>${prefix}::right_inner_finger</child>
         <axis>
           <xyz>0 -1 0</xyz>
@@ -339,22 +322,8 @@
         </axis>
       </joint>
-      <joint name="right_finger_joint2" type="revolute">
-        <pose frame="">0.017901 0 0.00651469 0 0 0</pose>
-        <parent>${prefix}::right_inner_knuckle</parent>
-        <child>${prefix}::right_inner_finger</child>
-        <axis>
-          <xyz>0 1 0</xyz>
-          <limit>
-            <lower>-0.8</lower>
-            <upper>0.8</upper>
-            <velocity>2.0</velocity>
-            <effort>1000</effort>
-          </limit>
-        </axis>
-      </joint>
       <plugin filename="librobotiq_gripper_gazebo_plugin.so" name="hrim_actuation_gripper_000000000004">
-        <joint>left_inner_knuckle_joint</joint>
-        <joint>left_outer_knuckle_joint</joint>
-        <joint>right_inner_knuckle_joint</joint>
+        <joint>robotiq_arg2f_base_link_to_left_inner_knuckle</joint>
+        <joint>robotiq_arg2f_base_link_to_left_outer_knuckle</joint>
+        <joint>robotiq_arg2f_base_link_to_right_inner_knuckle</joint>
         <joint>joint_finger</joint>
       </plugin>

Commit message: regenerate S85 urdf

File: robotiq_85_gripper_description/urdf/robotiq_85.urdf (robot description, URDF)
Before this commit: robot robotiq_85, 10 links, 9 joints
Joints:
- joint joint_finger: limit lower=0 upper=0.78 effort=1000 velocity=2.0 -> lower=0 upper=0.82589 effort=21.03 velocity=3.87
- joint left_outer_finger_to_inner: limit lower=0 upper=0.775 effort=1000 velocity=2.0 -> lower=0 upper=0.82589 effort=21.03 velocity=3.87
- joint right_outer_finger_to_inner: limit lower=0 upper=0.775 effort=1000 velocity=2.0 -> lower=0 upper=0.82589 effort=21.03 velocity=3.87
- joint robotiq_arg2f_base_link_to_left_inner_knuckle: limit lower=0 upper=0.8757 effort=1000 velocity=2.0 -> lower=0 upper=0.82589 effort=21.03 velocity=3.87
- joint robotiq_arg2f_base_link_to_left_outer_knuckle: limit lower=0.0 upper=0.78 effort=1000 velocity=2.0 -> lower=0 upper=0.82589 effort=21.03 velocity=3.87
- joint robotiq_arg2f_base_link_to_right_inner_knuckle: limit lower=0 upper=0.8757 effort=1000 velocity=2.0 -> lower=0 upper=0.82589 effort=21.03 velocity=3.87

Commit message: fix inertial values

File: robotiq_85_gripper_description/urdf/robotiq_85.urdf (robot description, URDF)
Before this commit: robot robotiq_85, 10 links, 9 joints
Links:
- link left_inner_finger: mass 0.22652 -> 0.037
- link left_inner_knuckle: mass 0.22652 -> 0.02731
- link left_outer_finger: mass 0.22652 -> 0.03848
- link left_outer_knuckle: mass 0.22652 -> 0.01252
- link right_inner_finger: mass 0.22652 -> 0.037
- link right_inner_knuckle: mass 0.22652 -> 0.02731
- link right_outer_finger: mass 0.22652 -> 0.03848
- link right_outer_knuckle: mass 0.22652 -> 0.01252
- link robotiq_arg2f_base_link: mass 0.22652 -> 0.55938

File: robotiq_85_gripper_description/urdf/robotiq_85.urdf.xacro (robot description, xacro)
@@ -4,7 +4,7 @@
     <link name="robotiq_arg2f_base_link">
       <inertial>
-        <origin xyz="8.625E-08 -4.6583E-06 0.03145" rpy="0 0 0" />
-        <mass value="0.22652" />
-        <inertia ixx="0.00020005" ixy="0" ixz="0" iyy="0.00017832" iyz="0" izz="0.00013478" />
+        <origin xyz="-0.00013 -0.00011 0.03284" rpy="0 0 0" />
+        <mass value="0.55938" />
+        <inertia ixx="605783E-9" ixy="-579.95E-9" ixz="2765.53E-9" iyy="720148E-9" iyz="618E-9" izz="510534E-9" />
       </inertial>
       <visual>
@@ -30,7 +30,7 @@
     <link name="left_outer_knuckle">
       <inertial>
-        <origin xyz="8.625E-08 -4.6583E-06 0.03145" rpy="0 0 0" />
-        <mass value="0.22652" />
-        <inertia ixx="0.00020005" ixy="0" ixz="0" iyy="0.00017832" iyz="0" izz="0.00013478" />
+        <origin xyz="0.01545 0 -0.00118" rpy="0 0 0" />
+        <mass value="0.01252" />
+        <inertia ixx="312.44E-9" ixy="0" ixz="-168.09E-9" iyy="2156E-9" iyz="0" izz="2027.51E-9" />
       </inertial>
       <visual>
@@ -56,7 +56,7 @@
     <link name="right_outer_knuckle">
       <inertial>
-        <origin xyz="8.625E-08 -4.6583E-06 0.03145" rpy="0 0 0" />
-        <mass value="0.22652" />
-        <inertia ixx="0.00020005" ixy="0" ixz="0" iyy="0.00017832" iyz="0" izz="0.00013478" />
+        <origin xyz="-0.01545 0 -0.00118" rpy="0 0 0" />
+        <mass value="0.01252" />
+        <inertia ixx="312.44E-9" ixy="0" ixz="-168.09E-9" iyy="2156E-9" iyz="0" izz="2027.51E-9" />
       </inertial>
       <visual>
@@ -82,7 +82,7 @@
     <link name="left_outer_finger">
       <inertial>
-        <origin xyz="8.625E-08 -4.6583E-06 0.03145" rpy="0 0 0" />
-        <mass value="0.22652" />
-        <inertia ixx="0.00020005" ixy="0" ixz="0" iyy="0.00017832" iyz="0" izz="0.00013478" />
+        <origin xyz="0.004 0 0.01892" rpy="0 0 0" />
+        <mass value="0.03848" />
+        <inertia ixx="12341E-9" ixy="0" ixz="-2152.21E-9" iyy="10617E-9" iyz="0" izz="4812.09E-9" />
       </inertial>
       <visual>
@@ -108,7 +108,7 @@
     <link name="right_outer_finger">
       <inertial>
-        <origin xyz="8.625E-08 -4.6583E-06 0.03145" rpy="0 0 0" />
-        <mass value="0.22652" />
-        <inertia ixx="0.00020005" ixy="0" ixz="0" iyy="0.00017832" iyz="0" izz="0.00013478" />
+        <origin xyz="-0.004 0 0.01892" rpy="0 0 0" />
+        <mass value="0.03848" />
+        <inertia ixx="12341E-9" ixy="0" ixz="-2152.21E-9" iyy="10617E-9" iyz="0" izz="4812.09E-9" />
       </inertial>
       <visual>
@@ -134,7 +134,7 @@
     <link name="left_inner_knuckle">
       <inertial>
-        <origin xyz="8.625E-08 -4.6583E-06 0.03145" rpy="0 0 0" />
-        <mass value="0.22652" />
-        <inertia ixx="0.00020005" ixy="0" ixz="0" iyy="0.00017832" iyz="0" izz="0.00013478" />
+        <origin xyz="0.01952 0 0.022" rpy="0 0 0" />
+        <mass value="0.02731" />
+        <inertia ixx="8621.3E-9" ixy="0" ixz="-3646.49E-9" iyy="8004.28E-9" iyz="0" izz="7704.42E-9" />
       </inertial>
       <visual>
@@ -160,7 +160,7 @@
     <link name="right_inner_knuckle">
       <inertial>
-        <origin xyz="8.625E-08 -4.6583E-06 0.03145" rpy="0 0 0" />
-        <mass value="0.22652" />
-        <inertia ixx="0.00020005" ixy="0" ixz="0" iyy="0.00017832" iyz="0" izz="0.00013478" />
+        <origin xyz="-0.01952 0 0.022" rpy="0 0 0" />
+        <mass value="0.02731" />
+        <inertia ixx="8621.3E-9" ixy="0" ixz="-3646.49E-9" iyy="8004.28E-9" iyz="0" izz="7704.42E-9" />
       </inertial>
       <visual>
@@ -186,7 +186,7 @@
     <link name="left_inner_finger">
       <inertial>
-        <origin xyz="8.625E-08 -4.6583E-06 0.03145" rpy="0 0 0" />
-        <mass value="0.22652" />
-        <inertia ixx="0.00020005" ixy="0" ixz="0" iyy="0.00017832" iyz="0" izz="0.00013478" />
+        <origin xyz="-0.01409 0 0.01569" rpy="0 0 0" />
+        <mass value="0.037" />
+        <inertia ixx="12446.57E-9" ixy="0" ixz="4167.81E-9" iyy="14201.18E-9" iyz="0" izz="4979.86E-9" />
       </inertial>
       <visual>
@@ -212,7 +212,7 @@
     <link name="right_inner_finger">
       <inertial>
-        <origin xyz="8.625E-08 -4.6583E-06 0.03145" rpy="0 0 0" />
-        <mass value="0.22652" />
-        <inertia ixx="0.00020005" ixy="0" ixz="0" iyy="0.00017832" iyz="0" izz="0.00013478" />
+        <origin xyz="0.01409 0 0.01569" rpy="0 0 0" />
+        <mass value="0.037" />
+        <inertia ixx="12446.57E-9" ixy="0" ixz="4167.81E-9" iyy="14201.18E-9" iyz="0" izz="4979.86E-9" />
       </inertial>
       <visual>

File: robotiq_85_gripper_description/urdf/robotiq_85_world.urdf.xacro (robot description, xacro)
@@ -1,5 +1,4 @@
 <?xml version="1.0"?>
 <robot xmlns:xacro="http://ros.org/wiki/xacro" name="robotiq_85" >
-  <!-- robotiq hande_gripper -->
   <xacro:include filename="$(find robotiq_85_gripper_description)/urdf/robotiq_85.urdf.xacro" />
   <xacro:robotiq_85 prefix="robotiq85"/>
@@ -10,12 +9,3 @@
     <child link="robotiq_arg2f_base_link"/>
   </joint>
-  <gazebo>
-    <plugin filename="libgazebo_ros_joint_state_publisher.so" name="mara_joint_state">
-      <ros>
-        <argument>~/out:=joint_states</argument>
-      </ros>
-      <update_rate>25</update_rate>
-      <joint_name>joint_finger</joint_name>
-    </plugin>
-  </gazebo>
 </robot>
