Commit message: ename multiple S85 and hande grippers

File: robotiq_85_gripper_description/urdf/robotiq_85.urdf (robot description, URDF)
Before this commit: robot robotiq_85, 10 links, 9 joints
Links:
- removed link left_inner_finger
- removed link left_inner_knuckle
- removed link left_outer_finger
- removed link left_outer_knuckle
- removed link right_inner_finger
- removed link right_inner_knuckle
- removed link right_outer_finger
- removed link right_outer_knuckle
- removed link robotiq_arg2f_base_link
- added link robotiq85left_inner_finger, mass 0.037; collision mesh filename=package://robotiq_85_gripper_description/meshes/2-F-85_4_l.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 scale=0.001 0.001 0.001; visual mesh filename=package://robotiq_85_gripper_description/meshes/2-F-85_4_l.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 scale=0.001 0.001 0.001
- added link robotiq85left_inner_knuckle, mass 0.02731; collision mesh filename=package://robotiq_85_gripper_description/meshes/2-F-85_2_l.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 scale=0.001 0.001 0.001; visual mesh filename=package://robotiq_85_gripper_description/meshes/2-F-85_2_l.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 scale=0.001 0.001 0.001
- added link robotiq85left_outer_finger, mass 0.03848; collision mesh filename=package://robotiq_85_gripper_description/meshes/2-F-85_3_l.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 scale=0.001 0.001 0.001; visual mesh filename=package://robotiq_85_gripper_description/meshes/2-F-85_3_l.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 scale=0.001 0.001 0.001
- added link robotiq85left_outer_knuckle, mass 0.01252; collision mesh filename=package://robotiq_85_gripper_description/meshes/2-F-85_1_l.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 scale=0.001 0.001 0.001; visual mesh filename=package://robotiq_85_gripper_description/meshes/2-F-85_1_l.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 scale=0.001 0.001 0.001
- added link robotiq85right_inner_finger, mass 0.037; collision mesh filename=package://robotiq_85_gripper_description/meshes/2-F-85_4_r.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 scale=0.001 0.001 0.001; visual mesh filename=package://robotiq_85_gripper_description/meshes/2-F-85_4_r.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 scale=0.001 0.001 0.001
- added link robotiq85right_inner_knuckle, mass 0.02731; collision mesh filename=package://robotiq_85_gripper_description/meshes/2-F-85_2_r.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 scale=0.001 0.001 0.001; visual mesh filename=package://robotiq_85_gripper_description/meshes/2-F-85_2_r.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 scale=0.001 0.001 0.001
- added link robotiq85right_outer_finger, mass 0.03848; collision mesh filename=package://robotiq_85_gripper_description/meshes/2-F-85_3_r.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 scale=0.001 0.001 0.001; visual mesh filename=package://robotiq_85_gripper_description/meshes/2-F-85_3_r.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 scale=0.001 0.001 0.001
- added link robotiq85right_outer_knuckle, mass 0.01252; collision mesh filename=package://robotiq_85_gripper_description/meshes/2-F-85_1_r.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 scale=0.001 0.001 0.001; visual mesh filename=package://robotiq_85_gripper_description/meshes/2-F-85_1_r.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 scale=0.001 0.001 0.001
- added link robotiq85robotiq_arg2f_base_link, mass 0.55938; collision mesh filename=package://robotiq_85_gripper_description/meshes/base_grippe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 scale=0.001 0.001 0.001; visual mesh filename=package://robotiq_85_gripper_description/meshes/base_grippe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 scale=0.001 0.001 0.001
Joints:
- removed joint joint_finger
- removed joint left_outer_finger_to_inner
- removed joint left_outer_knuckle_to_finger
- removed joint right_outer_finger_to_inner
- removed joint right_outer_knuckle_to_finger
- removed joint robotiq_arg2f_base_link_to_left_inner_knuckle
- removed joint robotiq_arg2f_base_link_to_left_outer_knuckle
- removed joint robotiq_arg2f_base_link_to_right_inner_knuckle
- added joint robotiq85joint_finger: type revolute, parent robotiq85robotiq_arg2f_base_link, child robotiq85right_outer_knuckle, origin xyz=-0.0306 0 0.05466 rpy=0 0 0, axis 0 1 0, limit lower=0 upper=0.82589 effort=21.03 velocity=3.87
- added joint robotiq85left_outer_finger_to_inner: type revolute, parent robotiq85left_outer_finger, child robotiq85left_inner_finger, origin xyz=0.00678 0 0.04703 rpy=0 0 0, axis 0 1 0, limit lower=0 upper=0.82589 effort=21.03 velocity=3.87, mimic joint=robotiq85joint_finger multiplier=1 offset=0
- added joint robotiq85left_outer_knuckle_to_finger: type fixed, parent robotiq85left_outer_knuckle, child robotiq85left_outer_finger, origin xyz=0.03142 0 -0.00453 rpy=0 0 0
- added joint robotiq85right_outer_finger_to_inner: type revolute, parent robotiq85right_outer_finger, child robotiq85right_inner_finger, origin xyz=-0.00678 0 0.04703 rpy=0 0 0, axis 0 -1 0, limit lower=0 upper=0.82589 effort=21.03 velocity=3.87, mimic joint=robotiq85joint_finger multiplier=1 offset=0
- added joint robotiq85right_outer_knuckle_to_finger: type fixed, parent robotiq85right_outer_knuckle, child robotiq85right_outer_finger, origin xyz=-0.03142 0 -0.00453 rpy=0 0 0
- added joint robotiq85robotiq_arg2f_base_link_to_robotiq85left_inner_knuckle: type revolute, parent robotiq85robotiq_arg2f_base_link, child robotiq85left_inner_knuckle, origin xyz=0.0127 0 0.06118 rpy=0 0 0, axis 0 -1 0, limit lower=0 upper=0.82589 effort=21.03 velocity=3.87, mimic joint=robotiq85joint_finger multiplier=1 offset=0
- added joint robotiq85robotiq_arg2f_base_link_to_robotiq85left_outer_knuckle: type revolute, parent robotiq85robotiq_arg2f_base_link, child robotiq85left_outer_knuckle, origin xyz=0.0306 0 0.05466 rpy=0 0 0, axis 0 -1 0, limit lower=0 upper=0.82589 effort=21.03 velocity=3.87, mimic joint=robotiq85joint_finger multiplier=1 offset=0
- added joint robotiq85robotiq_arg2f_base_link_to_robotiq85right_inner_knuckle: type revolute, parent robotiq85robotiq_arg2f_base_link, child robotiq85right_inner_knuckle, origin xyz=-0.0127 0 0.06118 rpy=0 0 0, axis 0 1 0, limit lower=0 upper=0.82589 effort=21.03 velocity=3.87, mimic joint=robotiq85joint_finger multiplier=1 offset=0

File: robotiq_85_gripper_description/urdf/robotiq_85.urdf.xacro (robot description, xacro)
@@ -1,6 +1,6 @@
 <?xml version="1.0"?>
 <robot xmlns:xacro="http://ros.org/wiki/xacro">
-  <xacro:macro name="robotiq_85"  params="prefix">
-    <link name="robotiq_arg2f_base_link">
+  <xacro:macro name="robotiq_85"  params="prefix MAC">
+    <link name="${prefix}robotiq_arg2f_base_link">
       <inertial>
         <origin xyz="-0.00013 -0.00011 0.03284" rpy="0 0 0" />
@@ -24,9 +24,9 @@
       </collision>
     </link>
-    <gazebo reference="robotiq_arg2f_base_link">
-      <material>Gazebo/Black</material>
-      <selfCollide>True</selfCollide>
-    </gazebo>
-    <link name="left_outer_knuckle">
+    <gazebo reference="${prefix}robotiq_arg2f_base_link">
+      <material>Gazebo/Black</material>
+      <selfCollide>True</selfCollide>
+    </gazebo>
+    <link name="${prefix}left_outer_knuckle">
       <inertial>
         <origin xyz="0.01545 0 -0.00118" rpy="0 0 0" />
@@ -50,9 +50,9 @@
       </collision>
     </link>
-    <gazebo reference="left_outer_knuckle">
+    <gazebo reference="${prefix}left_outer_knuckle">
       <material>Gazebo/Grey</material>
       <selfCollide>True</selfCollide>
     </gazebo>
-    <link name="right_outer_knuckle">
+    <link name="${prefix}right_outer_knuckle">
       <inertial>
         <origin xyz="-0.01545 0 -0.00118" rpy="0 0 0" />
@@ -76,9 +76,9 @@
       </collision>
     </link>
-    <gazebo reference="right_outer_knuckle">
+    <gazebo reference="${prefix}right_outer_knuckle">
       <material>Gazebo/Grey</material>
       <selfCollide>True</selfCollide>
     </gazebo>
-    <link name="left_outer_finger">
+    <link name="${prefix}left_outer_finger">
       <inertial>
         <origin xyz="0.004 0 0.01892" rpy="0 0 0" />
@@ -102,9 +102,9 @@
       </collision>
     </link>
-    <gazebo reference="left_outer_finger">
-      <material>Gazebo/Black</material>
-      <selfCollide>True</selfCollide>
-    </gazebo>
-    <link name="right_outer_finger">
+    <gazebo reference="${prefix}left_outer_finger">
+      <material>Gazebo/Black</material>
+      <selfCollide>True</selfCollide>
+    </gazebo>
+    <link name="${prefix}right_outer_finger">
       <inertial>
         <origin xyz="-0.004 0 0.01892" rpy="0 0 0" />
@@ -128,9 +128,9 @@
       </collision>
     </link>
-    <gazebo reference="right_outer_finger">
-      <material>Gazebo/Black</material>
-      <selfCollide>True</selfCollide>
-    </gazebo>
-    <link name="left_inner_knuckle">
+    <gazebo reference="${prefix}right_outer_finger">
+      <material>Gazebo/Black</material>
+      <selfCollide>True</selfCollide>
+    </gazebo>
+    <link name="${prefix}left_inner_knuckle">
       <inertial>
         <origin xyz="0.01952 0 0.022" rpy="0 0 0" />
@@ -154,9 +154,9 @@
       </collision>
     </link>
-    <gazebo reference="left_inner_knuckle">
+    <gazebo reference="${prefix}left_inner_knuckle">
       <material>Gazebo/Black</material>
       <selfCollide>False</selfCollide>
     </gazebo>
-    <link name="right_inner_knuckle">
+    <link name="${prefix}right_inner_knuckle">
       <inertial>
         <origin xyz="-0.01952 0 0.022" rpy="0 0 0" />
@@ -180,9 +180,9 @@
       </collision>
     </link>
-    <gazebo reference="right_inner_knuckle">
+    <gazebo reference="${prefix}right_inner_knuckle">
       <material>Gazebo/Black</material>
       <selfCollide>False</selfCollide>
     </gazebo>
-    <link name="left_inner_finger">
+    <link name="${prefix}left_inner_finger">
       <inertial>
         <origin xyz="-0.01409 0 0.01569" rpy="0 0 0" />
@@ -206,9 +206,9 @@
       </collision>
     </link>
-    <gazebo reference="left_inner_finger">
+    <gazebo reference="${prefix}left_inner_finger">
       <material>Gazebo/Black</material>
       <selfCollide>False</selfCollide>
     </gazebo>
-    <link name="right_inner_finger">
+    <link name="${prefix}right_inner_finger">
       <inertial>
         <origin xyz="0.01409 0 0.01569" rpy="0 0 0" />
@@ -232,70 +232,70 @@
       </collision>
     </link>
-    <gazebo reference="right_inner_finger">
+    <gazebo reference="${prefix}right_inner_finger">
       <material>Gazebo/Black</material>
       <selfCollide>False</selfCollide>
     </gazebo>
-    <joint name="robotiq_arg2f_base_link_to_left_outer_knuckle" type="revolute">
+    <joint name="${prefix}robotiq_arg2f_base_link_to_${prefix}left_outer_knuckle" type="revolute">
       <origin xyz="0.0306 0 0.05466" rpy="0 0 0" />
-      <parent link="robotiq_arg2f_base_link" />
-      <child link="left_outer_knuckle" />
+      <parent link="${prefix}robotiq_arg2f_base_link" />
+      <child link="${prefix}left_outer_knuckle" />
       <axis xyz="0 -1 0" />
       <limit lower="0" upper="0.82589" velocity="3.87" effort="21.03" />
-      <mimic joint="joint_finger" multiplier="1" offset="0"/>
-    </joint>
-    <joint name="joint_finger" type="revolute">
+      <mimic joint="${prefix}joint_finger" multiplier="1" offset="0"/>
+    </joint>
+    <joint name="${prefix}joint_finger" type="revolute">
       <origin xyz="-0.0306 0 0.05466" rpy="0 0 0" />
-      <parent link="robotiq_arg2f_base_link" />
-      <child link="right_outer_knuckle" />
+      <parent link="${prefix}robotiq_arg2f_base_link" />
+      <child link="${prefix}right_outer_knuckle" />
       <axis xyz="0 1 0" />
       <limit lower="0" upper="0.82589" velocity="3.87" effort="21.03" />
     </joint>
-    <joint name="robotiq_arg2f_base_link_to_left_inner_knuckle" type="revolute">
+    <joint name="${prefix}robotiq_arg2f_base_link_to_${prefix}left_inner_knuckle" type="revolute">
       <origin xyz="0.0127 0 0.06118" rpy="0 0 0" />
-      <parent link="robotiq_arg2f_base_link" />
-      <child link="left_inner_knuckle" />
+      <parent link="${prefix}robotiq_arg2f_base_link" />
+      <child link="${prefix}left_inner_knuckle" />
       <axis xyz="0 -1 0" />
       <limit lower="0" upper="0.82589" velocity="3.87" effort="21.03" />
-      <mimic joint="joint_finger" multiplier="1" offset="0"/>
-    </joint>
-    <joint name="robotiq_arg2f_base_link_to_right_inner_knuckle" type="revolute">
+      <mimic joint="${prefix}joint_finger" multiplier="1" offset="0"/>
+    </joint>
+    <joint name="${prefix}robotiq_arg2f_base_link_to_${prefix}right_inner_knuckle" type="revolute">
       <origin xyz="-0.0127 0 0.06118" rpy="0 0 0" />
-      <parent link="robotiq_arg2f_base_link" />
-      <child link="right_inner_knuckle" />
+      <parent link="${prefix}robotiq_arg2f_base_link" />
+      <child link="${prefix}right_inner_knuckle" />
       <axis xyz="0 1 0" />
       <limit lower="0" upper="0.82589" velocity="3.87" effort="21.03" />
-      <mimic joint="joint_finger" multiplier="1" offset="0"/>
-    </joint>
-    <joint name="left_outer_finger_to_inner" type="revolute">
+      <mimic joint="${prefix}joint_finger" multiplier="1" offset="0"/>
+    </joint>
+    <joint name="${prefix}left_outer_finger_to_inner" type="revolute">
       <origin xyz="0.00678 0 0.04703" rpy="0 0 0" />
-      <parent link="left_outer_finger" />
-      <child link="left_inner_finger" />
+      <parent link="${prefix}left_outer_finger" />
+      <child link="${prefix}left_inner_finger" />
       <axis xyz="0 1 0" />
       <limit lower="0" upper="0.82589" velocity="3.87" effort="21.03" />
-      <mimic joint="joint_finger" multiplier="1" offset="0"/>
-    </joint>
-    <joint name="right_outer_finger_to_inner" type="revolute">
+      <mimic joint="${prefix}joint_finger" multiplier="1" offset="0"/>
+    </joint>
+    <joint name="${prefix}right_outer_finger_to_inner" type="revolute">
       <origin xyz="-0.00678 0 0.04703" rpy="0 0 0" />
-      <parent link="right_outer_finger" />
-      <child link="right_inner_finger" />
+      <parent link="${prefix}right_outer_finger" />
+      <child link="${prefix}right_inner_finger" />
       <axis xyz="0 -1 0" />
       <limit lower="0" upper="0.82589" velocity="3.87" effort="21.03" />
-      <mimic joint="joint_finger" multiplier="1" offset="0"/>
-    </joint>
-    <joint name="left_outer_knuckle_to_finger" type="fixed">
+      <mimic joint="${prefix}joint_finger" multiplier="1" offset="0"/>
+    </joint>
+    <joint name="${prefix}left_outer_knuckle_to_finger" type="fixed">
       <origin xyz="0.03142 0 -0.00453" rpy="0 0 0" />
-      <parent link="left_outer_knuckle" />
-      <child link="left_outer_finger" />
-    </joint>
-    <joint name="right_outer_knuckle_to_finger" type="fixed">
+      <parent link="${prefix}left_outer_knuckle" />
+      <child link="${prefix}left_outer_finger" />
+    </joint>
+    <joint name="${prefix}right_outer_knuckle_to_finger" type="fixed">
       <origin xyz="-0.03142 0 -0.00453" rpy="0 0 0" />
-      <parent link="right_outer_knuckle" />
-      <child link="right_outer_finger" />
+      <parent link="${prefix}right_outer_knuckle" />
+      <child link="${prefix}right_outer_finger" />
     </joint>
     <gazebo>
-      <joint name="left_inner_knuckle_to_finger" type="revolute">
+      <joint name="${prefix}left_inner_knuckle_to_finger" type="revolute">
         <pose frame="">-0.0179 0 0.00652 0 0 0</pose>
-        <parent>${prefix}::left_inner_knuckle</parent>
-        <child>${prefix}::left_inner_finger</child>
+        <parent>${prefix}left_inner_knuckle</parent>
+        <child>${prefix}left_inner_finger</child>
         <axis>
           <xyz>0 1 0</xyz>
@@ -308,8 +308,8 @@
         </axis>
       </joint>
-      <joint name="right_inner_knuckle_to_finger" type="revolute">
+      <joint name="${prefix}right_inner_knuckle_to_finger" type="revolute">
         <pose frame="">0.0179 0 0.00652 0 0 0</pose>
-        <parent>${prefix}::right_inner_knuckle</parent>
-        <child>${prefix}::right_inner_finger</child>
+        <parent>${prefix}right_inner_knuckle</parent>
+        <child>${prefix}right_inner_finger</child>
         <axis>
           <xyz>0 -1 0</xyz>
@@ -322,12 +322,12 @@
         </axis>
       </joint>
-      <plugin filename="librobotiq_gripper_gazebo_plugin.so" name="hrim_actuation_gripper_000000000004">
+      <plugin filename="librobotiq_gripper_gazebo_plugin.so" name="hrim_actuator_gripper${MAC}">
         <kp>10</kp>
         <ki>10</ki>
         <kd>0.1</kd>
-        <joint>robotiq_arg2f_base_link_to_left_inner_knuckle</joint>
-        <joint>robotiq_arg2f_base_link_to_left_outer_knuckle</joint>
-        <joint>robotiq_arg2f_base_link_to_right_inner_knuckle</joint>
-        <joint>joint_finger</joint>
+        <joint>${prefix}robotiq_arg2f_base_link_to_${prefix}left_inner_knuckle</joint>
+        <joint>${prefix}robotiq_arg2f_base_link_to_${prefix}left_outer_knuckle</joint>
+        <joint>${prefix}robotiq_arg2f_base_link_to_${prefix}right_inner_knuckle</joint>
+        <joint>${prefix}joint_finger</joint>
       </plugin>
       <plugin filename="libgazebo_ros_joint_state_publisher.so" name="mara_joint_state">
@@ -336,5 +336,5 @@
         </ros>
         <update_rate>25</update_rate>
-        <joint_name>joint_finger</joint_name>
+        <joint_name>${prefix}joint_finger</joint_name>
       </plugin>
     </gazebo>

File: robotiq_85_gripper_description/urdf/robotiq_85_world.urdf.xacro (robot description, xacro)
@@ -2,5 +2,5 @@
 <robot xmlns:xacro="http://ros.org/wiki/xacro" name="robotiq_85" >
   <xacro:include filename="$(find robotiq_85_gripper_description)/urdf/robotiq_85.urdf.xacro" />
-  <xacro:robotiq_85 prefix="robotiq85"/>
+  <xacro:robotiq_85 prefix="robotiq85" MAC="_000000000004"/>
   <link name="world" />
   <joint name="world_to_robotiq_arg2f_base" type="fixed">

File: robotiq_hande_gripper_description/urdf/robotiq_hande.urdf (robot description, URDF)
Before this commit: robot robotiq_hande, 4 links, 3 joints
Links:
- removed link left_finger
- removed link right_finger
- removed link robotiq_hande_base_link
- added link handeleft_finger, mass 0.03804; collision mesh filename=package://robotiq_hande_gripper_description/meshes/finger_1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 scale=0.001 0.001 0.001; visual mesh filename=package://robotiq_hande_gripper_description/meshes/finger_1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 scale=0.001 0.001 0.001
- added link handeright_finger, mass 0.03804; collision mesh filename=package://robotiq_hande_gripper_description/meshes/finger_2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 scale=0.001 0.001 0.001; visual mesh filename=package://robotiq_hande_gripper_description/meshes/finger_2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 scale=0.001 0.001 0.001
- added link handerobotiq_hande_base_link, mass 0.86387; collision mesh filename=package://robotiq_hande_gripper_description/meshes/hand-e.d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 scale=0.001 0.001 0.001; visual mesh filename=package://robotiq_hande_gripper_description/meshes/hand-e.d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 scale=0.001 0.001 0.001
Joints:
- removed joint joint_finger
- removed joint robotiq_hande_base_to_right_finger
- added joint handejoint_finger: type prismatic, parent handerobotiq_hande_base_link, child handeleft_finger, origin xyz=0 0 0.099 rpy=0 0 0, axis -1 0 0, limit lower=0 upper=0.025 effort=130 velocity=0.15
- added joint robotiq_hande_base_to_handeright_finger: type prismatic, parent handerobotiq_hande_base_link, child handeright_finger, origin xyz=0 0 0.099 rpy=0 0 0, axis 1 0 0, limit lower=0 upper=0.025 effort=130 velocity=0.15, mimic joint=handejoint_finger multiplier=1 offset=0

File: robotiq_hande_gripper_description/urdf/robotiq_hande.urdf.xacro (robot description, xacro)
@@ -1,6 +1,6 @@
 <?xml version="1.0"?>
 <robot xmlns:xacro="http://ros.org/wiki/xacro">
-  <xacro:macro name="robotiq_hande"  params="prefix">
-    <link name="robotiq_hande_base_link">
+  <xacro:macro name="robotiq_hande"  params="prefix MAC">
+    <link name="${prefix}robotiq_hande_base_link">
       <inertial>
         <origin xyz="0 0 0.04607" rpy="0 0 0" />
@@ -24,9 +24,9 @@
       </collision>
     </link>
-    <gazebo reference="robotiq_hande_base_link">
+    <gazebo reference="${prefix}robotiq_hande_base_link">
       <material>Gazebo/Black</material>
       <selfCollide>True</selfCollide>
     </gazebo>
-    <link name="left_finger">
+    <link name="${prefix}left_finger">
       <inertial>
         <origin rpy="0 0 0" xyz="0.02262 -0.00759 0.00738"/>
@@ -50,9 +50,9 @@
       </collision>
     </link>
-    <gazebo reference="left_finger">
+    <gazebo reference="${prefix}left_finger">
       <material>Gazebo/Grey</material>
       <selfCollide>True</selfCollide>
     </gazebo>
-    <link name="right_finger">
+    <link name="${prefix}right_finger">
       <inertial>
         <origin rpy="0 0 0" xyz="-0.02262 0.00759 0.00738"/>
@@ -76,30 +76,30 @@
       </collision>
     </link>
-    <gazebo reference="right_finger">
+    <gazebo reference="${prefix}right_finger">
       <material>Gazebo/Grey</material>
       <selfCollide>True</selfCollide>
     </gazebo>
-    <joint name="joint_finger" type="prismatic">
+    <joint name="${prefix}joint_finger" type="prismatic">
       <origin rpy="0 0 0" xyz="0 0 0.099"/>
-      <parent link="robotiq_hande_base_link"/>
-      <child link="left_finger"/>
+      <parent link="${prefix}robotiq_hande_base_link"/>
+      <child link="${prefix}left_finger"/>
       <axis xyz="-1 0 0"/>
       <limit effort="130" lower="0" upper="0.025" velocity="0.15"/>
     </joint>
-    <joint name="robotiq_hande_base_to_right_finger" type="prismatic">
+    <joint name="robotiq_hande_base_to_${prefix}right_finger" type="prismatic">
       <origin rpy="0 0 0" xyz="0 0 0.099"/>
-      <parent link="robotiq_hande_base_link"/>
-      <child link="right_finger"/>
+      <parent link="${prefix}robotiq_hande_base_link"/>
+      <child link="${prefix}right_finger"/>
       <axis xyz="1 0 0"/>
       <limit effort="130" lower="0" upper="0.025" velocity="0.15"/>
-      <mimic joint="joint_finger" multiplier="1" offset="0"/>
+      <mimic joint="${prefix}joint_finger" multiplier="1" offset="0"/>
     </joint>
     <gazebo>
-      <plugin filename="librobotiq_gripper_gazebo_plugin.so" name="hrim_actuation_gripper_000000000004">
+      <plugin filename="librobotiq_gripper_gazebo_plugin.so" name="hrim_actuator_gripper${MAC}">
         <kp>500</kp>
         <ki>3</ki>
         <kd>9</kd>
-        <joint>joint_finger</joint>
-        <joint>robotiq_hande_base_to_right_finger</joint>
+        <joint>${prefix}joint_finger</joint>
+        <joint>robotiq_hande_base_to_${prefix}right_finger</joint>
       </plugin>
       <plugin filename="libgazebo_ros_joint_state_publisher.so" name="mara_joint_state">
@@ -108,5 +108,5 @@
         </ros>
         <update_rate>25</update_rate>
-        <joint_name>joint_finger</joint_name>
+        <joint_name>${prefix}joint_finger</joint_name>
       </plugin>
     </gazebo>

File: robotiq_hande_gripper_description/urdf/robotiq_hande_world.urdf.xacro (robot description, xacro)
@@ -3,5 +3,5 @@
   <!-- robotiq_hande_gripper -->
   <xacro:include filename="$(find robotiq_hande_gripper_description)/urdf/robotiq_hande.urdf.xacro" />
-  <xacro:robotiq_hande prefix=""/>
+  <xacro:robotiq_hande prefix="hande" MAC="_000000000004"/>
   <link name="world" />
   <joint name="world_to_robotiq_adapter" type="fixed">
